File: modules/MPU-65X/system.kicad_sch (KiCad schematic)
At the start: 2 parts, among them J1 CardConnector

Commit message: mpu-65x circuit & pcb
Parts:
- added C10, C11, C12, C6, C7, C8, C9: 100nF, IMNOTWOPR:C_Rect_P200mil, symbol IMNOTWOPR:C
- added U3: 74NC00, IMNOTWOPR:DIP-14N, symbol IMNOTWOPR:7400
- renumbered J1 to J2
Connections:
- net GND: now also C10.2, C11.2, C12.2, C6.2, C7.2, C8.2, C9.2, U3.7 (GND)
- net VCC: now also C10.1, C11.1, C12.1, C6.1, C7.1, C8.1, C9.1, U3.14 (VCC)

Commit message: Formatting and MPU-65X work
Connections:
- net ~{RESET}: now reaches J2.b15 (~{RESET})
- no-connect marks 78 -> 77
Changed lines of the file:
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@@
-	)
-	(no_connect
-		(at 63.5 60.96)
 	)
 	(no_connect
@@
 			(hide yes)
 			(show_name no)
+			(do_not_autoplace no)
+			(effects
+				(font
+					(size 1.27 1.27)
+				)
+				(justify right)
+			)
+		)
+	)
+	(global_label "~{RESET}"
+		(shape passive)
+		(at 63.5 60.96 180)
+		(fields_autoplaced yes)
+		(effects
+			(font
+				(size 1.27 1.27)
+			)
+			(justify right)
+		)
+		(property "Intersheetrefs" "${INTERSHEET_REFS}"
+			(at 55.6906 60.96 0)
+			(hide yes)
+			(show_name no)
