File: modules/PWR-CTRL/system.kicad_sch (KiCad schematic)
At the start: 2 parts, among them J1 CardConnector

Commit message: added joshua
Connections:
- net +12V: no longer J1.a3 (+12V)
- net +12V2: no longer J1.c3 (+12V2)
- net +5V: no longer J1.a1 (+5V), J1.a2 (+5V), J1.a31 (+5V), J1.a32 (+5V), J1.b32 (+5V)
- net -12V: no longer J1.b3 (-12V)
- net GND: no longer J1.b31 (GND), J1.c12 (GND), J1.c18 (GND), J1.c24 (GND), J1.c31 (GND), J1.c32 (GND), J1.c6 (GND)
- no-connect marks 71 -> 83

Commit message: added i2c pullups to pwr-ctrl
Connections:
- net +5V: now also J1.a1 (+5V), J1.a2 (+5V)
- net I2C_SCL: now reaches J1.c7 (RESERVED)
- net I2C_SDA: now reaches J1.c8 (RESERVED)
- no-connect marks 83 -> 82
Changed lines of the file:
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@@
+	)
+	(no_connect
+		(at 101.6 68.58)
 	)
 	(no_connect
@@
 	)
 	(no_connect
-		(at 101.6 40.64)
-	)
-	(no_connect
 		(at 101.6 30.48)
 	)
@@
 	)
 	(no_connect
+		(at 101.6 83.82)
+	)
+	(no_connect
 		(at 63.5 63.5)
 	)
@@
 	)
 	(no_connect
-		(at 101.6 43.18)
-	)
-	(no_connect
-		(at 25.4 25.4)
-	)
-	(no_connect
 		(at 101.6 76.2)
 	)
@@
 	)
 	(no_connect
-		(at 25.4 27.94)
-	)
-	(no_connect
 		(at 101.6 78.74)
 	)
@@
 	(no_connect
 		(at 25.4 38.1)
+	)
+	(no_connect
+		(at 101.6 53.34)
 	)
 	(no_connect
@@
 		)
 	)
+	(global_label "+5V"
+		(shape output)
+		(at 25.4 27.94 180)
+		(fields_autoplaced yes)
+		(effects
+			(font
+				(size 1.27 1.27)
+			)
+			(justify right)
+		)
+		(property "Intersheetrefs" "${INTERSHEET_REFS}"
+			(at 18.4492 27.94 0)
+			(hide yes)
+			(show_name no)
+			(do_not_autoplace no)
+			(effects
+				(font
+					(size 1.27 1.27)
+				)
+				(justify right)
+			)
+		)
+	)
 	(global_label "PWROK"
 		(shape output)
@@
 		)
 	)
+	(global_label "I2C_SDA"
+		(shape passive)
+		(at 101.6 43.18 180)
+		(fields_autoplaced yes)
+		(effects
+			(font
+				(size 1.27 1.27)
+			)
+			(justify right)
+		)
+		(property "Intersheetrefs" "${INTERSHEET_REFS}"
+			(at 91.9157 43.18 0)
+			(hide yes)
+			(show_name no)
+			(do_not_autoplace no)
+			(effects
+				(font
+					(size 1.27 1.27)
+				)
+				(justify right)
+			)
+		)
+	)
 	(global_label "GND"
 		(shape output)
@@
 		(property "Intersheetrefs" "${INTERSHEET_REFS}"
 			(at 93.4743 27.94 0)
+			(hide yes)
+			(show_name no)
+			(do_not_autoplace no)
+			(effects
+				(font
+					(size 1.27 1.27)
+				)
+				(justify right)
+			)
+		)
+	)
+	(global_label "+5V"
+		(shape output)
+		(at 25.4 25.4 180)
+		(fields_autoplaced yes)
+		(effects
+			(font
+				(size 1.27 1.27)
+			)
+			(justify right)
+		)
+		(property "Intersheetrefs" "${INTERSHEET_REFS}"
+			(at 18.4492 25.4 0)
 			(hide yes)
 			(show_name no)
@@
 			(hide yes)
 			(show_name no)
+			(do_not_autoplace no)
+			(effects
+				(font
+					(size 1.27 1.27)
+				)
+				(justify right)
+			)
+		)
+	)
+	(global_label "I2C_SCL"
+		(shape passive)
+		(at 101.6 40.64 180)
+		(fields_autoplaced yes)
+		(effects
+			(font
+				(size 1.27 1.27)
+			)
+			(justify right)
+		)
+		(property "Intersheetrefs" "${INTERSHEET_REFS}"
+			(at 91.9762 40.64 0)
+			(hide yes)
+			(show_name no)
