File: modules/MSD-65/system.kicad_sch (KiCad schematic)
At the start: 2 parts, among them J1 CardConnector

Commit message: added bus line analyzer
Parts:
- renumbered J1 to J2
Connections:
- net SPI_MOSI: now reaches J2.c10 (SPI_MOSI)
- net SPI_MISO: now reaches J2.c11 (SPI_MISO)
- net SPI_SCK: now reaches J2.c9 (SPI_SCK)
- no-connect marks 80 -> 77
Other:
- title: TITLE -> MSD-65
Changed lines of the file:
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@@
 	(paper "A4")
 	(title_block
-		(title "TITLE")
+		(title "MSD-65")
 		(rev "A")
 		(company "THE HOUSE OF GALAHAD")
 		(comment 1 "IMNOTWOPR")
-		(comment 2 "CARD TEMPLATE")
+		(comment 2 "microSD CARD READER")
 	)
 	(junction
@@
 	)
 	(no_connect
-		(at 101.6 45.72)
-	)
-	(no_connect
 		(at 25.4 81.28)
 	)
@@
 	)
 	(no_connect
-		(at 101.6 48.26)
-	)
-	(no_connect
 		(at 63.5 60.96)
 	)
@@
 	(no_connect
 		(at 25.4 58.42)
-	)
-	(no_connect
-		(at 101.6 50.8)
 	)
 	(no_connect
@@
 		)
 	)
+	(global_label "SPI_SCK"
+		(shape passive)
+		(at 101.6 45.72 180)
+		(fields_autoplaced yes)
+		(effects
+			(font
+				(size 1.27 1.27)
+			)
+			(justify right)
+		)
+		(property "Intersheetrefs" "${INTERSHEET_REFS}"
+			(at 91.7343 45.72 0)
+			(hide yes)
+			(show_name no)
+			(do_not_autoplace no)
+			(effects
+				(font
+					(size 1.27 1.27)
+				)
+				(justify right)
+			)
+		)
+	)
 	(global_label "GND"
 		(shape output)
@@
 		)
 	)
+	(global_label "SPI_MISO"
+		(shape passive)
+		(at 101.6 50.8 180)
+		(fields_autoplaced yes)
+		(effects
+			(font
+				(size 1.27 1.27)
+			)
+			(justify right)
+		)
+		(property "Intersheetrefs" "${INTERSHEET_REFS}"
+			(at 90.8876 50.8 0)
+			(hide yes)
+			(show_name no)
+			(do_not_autoplace no)
+			(effects
+				(font
+					(size 1.27 1.27)
+				)
+				(justify right)
+			)
+		)
+	)
 	(global_label "GND"
 		(shape output)
@@
 		(property "Intersheetrefs" "${INTERSHEET_REFS}"
 			(at 93.4743 27.94 0)
+			(hide yes)
+			(show_name no)
+			(do_not_autoplace no)
+			(effects
+				(font
+					(size 1.27 1.27)
+				)
+				(justify right)
+			)
+		)
+	)
+	(global_label "SPI_MOSI"
+		(shape passive)
+		(at 101.6 48.26 180)
+		(fields_autoplaced yes)
+		(effects
+			(font
+				(size 1.27 1.27)
+			)
+			(justify right)
+		)
+		(property "Intersheetrefs" "${INTERSHEET_REFS}"
+			(at 90.8876 48.26 0)
 			(hide yes)
 			(show_name no)
@@
 		(in_pos_files yes)
 		(dnp no)
-		(property "Reference" "J1"
+		(property "Reference" "J2"
 			(at 73.66 22.86 0)
 			(show_name no)
@@
 		)
 		(instances
-			(project "TEMPLATE"
+			(project "MSD-65"
 				(path "/1bc24577-9a03-4fc2-ac64-d8d0370a6427"
-					(reference "J1")
+					(reference "J2")
 					(unit 2)
 				)
@@
 		(in_pos_files yes)
 		(dnp no)
-		(property "Reference" "J1"
+		(property "Reference" "J2"
 			(at 111.76 22.86 0)
 			(show_name no)
@@
 		)
 		(instances
-			(project "TEMPLATE"
+			(project "MSD-65"
 				(path "/1bc24577-9a03-4fc2-ac64-d8d0370a6427"
-					(reference "J1")
+					(reference "J2")
 					(unit 3)
 				)
@@
 		)
 		(instances
-			(project "TEMPLATE"
+			(project "MSD-65"
 				(path "/1bc24577-9a03-4fc2-ac64-d8d0370a6427"
 					(reference "#FLG01")
@@
 		(in_pos_files yes)
 		(dnp no)
-		(property "Reference" "J1"
+		(property "Reference" "J2"
 			(at 35.56 22.86 0)
 			(show_name no)
@@
 		)
 		(instances
-			(project "TEMPLATE"
+			(project "MSD-65"
 				(path "/1bc24577-9a03-4fc2-ac64-d8d0370a6427"
-					(reference "J1")
+					(reference "J2")
 					(unit 1)
 				)
@@
 		)
 		(instances
-			(project "TEMPLATE"
+			(project "MSD-65"
 				(path "/1bc24577-9a03-4fc2-ac64-d8d0370a6427"
 					(reference "MH1")
@@
 		)
 		(instances
-			(project "TEMPLATE"
+			(project "MSD-65"
 				(path "/1bc24577-9a03-4fc2-ac64-d8d0370a6427"
 					(reference "#FLG02")
