File: modules/PWR/system.kicad_sch (KiCad schematic)
At the start: 2 parts, among them J1 CardConnector

Commit message: pwr pcb
Other:
- title: PWR-CTRL -> PWR
Changed lines of the file:
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@@
 	(paper "A4")
 	(title_block
-		(title "PWR-CTRL")
+		(title "PWR")
 		(rev "A")
 		(company "THE HOUSE OF GALAHAD")
 		(comment 1 "IMNOTWOPR")
 		(comment 2 "POWER CONTROL")
+		(comment 3 "75-1010-01")
 	)
 	(junction
@@
 		)
 		(instances
-			(project "PWR-CTRL"
+			(project "PWR"
 				(path "/1bc24577-9a03-4fc2-ac64-d8d0370a6427"
 					(reference "J1")
@@
 		)
 		(instances
-			(project "PWR-CTRL"
+			(project "PWR"
 				(path "/1bc24577-9a03-4fc2-ac64-d8d0370a6427"
 					(reference "#FLG04")
@@
 		)
 		(instances
-			(project "PWR-CTRL"
+			(project "PWR"
 				(path "/1bc24577-9a03-4fc2-ac64-d8d0370a6427"
 					(reference "#FLG07")
@@
 		)
 		(instances
-			(project "PWR-CTRL"
+			(project "PWR"
 				(path "/1bc24577-9a03-4fc2-ac64-d8d0370a6427"
 					(reference "J1")
@@
 		)
 		(instances
-			(project "PWR-CTRL"
+			(project "PWR"
 				(path "/1bc24577-9a03-4fc2-ac64-d8d0370a6427"
 					(reference "#FLG01")
@@
 		)
 		(instances
-			(project "PWR-CTRL"
+			(project "PWR"
 				(path "/1bc24577-9a03-4fc2-ac64-d8d0370a6427"
 					(reference "J1")
@@
 		)
 		(instances
-			(project "PWR-CTRL"
+			(project "PWR"
 				(path "/1bc24577-9a03-4fc2-ac64-d8d0370a6427"
 					(reference "MH1")
@@
 		)
 		(instances
-			(project "PWR-CTRL"
+			(project "PWR"
 				(path "/1bc24577-9a03-4fc2-ac64-d8d0370a6427"
 					(reference "#FLG03")
@@
 		)
 		(instances
-			(project "PWR-CTRL"
+			(project "PWR"
 				(path "/1bc24577-9a03-4fc2-ac64-d8d0370a6427"
 					(reference "#FLG06")
@@
 		)
 		(instances
-			(project "PWR-CTRL"
+			(project "PWR"
 				(path "/1bc24577-9a03-4fc2-ac64-d8d0370a6427"
 					(reference "#FLG05")
