File: modules/BLA/BLA.kicad_pcb (KiCad board)
At the start: 2 copper layers, 160 x 100 mm, 152 parts, among them J1 CardConnector, U1 74HCT245N, U2 74HCT245N, U3 74HCT245N, U4 74HCT245N, U5 74HCT245N, U6 74HCT245N

Commit message: bla pcb and schematic
Parts:
- added C1: 100n, IMNOTWOPR:C_Rect_P200mil, F.Cu at (137.5, 95.0)
- added C2: 100n, IMNOTWOPR:C_Rect_P200mil, F.Cu at (137.5, 99.4)
- added C3: 100n, IMNOTWOPR:C_Rect_P200mil, F.Cu at (137.5, 103.9)
- added C4: 100n, IMNOTWOPR:C_Rect_P200mil, F.Cu at (137.5, 108.3)
- added C5: 100n, IMNOTWOPR:C_Rect_P200mil, F.Cu at (137.5, 112.8)
- added C6: 100n, IMNOTWOPR:C_Rect_P200mil, F.Cu at (137.5, 117.2)
- added C7: 47µF, IMNOTWOPR:CP_Radial_Tantal_P100mil, F.Cu at (197.2, 56.9)
- added SW1: MUTE, IMNOTWOPR:PanelConnector_1x03, F.Cu at (135.0, 66.7)
- D35: value ~{ABORT} -> ~{RESET}
- D36: value ~{RESET} -> ~{IRQ}
- D37: value ~{IRQ} -> ~{NMI}
- D38: value ~{NMI} -> READY
- D39: value READY -> ~{HALT_REQ}
- D40: value SYNC -> ~{HALT_ACK}
- D41: value ~{HALT_REQ} -> ~{BUS_REQ}
- D42: value ~{HALT_ACK} -> ~{BUS_ACK}
- D43: value ~{BUS_REQ} -> ~{ABORT}
- D44: value ~{BUS_ACK} -> SYNC
- moved U2 43.2 mm to (181.4, 95.0)
- moved U1 38.0 mm to (181.4, 67.1)
- moved U5 28.0 mm to (156.6, 95.0)
- moved U3 23.1 mm to (181.4, 122.9)
- moved U6 17.7 mm to (156.6, 122.9)
- moved U4 6.84 mm to (156.6, 67.1)
- moved R17 1.27 mm to (102.0, 96.3)
- moved R18 1.27 mm to (102.0, 101.3)
- moved R19 1.27 mm to (102.0, 106.4)
- moved R20 1.27 mm to (102.0, 111.4)
- moved R21 1.27 mm to (102.0, 116.5)
- moved R22 1.27 mm to (102.0, 121.5)
- moved R23 1.27 mm to (102.0, 126.6)
- moved R24 1.27 mm to (102.0, 131.6)
- moved R41 1.27 mm to (102.0, 98.8)
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Connections:
- D38 pad 1: Net-(D38-K) -> GND
- D38 pad 2: +5V -> Net-(D38-A)
- D39 pad 1: GND -> Net-(D39-K)
- D39 pad 2: Net-(D39-A) -> +5V
- D40 pad 1: GND -> Net-(D40-K)
- D40 pad 2: Net-(D40-A) -> +5V
- D44 pad 1: Net-(D44-K) -> +5V
- D44 pad 2: +5V -> Net-(D44-A)
- J1 pad a1: VCC -> +5V
- J1 pad a2: VCC -> +5V
- J1 pad a31: VCC -> +5V
- J1 pad a32: VCC -> +5V
- J1 pad b1: VCC -> +5V
- J1 pad b32: VCC -> +5V
- R62 pad 1: +5V -> GND
- R63 pad 1: GND -> +5V
- R64 pad 1: GND -> +5V
- R68 pad 1: +5V -> GND
- R86 pad 2: Net-(D38-K) -> Net-(D38-A)
- R87 pad 2: Net-(D39-A) -> Net-(D39-K)
- R88 pad 2: Net-(D40-A) -> Net-(D40-K)
- R92 pad 2: Net-(D44-K) -> Net-(D44-A)
- U5 pad 4: ~{ABORT} -> ~{RESET}
- U5 pad 5: ~{RESET} -> ~{IRQ}
- U5 pad 6: ~{IRQ} -> ~{NMI}
- U5 pad 7: ~{NMI} -> READY
- U5 pad 8: READY -> ~{HALT_REQ}
- U5 pad 9: SYNC -> ~{HALT_ACK}
- U6 pad 2: ~{HALT_REQ} -> ~{BUS_REQ}
- U6 pad 3: ~{HALT_ACK} -> ~{BUS_ACK}
- U6 pad 4: ~{BUS_REQ} -> ~{ABORT}
- U6 pad 5: ~{BUS_ACK} -> SYNC
Routing:
- net +5V: track 0.00 -> 130.4 mm
- net A_{1}: track 0.00 -> 34.3 mm
- net A_{5}: track 0.00 -> 34.3 mm
- net A_{4}: track 0.00 -> 34.3 mm
- net A_{3}: track 0.00 -> 34.3 mm
- net A_{2}: track 0.00 -> 34.3 mm
- net A_{0}: track 0.00 -> 34.3 mm
- net A_{7}: track 0.00 -> 34.3 mm
- net A_{6}: track 0.00 -> 34.3 mm
- net GND: track 0.00 -> 15.0 mm
Other:
- board text removed: "Mounting holes are optional Keepout areas are for for guide rails"

Commit message: project cleanup
Parts:
- moved C1 94.2 mm to (231.5, 88.0)
- moved C2 94.2 mm to (231.5, 92.5)
- moved C3 94.2 mm to (231.5, 96.9)
- moved C4 94.2 mm to (231.5, 101.3)
- moved C5 94.2 mm to (231.5, 105.8)
- moved C6 94.2 mm to (231.5, 110.2)
- moved SW1 37.9 mm to (168.9, 49.9), turned to 180 degrees
- moved R57 7.11 mm to (128.0, 51.7)
- moved R96 7.06 mm to (128.0, 138.3)
- moved R81 6.96 mm to (128.0, 54.5)
- moved R72 6.92 mm to (128.0, 135.5)
- moved R58 6.80 mm to (128.0, 57.3)
- moved R95 6.76 mm to (128.0, 132.7)
- moved R82 6.67 mm to (128.0, 60.1)
- moved R71 6.63 mm to (128.0, 129.9)
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Routing:
- net MUTE: track 0.00 -> 122.5 mm
- net ~{ABORT}: track 0.00 -> 59.6 mm
- net VPB: track 0.00 -> 59.6 mm
- net MLB: track 0.00 -> 59.6 mm
- net ~{BUS_REQ}: track 0.00 -> 59.6 mm
- net VDA: track 0.00 -> 59.6 mm
- net SYNC: track 0.00 -> 59.6 mm
- net ~{BUS_ACK}: track 0.00 -> 59.6 mm
- net VPA: track 0.00 -> 59.6 mm
- net ~{IRQ}: track 0.00 -> 56.5 mm
- net ~{NMI}: track 0.00 -> 56.5 mm
- net ~{HALT_REQ}: track 0.00 -> 56.5 mm
- net D_{1}: track 0.00 -> 56.5 mm
- net Φ_{2}: track 0.00 -> 56.5 mm
- net R~{W}: track 0.00 -> 56.5 mm
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