File: modules/MPU/MPU.kicad_pcb (KiCad board)
At the start: 2 copper layers, 160 x 100 mm, 2 parts, among them J1 CardConnector

Commit message: mpu wip
Parts:
- added C1: 47u, IMNOTWOPR:CP_Radial_Tantal_P100mil, F.Cu at (105.4, 87.4)
- added C2: 100n, FormantKO:C_Rect_P200mil, F.Cu at (195.7, 79.8)
- added C4: 100n, FormantKO:C_Rect_P200mil, F.Cu at (183.1, 82.9)
- added C5: 100n, FormantKO:C_Rect_P200mil, F.Cu at (183.0, 53.1)
- added C6: 100n, FormantKO:C_Rect_P200mil, F.Cu at (195.7, 50.5)
- added R1: 10k, IMNOTWOPR:R_Axial_DIN0207_P400mil, F.Cu at (100.0, 77.2)
- added R2: 10k, IMNOTWOPR:R_Axial_DIN0207_P400mil, F.Cu at (100.0, 81.1)
- added U1: 74HCT541, IMNOTWOPR:DIP-20N, F.Cu at (195.7, 65.8)
- added U3: W65C02, IMNOTWOPR:DIP-40W, F.Cu at (127.2, 92.5)
- added U4: 74HCT541, IMNOTWOPR:DIP-20N, F.Cu at (195.7, 93.7)
- added U6: 74HCT245N, IMNOTWOPR:DIP-20N, F.Cu at (183.0, 68.3)
- added U7: 74HCT541, IMNOTWOPR:DIP-20N, F.Cu at (170.3, 88.7)
- added U8: 74HCT541, IMNOTWOPR:DIP-20N, F.Cu at (183.0, 98.8)
- added Y1: 1Mhz, Oscillator:Oscillator_DIP-14, F.Cu at (151.3, 91.2)
Connections:
- net VCC renamed +5V
- J1 pad a10: unconnected-(J1A-A_{6}-Pada10) -> Net-(J1A-A_{6})
- J1 pad a11: unconnected-(J1A-A_{7}-Pada11) -> Net-(J1A-A_{7})
- J1 pad a12: unconnected-(J1A-A_{8}-Pada12) -> Net-(J1A-A_{8})
- J1 pad a13: unconnected-(J1A-A_{9}-Pada13) -> Net-(J1A-A_{9})
- J1 pad a14: unconnected-(J1A-A_{10}-Pada14) -> Net-(J1A-A_{10})
- J1 pad a15: unconnected-(J1A-A_{11}-Pada15) -> Net-(J1A-A_{11})
- J1 pad a16: unconnected-(J1A-A_{12}-Pada16) -> Net-(J1A-A_{12})
- J1 pad a17: unconnected-(J1A-A_{13}-Pada17) -> Net-(J1A-A_{13})
- J1 pad a18: unconnected-(J1A-A_{14}-Pada18) -> Net-(J1A-A_{14})
- J1 pad a19: unconnected-(J1A-A_{15}-Pada19) -> Net-(J1A-A_{15})
- J1 pad a4: unconnected-(J1A-A_{0}-Pada4) -> Net-(J1A-A_{0})
- J1 pad a5: unconnected-(J1A-A_{1}-Pada5) -> Net-(J1A-A_{1})
- J1 pad a6: unconnected-(J1A-A_{2}-Pada6) -> Net-(J1A-A_{2})
- J1 pad a7: unconnected-(J1A-A_{3}-Pada7) -> Net-(J1A-A_{3})
- J1 pad a8: unconnected-(J1A-A_{4}-Pada8) -> Net-(J1A-A_{4})
- J1 pad a9: unconnected-(J1A-A_{5}-Pada9) -> Net-(J1A-A_{5})
- J1 pad b10: unconnected-(J1B-D_{6}-Padb10) -> Net-(J1B-D_{6})
- J1 pad b11: unconnected-(J1B-D_{7}-Padb11) -> Net-(J1B-D_{7})
- J1 pad b12: unconnected-(J1B-Φ_{2}-Padb12) -> Net-(J1B-Φ_{2})
- J1 pad b13: unconnected-(J1B-R~{W}-Padb13) -> Net-(J1B-R~{W})
- J1 pad b14: unconnected-(J1B-VALID-Padb14) -> Net-(J1B-~{VALID})
- J1 pad b15: unconnected-(J1B-~{RESET}-Padb15) -> Net-(J1B-~{RESET})
- J1 pad b16: unconnected-(J1B-~{IRQ}-Padb16) -> Net-(J1B-~{IRQ})
- J1 pad b17: unconnected-(J1B-~{NMI}-Padb17) -> Net-(J1B-~{NMI})
- J1 pad b18: unconnected-(J1B-RDY-Padb18) -> /READY
- J1 pad b19: unconnected-(J1B-~{HALT-REQ}-Padb19) -> Net-(J1B-~{BUSREQ0})
- J1 pad b20: unconnected-(J1B-~{HALT-ACK}-Padb20) -> Net-(J1B-~{BUSGNT0})
- J1 pad b24: unconnected-(J1B-SYNC-Padb24) -> Net-(J1B-SYNC)
- J1 pad b25: unconnected-(J1B-VPB-Padb25) -> Net-(J1B-VPB)
- J1 pad b26: unconnected-(J1B-MLB-Padb26) -> Net-(J1B-MLB)
- J1 pad b4: unconnected-(J1B-D_{0}-Padb4) -> Net-(J1B-D_{0})
- J1 pad b5: unconnected-(J1B-D_{1}-Padb5) -> Net-(J1B-D_{1})
- J1 pad b6: unconnected-(J1B-D_{2}-Padb6) -> Net-(J1B-D_{2})
- J1 pad b7: unconnected-(J1B-D_{3}-Padb7) -> Net-(J1B-D_{3})
- J1 pad b8: unconnected-(J1B-D_{4}-Padb8) -> Net-(J1B-D_{4})
- J1 pad b9: unconnected-(J1B-D_{5}-Padb9) -> Net-(J1B-D_{5})
- J1 pad c1: GND -> unconnected-(J1C-+5VSB-Padc1)
- J1 pad c3: GND -> unconnected-(J1C-+12V2-Padc3)
- J1 pad c30: GND -> unconnected-(J1C-+12V2-Padc30)
Routing:
- net Net-(J1B-~{VALID}): track 0.00 -> 34.6 mm
- net Net-(J1B-R~{W}): track 0.00 -> 34.6 mm
- net Net-(J1B-Φ_{2}): track 0.00 -> 34.6 mm
- net Net-(J1B-~{BUSGNT0}): track 0.00 -> 30.6 mm
- net Net-(J1B-~{IRQ}): track 0.00 -> 29.5 mm
- net Net-(J1B-D_{1}): track 0.00 -> 29.5 mm
- net Net-(J1B-D_{7}): track 0.00 -> 29.5 mm
- net Net-(J1B-D_{5}): track 0.00 -> 29.5 mm
- net Net-(J1B-D_{4}): track 0.00 -> 29.5 mm
- net Net-(J1B-D_{3}): track 0.00 -> 29.5 mm
- net Net-(J1B-D_{2}): track 0.00 -> 29.5 mm
- net Net-(J1B-D_{0}): track 0.00 -> 29.5 mm
- net Net-(J1B-~{RESET}): track 0.00 -> 29.5 mm
- net Net-(J1B-~{NMI}): track 0.00 -> 29.5 mm
- net Net-(J1B-D_{6}): track 0.00 -> 29.5 mm
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Other:
- board text removed: "Mounting holes are optional Keepout areas are for for guide rails"
