File: modules/MSD/system.kicad_sch (KiCad schematic)
At the start: 2 parts, among them J1 CardConnector

Commit message: minor PW PCB tweaks
Parts:
- renumbered J1 to J2
Connections:
- net GND: no longer J2.c1 (GND), J2.c3 (GND), J2.c30 (GND)
- net SPI_MOSI: now reaches J2.c10 (SPI_MOSI)
- net SPI_MISO: now reaches J2.c11 (SPI_MISO)
- net SPI_SCK: now reaches J2.c9 (SPI_SCK)
- no-connect marks 78 -> 77
Other:
- title: MPU-65 -> MSD-65
- moved on the sheet: J2C
