File: system/BACKPLANE/BACKPLANE.kicad_sch (KiCad schematic)
At the start: 48 parts, among them J1 BusConnector, J10 BusConnector, J11 BusConnector, J12 BusConnector, J13 BusConnector, J14 BusConnector, J15 BusConnector, J16 BusConnector, J17 BusConnector, J18 BusConnector, J19 BusConnector, J2 BusConnector, J20 BusConnector, J21 BusConnector, J22 BusConnector, J23 BusConnector, J24 BusConnector, J25 BusConnector, J26 BusConnector, J29 ATX-24, J3 BusConnector, J30 ATX-04, J4 BusConnector, J5 BusConnector, J6 BusConnector, J7 BusConnector, J8 BusConnector, J9 BusConnector

Commit message: added i2c pullsups to backplane
Parts:
- added JP1: I2C PULLUPS, FormantKO:Jumper_1x02, symbol Jumper:Jumper_2_Bridged
- added R1, R2: 4k7Ω, IMNOTWOPR:R_Axial_DIN0207_P400mil, symbol IMNOTWOPR:R
Connections:
- net +5V: now also JP1.1 (A)
- net c7: now also R1.1
- net c8: now also R2.1
- new net: JP1.2 (B), R1.2, R2.2
Other:
- note added: "SCL"
- note added: "SDA"
- moved on the sheet: J10C, J11C, J12C, J13C, J14C, J15C, J16C, J17C, J18C, J19C, J1C, J20C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

Commit message: backplane updates and notes
Parts:
- removed J21, J22, J23, J24, J25, J26: BusConnector, IMNOTWOPR:SystemConnector_Female, symbol IMNOTWOPR:BusConnector
- added H21, H22, H23, H24, H25, H26, H27, H28, H29, H30, H31, H32, H33, H34, H35, H36, H37, H38, H39, H40, H41, H42, H43, H44, H45, H46, H47, H48, H49, H50, H51, H52, H53, H54, H55, H56: MountingHole, IMNOTWOPR:MountingHole_2.7mm_M2.5, symbol FormantKO:MountingHole
- H1, H10, H11, H12, H13, H14, H15, H16, H17, H18, H19, H2, H20, H3, H4, H5, H6, H7, H8, H9: footprint FormantKO:MountingHole_2.7mm_M2.5 -> IMNOTWOPR:MountingHole_2.7mm_M2.5

Commit message: backplane pcb
Parts:
- removed J30: ATX-04, IMNOTWOPR:ATX-04, symbol IMNOTWOPR:ATX-04
- added J21: ATX-08, IMNOTWOPR:ATX-08, symbol IMNOTWOPR:ATX-08
Connections:
- net +12V2: now also J21.5 (+12V2), J21.6 (+12V2), J21.7 (+12V2), J21.8 (+12V2)
- net GND: now also J21.1 (GND), J21.2 (GND), J21.3 (GND), J21.4 (GND)
Changed lines of the file:
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@@
 	(global_label "+12V2"
 		(shape output)
-		(at 513.08 359.41 0)
+		(at 513.08 367.03 0)
 		(fields_autoplaced yes)
 		(effects
@@
 		)
 		(property "Intersheetrefs" "${INTERSHEET_REFS}"
-			(at 522.3547 359.41 0)
+			(at 522.3547 367.03 0)
 			(hide yes)
 			(show_name no)
@@
 		)
 	)
+	(global_label "+12V2"
+		(shape output)
+		(at 513.08 374.65 0)
+		(fields_autoplaced yes)
+		(effects
+			(font
+				(size 1.27 1.27)
+			)
+			(justify left)
+		)
+		(property "Intersheetrefs" "${INTERSHEET_REFS}"
+			(at 522.3547 374.65 0)
+			(hide yes)
+			(show_name no)
+			(do_not_autoplace no)
+			(effects
+				(font
+					(size 1.27 1.27)
+				)
+				(justify left)
+			)
+		)
+	)
 	(global_label "b27"
 		(shape passive)
@@
 		)
 	)
+	(global_label "GND"
+		(shape output)
+		(at 513.08 359.41 0)
+		(fields_autoplaced yes)
+		(effects
+			(font
+				(size 1.27 1.27)
+			)
+			(justify left)
+		)
+		(property "Intersheetrefs" "${INTERSHEET_REFS}"
+			(at 519.9357 359.41 0)
+			(hide yes)
+			(show_name no)
+			(do_not_autoplace no)
+			(effects
+				(font
+					(size 1.27 1.27)
+				)
+				(justify left)
+			)
+		)
+	)
 	(global_label "+5VSB"
 		(shape input)
@@
 	(global_label "GND"
 		(shape output)
-		(at 513.08 354.33 0)
+		(at 513.08 356.87 0)
 		(fields_autoplaced yes)
 		(effects
@@
 		)
 		(property "Intersheetrefs" "${INTERSHEET_REFS}"
-			(at 519.9357 354.33 0)
+			(at 519.9357 356.87 0)
 			(hide yes)
 			(show_name no)
@@
 	)
 	(global_label "GND"
+		(shape output)
+		(at 513.08 361.95 0)
+		(fields_autoplaced yes)
+		(effects
+			(font
+				(size 1.27 1.27)
+			)
+			(justify left)
+		)
+		(property "Intersheetrefs" "${INTERSHEET_REFS}"
+			(at 519.9357 361.95 0)
+			(hide yes)
+			(show_name no)
+			(do_not_autoplace no)
+			(effects
+				(font
+					(size 1.27 1.27)
+				)
+				(justify left)
+			)
+		)
+	)
+	(global_label "GND"
 		(shape passive)
 		(at 703.58 116.84 180)
@@
 		)
 	)
+	(global_label "+12V2"
+		(shape output)
+		(at 513.08 372.11 0)
+		(fields_autoplaced yes)
+		(effects
+			(font
+				(size 1.27 1.27)
+			)
+			(justify left)
+		)
+		(property "Intersheetrefs" "${INTERSHEET_REFS}"
+			(at 522.3547 372.11 0)
+			(hide yes)
+			(show_name no)
+			(do_not_autoplace no)
+			(effects
+				(font
+					(size 1.27 1.27)
+				)
+				(justify left)
+			)
+		)
+	)
 	(global_label "GND"
 		(shape passive)
@@
 	(global_label "GND"
 		(shape output)
-		(at 513.08 351.79 0)
+		(at 513.08 354.33 0)
 		(fields_autoplaced yes)
 		(effects
@@
 		)
 		(property "Intersheetrefs" "${INTERSHEET_REFS}"
-			(at 519.9357 351.79 0)
+			(at 519.9357 354.33 0)
 			(hide yes)
 			(show_name no)
@@
 	(global_label "+12V2"
 		(shape output)
-		(at 513.08 361.95 0)
+		(at 513.08 369.57 0)
 		(fields_autoplaced yes)
 		(effects
@@
 		)
 		(property "Intersheetrefs" "${INTERSHEET_REFS}"
-			(at 522.3547 361.95 0)
+			(at 522.3547 369.57 0)
 			(hide yes)
 			(show_name no)
@@
 	)
 	(symbol
+		(lib_id "IMNOTWOPR:ATX-08")
+		(at 504.19 358.14 0)
+		(unit 1)
+		(body_style 1)
+		(exclude_from_sim no)
+		(in_bom yes)
+		(on_board yes)
+		(in_pos_files yes)
+		(dnp no)
+		(fields_autoplaced yes)
+		(property "Reference" "J21"
+			(at 504.19 346.71 0)
+			(show_name no)
+			(do_not_autoplace no)
+			(effects
+				(font
+					(size 1.27 1.27)
+				)
+			)
+		)
+		(property "Value" "ATX-08"
+			(at 504.19 349.25 0)
+			(show_name no)
+			(do_not_autoplace no)
+			(effects
+				(font
+					(size 1.27 1.27)
+				)
+			)
+		)
+		(property "Footprint" "IMNOTWOPR:ATX-08"
+			(at 504.19 358.14 0)
+			(hide yes)
+			(show_name no)
+			(do_not_autoplace no)
+			(effects
+				(font
+					(size 1.27 1.27)
+				)
+			)
+		)
+		(property "Datasheet" ""
+			(at 504.19 358.14 0)
+			(hide yes)
+			(show_name no)
+			(do_not_autoplace no)
+			(effects
+				(font
+					(size 1.27 1.27)
+				)
+			)
+		)
+		(property "Description" "Generic connector, double row, 02x02, top/bottom pin numbering scheme (row 1: 1...pins_per_row, row2: pins_per_row+1 ... num_pins), script generated (kicad-library-utils/schlib/autogen/connector/)"
+			(at 504.19 358.14 0)
+			(hide yes)
+			(show_name no)
+			(do_not_autoplace no)
+			(effects
+				(font
+					(size 1.27 1.27)
+				)
+			)
+		)
+		(pin "6"
+		)
+		(pin "5"
+		)
+		(pin "4"
+		)
+		(pin "1"
+		)
+		(pin "2"
+		)
+		(pin "7"
+		)
+		(pin "3"
+		)
+		(pin "8"
+		)
+		(instances
+			(project "BACKPLANE"
+				(path "/ad2d789c-a8c8-48c5-8f34-468c01c0c6c9"
+					(reference "J21")
+					(unit 1)
+				)
+			)
+		)
+	)
+	(symbol
 		(lib_id "IMNOTWOPR:BusConnector")
 		(at 124.46 241.3 0)
@@
 					(unit 1)
 				)
-			)
-		)
-	)
-	(symbol
-		(lib_id "IMNOTWOPR:ATX-04")
-		(at 504.19 355.6 0)
-		(unit 1)
-		(body_style 1)
-		(exclude_from_sim no)
-		(in_bom yes)
-		(on_board yes)
-		(in_pos_files yes)
-		(dnp no)
-		(property "Reference" "J30"
-			(at 503.936 345.44 0)
-			(show_name no)
-			(do_not_autoplace no)
-			(effects
-				(font
-					(size 1.27 1.27)
-				)
-			)
-		)
-		(property "Value" "ATX-04"
-			(at 504.19 347.98 0)
-			(show_name no)
-			(do_not_autoplace no)
-			(effects
-				(font
-					(size 1.27 1.27)
-				)
-			)
-		)
-		(property "Footprint" "IMNOTWOPR:ATX-04"
-			(at 504.19 355.6 0)
-			(hide yes)
-			(show_name no)
-			(do_not_autoplace no)
-			(effects
-				(font
-					(size 1.27 1.27)
-				)
-			)
-		)
-		(property "Datasheet" ""
-			(at 504.19 355.6 0)
-			(hide yes)
-			(show_name no)
-			(do_not_autoplace no)
-			(effects
-				(font
-					(size 1.27 1.27)
-				)
-			)
-		)
-		(property "Description" "Generic connector, double row, 02x02, top/bottom pin numbering scheme (row 1: 1...pins_per_row, row2: pins_per_row+1 ... num_pins), script generated (kicad-library-utils/schlib/autogen/connector/)"
-			(at 504.19 355.6 0)
-			(hide yes)
-			(show_name no)
-			(do_not_autoplace no)
-			(effects
-				(font
-					(size 1.27 1.27)
-				)
-			)
-		)
-		(pin "4"
-		)
-		(pin "3"
-		)
-		(pin "2"
-		)
-		(pin "1"
-		)
-		(instances
-			(project "BACKPLANE"
-				(path "/ad2d789c-a8c8-48c5-8f34-468c01c0c6c9"
-					(reference "J30")
-					(unit 1)
-				)

Commit message: version 1 of pwr module, power panel, & backplane pcb
Other:
- moved on the sheet: H1, H10, H11, H12, H13, H14, H15, H16, H17, H18, H19, H2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
