File: modules/TEMPLATE/TEMPLATE.kicad_pcb (KiCad board)
At the start: 2 copper layers, 160 x 100 mm, 2 parts, among them J1 CardConnector

Commit message: work on mpx module
Other:
- board text added: "${COMPANY} - ${COMMENT1} - ${COMMENT4} - ${TITLE} - ${COMMENT2} - REVISION ${REVISION} ${CURRENT_DATE}"
- board text removed: "${COMPANY} - ${COMMENT1} - ${TITLE} - ${COMMENT2} - REVISION ${REVISION} ${CURRENT_DATE}"
Changed lines of the file:
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@@
 		(comment 2 "TEMPLATE")
 		(comment 3 "DO NOT FOLD, SPINDLE OR MUTILATE")
+		(comment 4 "75-2000-01")
 	)
 	(layers
@@
 		(layer "Edge.Cuts")
 	)
-	(gr_text "${COMPANY} - ${COMMENT1} - ${TITLE} - ${COMMENT2} - REVISION ${REVISION} ${CURRENT_DATE}"
+	(gr_text "${COMPANY} - ${COMMENT1} - ${COMMENT4} - ${TITLE} - ${COMMENT2} - REVISION ${REVISION} ${CURRENT_DATE}"
 		(at 134.99 45.94 0)
 		(layer "F.SilkS")
@@
 		)
 	)
-	(gr_text "${COMPANY} - ${COMMENT1} - ${TITLE} - ${COMMENT2} - REVISION ${REVISION} ${CURRENT_DATE}"
+	(gr_text "${COMPANY} - ${COMMENT1} - ${COMMENT4} - ${TITLE} - ${COMMENT2} - REVISION ${REVISION} ${CURRENT_DATE}"
 		(at 134.99 45.94 0)
 		(layer "B.SilkS")
