File: modules/TEMPLATE/system.kicad_sch (KiCad schematic)
At the start: 0 parts

Commit message: added 9V power supply
Other:
- company: THE HOUSE OF GALAHAD -> ${COMPANY_NAME}
- title: TITLE -> ${MODULE_NAME}
Changed lines of the file:
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@@
 	(paper "A3")
 	(title_block
-		(title "TITLE")
+		(title "${MODULE_NAME}")
 		(rev "A")
-		(company "THE HOUSE OF GALAHAD")
-		(comment 1 "IMNOTWOPR")
-		(comment 2 "CARD TEMPLATE")
-		(comment 3 "75-1000-01")
+		(company "${COMPANY_NAME}")
+		(comment 1 "${PROJECT_NAME}")
+		(comment 2 "${MODULE_DESCRIPTION}")
+		(comment 3 "${PART_NUMBER}")
 	)
 	(sheet_instances
