File: modules/CTL/CTL.kicad_pcb (KiCad board)
At the start: 2 copper layers, 160 x 100 mm, 2 parts, among them J1 CardConnector

Commit message: cleanup; added ext board
Changed lines of the file:
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@@
 	(paper "A4")
 	(title_block
-		(title "TITLE")
+		(title "CTL")
 		(rev "A")
 		(company "THE HOUSE OF GALAHAD")
 		(comment 1 "IMNOTWOPR")
-		(comment 2 "TEMPLATE")
+		(comment 2 "PROCESSOR CONTROL")
 		(comment 3 "DO NOT FOLD, SPINDLE OR MUTILATE")
-		(comment 4 "75-2000-01")
+		(comment 4 "75-1001-01")
 	)
 	(layers
