File: panels/MPX/MPX.kicad_pcb (KiCad board)
At the start: 2 copper layers, 40.3 x 128.4 mm, 5 parts

Commit message: cleanup; added ext board
Parts:
- added REF**: DB-9 Panel, IMNOTWOPR:DB-9 Panel, F.Cu at (77.9, 129.8)
- moved H2 20.3 mm to (119.4, 42.5)
- moved H4 20.3 mm to (119.4, 164.9)
Other:
- board size 40.3 x 128.4 mm -> 60.1 x 128.4 mm
- board text added: "MPU-65X"
- board text removed: "MOD"
