File: panels/PWR/PWR.kicad_pcb (KiCad board)
At the start: 2 copper layers, 40.3 x 128.4 mm, 13 parts

Commit message: mega updates.  psg module.  ferrous & example makefiles overhaul
Other:
- board text added: "${TITLE}"
- board text removed: "PWR"
Changed lines of the file:
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@@
 		)
 	)
-	(gr_text "PWR"
+	(gr_text "${TITLE}"
 		(at 86.395894 42.715428 0)
 		(layer "F.SilkS")
