File: modules/MPX/MPX.kicad_sch (KiCad schematic)
At the start: 21 parts, among them J1 DE9_Socket, U1 W65C02, U2 28C256, U3 74NC00, U4 62256, U5 W65C51, U6 W65C22, U7 MAX232, U8 MAX3243IDBR, Y1 1Mhz, Y2 Crystal

Commit message: project cleanup
Parts:
- removed U8: MAX3243IDBR, IMNOTWOPR:SOP65P780X200-28N, symbol IMNOTWOPR:MAX3243IDBR
- added RV1: 10kΩ, Potentiometer_THT:Potentiometer_Bourns_3266Y_Vertical, symbol Device:R_Potentiometer_Trim
- added U9: LCD-016M002B, Connector_PinHeader_2.54mm:PinHeader_1x16_P2.54mm_Vertical, symbol IMNOTWOPR:LCD-016M002B
- J1: footprint Connector_Dsub:DSUB-9_Socket_Horizontal_P2.77x2.54mm_EdgePinOffset9.40mm -> Connector_IDC:IDC-Header_2x05_P2.54mm_Vertical
Connections:
- net A_{0}: no longer U1.9 (A_{0})
- net A_{15}: now also U1.25 (A_{15})
- net A_{1}: no longer U1.10 (A_{1})
- net A_{2}: no longer U1.11 (A_{2})
- net A_{3}: no longer U1.12 (A_{3})
- net A_{4}: no longer U1.13 (A_{4})
- net A_{5}: no longer U1.14 (A_{5})
- net A_{6}: no longer U1.15 (A_{6})
- net A_{7}: no longer U1.16 (A_{7})
- net GND: now also RV1.1, U9.1 (V_{SS}), U9.16 (K)
- net PB_{0}: now reaches U6.10 (PB_{0})
- net PB_{0}: now also U6.12 (PB_{2}), U6.13 (PB_{3}), U6.15 (PB_{5}), U6.17 (PB_{7}), U9.11 (DB_{4})
- net D_{0} renamed D0
- net D_{1} renamed D1
- net D_{2} renamed D2
- net D_{3} renamed D3
- net D_{4} renamed D4
- net D_{5} renamed D5
- net D_{6} renamed D6
- net D_{7} renamed D7
- net VCC renamed +5V
- net +5V: now also U9.15 (A/V_{EE}), U9.2 (V_{DD})
- new net: RV1.2, U9.3 (V_{O})
- new net A0: U1.9 (A_{0})
- new net A1: U1.10 (A_{1})
- new net PB_{1}: U9.12 (DB_{5})
- new net PB_{2}: U9.13 (DB_{6})
- new net PB_{3}: U9.14 (DB_{7})
- new net PB_{4}: U9.4 (RS)
- new net PB_{5}: U9.5 (R/~{W})
- new net PB_{6}: U9.6 (E)
- no-connect marks 12 -> 17
Other:
- moved on the sheet: D1, D2, R1, R2

Commit message: work on mpx module
Parts:
- removed C1, C2, C3, C4: 1µF, IMNOTWOPR:C_Rect_P200mil, symbol IMNOTWOPR:C
- removed C5: 20pF, IMNOTWOPR:C_Rect_P200mil, symbol IMNOTWOPR:C
- removed D1: T_{X}D, LED_THT:LED_D5.0mm_Horizontal_O1.27mm_Z3.0mm, symbol Device:LED_Dual_Bidirectional
- removed D2: R_{X}D, LED_THT:LED_D5.0mm_Horizontal_O1.27mm_Z3.0mm, symbol Device:LED_Dual_Bidirectional
- removed J1: DE9_Socket, Connector_IDC:IDC-Header_2x05_P2.54mm_Vertical, symbol Connector:DE9_Socket
- removed R1, R2: 1kΩ, IMNOTWOPR:R_Axial_DIN0207_P400mil, symbol IMNOTWOPR:R
- removed R3: 1MΩ, IMNOTWOPR:R_Axial_DIN0207_P400mil, symbol IMNOTWOPR:R
- removed RV1: 10kΩ, Potentiometer_THT:Potentiometer_Bourns_3266Y_Vertical, symbol Device:R_Potentiometer_Trim
- removed U2: 28C256, IMNOTWOPR:ZIF-28W, symbol Memory_EEPROM:28C256
- removed U3: 74NC00, IMNOTWOPR:DIP-14N, symbol IMNOTWOPR:7400
- removed U4: 62256, Package_DIP:DIP-28_W15.24mm, symbol Memory_RAM:CY62256-70PC
- removed U6: W65C22, IMNOTWOPR:DIP-40W, symbol IMNOTWOPR:W65C22
- removed U7: MAX232, IMNOTWOPR:DIP-16N, symbol IMNOTWOPR:MAX232
- removed U9: LCD-016M002B, Connector_PinHeader_2.54mm:PinHeader_1x16_P2.54mm_Vertical, symbol IMNOTWOPR:LCD-016M002B
- removed Y2: Crystal, Crystal:Crystal_HC49-U_Horizontal, symbol Device:Crystal
- added RN1: 10kΩ, Resistor_THT:R_Array_SIP9, symbol Device:R_Network08_Split
- added SW1: PAGE SELECT, Button_Switch_THT:SW_DIP_SPSTx08_Slide_9.78x22.5mm_W7.62mm_P2.54mm, symbol Switch:SW_DIP_x08
- added U10: 74AHCT244, IMNOTWOPR:DIP-20N, symbol 74xx:74AHCT244
- added U12: 74HC138, IMNOTWOPR:DIP-16N, symbol 74xx:74HC138
- added U14: 74HC688, IMNOTWOPR:DIP-20N, symbol 74xx:74HC688
- added U2: CY62256-70PC, IMNOTWOPR:DIP-28W, symbol Memory_RAM:CY62256-70PC
- added U3: 28C256, IMNOTWOPR:ZIF-28W, symbol Memory_EEPROM:28C256
- added U4: W65C22, IMNOTWOPR:DIP-40W, symbol IMNOTWOPR:W65C22
- added U6: MAX232, IMNOTWOPR:DIP-16N, symbol IMNOTWOPR:MAX232
- added U7, U8: 74AHCT541, IMNOTWOPR:DIP-20N, symbol 74xx:74AHCT541
- added U9: 74AHCT245, IMNOTWOPR:DIP-20N, symbol 74xx:74HC245
- U1: Name SOPHRONIA -> (none)
- U5: Name EULALIA -> (none)
Connections:
- net A_{0} is gone; now on net A0: U5.13 (RS_{0})
- net A_{1} is gone; now on net A1: U5.14 (RS_{1})
- net +5V: now also U5.2 (CS_{0}), SW1.1, SW1.2, SW1.3, SW1.4, SW1.5, SW1.6, SW1.7, SW1.8, U10.20 (VCC), U12.16 (VCC), U12.6 (G1), U14.20 (VCC), U2.28 (VCC), U3.28 (VCC), U4.20 (V_{DD}), U4.24 (CS_{1}), U6.16 (VCC), U7.20 (VCC), U8.20 (VCC), U9.20 (VCC)
- net A0: now also U2.10 (A0), U3.10 (A0), U4.38 (RS_{0}), U7.2 (A0)
- net A1: now also U2.9 (A1), U3.9 (A1), U4.37 (RS_{1}), U7.3 (A1)
- net A2: now also U1.11 (A_{2}), U2.8 (A2), U3.8 (A2), U4.36 (RS_{2}), U7.4 (A2)
- net A3: now also U1.12 (A_{3}), U2.7 (A3), U3.7 (A3), U4.35 (RS_{3}), U7.5 (A3)
- net A4: now also U1.13 (A_{4}), U12.1 (A0), U2.6 (A4), U3.6 (A4), U7.6 (A4)
- net A5: now also U1.14 (A_{5}), U12.2 (A1), U2.5 (A5), U3.5 (A5), U7.7 (A5)
- net A6: now also U1.15 (A_{6}), U12.3 (A2), U2.4 (A6), U3.4 (A6), U7.8 (A6)
- net A7: now also U1.16 (A_{7}), U12.5 (~{G2B}), U2.3 (A7), U3.3 (A7), U7.9 (A7)
- net D0: now also U2.11 (Q0), U3.11 (D0), U9.2 (A0); no longer U5.18 (D_{0})
- net D1: now also U2.12 (Q1), U3.12 (D1), U9.3 (A1); no longer U5.19 (D_{1})
- net D2: now also U2.13 (Q2), U3.13 (D2), U9.4 (A2); no longer U5.20 (D_{2})
- net D3: now also U2.15 (Q3), U3.15 (D3), U9.5 (A3); no longer U5.21 (D_{3})
- net D4: now also U2.16 (Q4), U3.16 (D4), U9.6 (A4); no longer U5.22 (D_{4})
- net D5: now also U2.17 (Q5), U3.17 (D5), U9.7 (A5); no longer U5.23 (D_{5})
- net D6: now also U2.18 (Q6), U3.18 (D6), U9.8 (A6); no longer U5.24 (D_{6})
- net D7: now also U2.19 (Q7), U3.19 (D7), U9.9 (A7); no longer U5.25 (D_{7})
- net GND: now also RN1.1 (R1), RN1.1 (R1), RN1.1 (R1), RN1.1 (R1), RN1.1 (R1), RN1.1 (R1), RN1.1 (R1), RN1.1 (R1), U10.10 (GND), U12.8 (GND), U14.1 (G), U14.10 (GND), U2.14 (GND), U3.14 (GND), U4.1 (V_{SS}), U6.15 (GND), U7.10 (GND), U8.10 (GND), U9.10 (GND)
- net ~{ACIA ENABLED}: now reaches U5.3 (~{CS_{1}})
- net ~{ACIA ENABLED}: now also U12.14 (~{Y1})
- net A_{10} renamed A10
- net A10: now also U14.14 (R5), U2.21 (A10), U3.21 (A10), U8.4 (A2)
- net A_{11} renamed A11
- net A11: now also U14.12 (R4), U2.23 (A11), U3.23 (A11), U8.5 (A3)
- net A_{12} renamed A12
- net A12: now also U14.9 (R3), U2.2 (A12), U3.2 (A12), U8.6 (A4); no longer U5.2 (CS_{0})
- net A_{13} renamed A13
- net A13: now also U14.7 (R2), U2.26 (A13), U3.26 (A13), U8.7 (A5)
- net A_{14} renamed A14
- net A14: now also U14.5 (R1), U2.1 (A14), U3.1 (A14), U8.8 (A6)
- net A_{15} renamed A15
- net A15: now also U14.3 (R0), U8.9 (A7)
- net A_{8} renamed A8
- net A8: now also U14.18 (R7), U2.25 (A8), U3.25 (A8), U8.2 (A0)
- net A_{9} renamed A9
- net A9: now also U14.16 (R6), U2.24 (A9), U3.24 (A9), U8.3 (A1)
- net ~{RESET}: no longer names the net of U1.40 (~{RES})
- net ~{RESET}: no longer U5.4 (~{RES})
- new net: RN1.8 (R7.2), SW1.10, U14.15 (P6)
- new net: RN1.5 (R4.2), SW1.13, U14.8 (P3)
- new net: RN1.7 (R6.2), SW1.11, U14.13 (P5)
- new net: RN1.6 (R5.2), SW1.12, U14.11 (P4)
- new net: RN1.9 (R8.2), SW1.9, U14.17 (P7)
- new net: U12.4 (~{G2A}), U14.19 (P=R)
- new net: RN1.2 (R1.2), SW1.16, U14.2 (P0)
- new net: RN1.3 (R2.2), SW1.15, U14.4 (P1)
- new net: RN1.4 (R3.2), SW1.14, U14.6 (P2)
- new net BA0: U7.18 (Y0)
- new net BA1: U7.17 (Y1)
- new net BA10: U8.16 (Y2)
- new net BA11: U8.15 (Y3)
- new net BA12: U8.14 (Y4)
- new net BA13: U8.13 (Y5)
- new net BA14: U8.12 (Y6)
- new net BA15: U8.11 (Y7)
- new net BA2: U7.16 (Y2)
- new net BA3: U7.15 (Y3)
- new net BA4: U7.14 (Y4)
- new net BA5: U7.13 (Y5)
- new net BA6: U7.12 (Y6)
- new net BA7: U7.11 (Y7)
- new net BA8: U8.18 (Y0)
- new net BA9: U8.17 (Y1)
- new net BD0: U9.18 (B0)
- new net BD1: U9.17 (B1)
- new net BD2: U9.16 (B2)
- new net BD3: U9.15 (B3)
- new net BD4: U9.14 (B4)
- new net BD5: U9.13 (B5)
- new net BD6: U9.12 (B6)
- new net BD7: U9.11 (B7)
- new net R_{X}1: U6.13 (R1IN)
- new net T_{X}1: U6.14 (T1OUT)
- new net ~{VIA ENABLED}: U12.15 (~{Y0}), U4.23 (~{CS_{2}})
- no-connect marks 17 -> 7
Other:
- note added: "ADDRESS BUS BUFFERING A0..A7"
- note added: "ADDRESS BUS BUFFERING A8..A15"
- note added: "ADDRESS DECODING"
- note added: "CONTROL SIGNAL BUFFERING"
- note added: "DATA BUS TRANSCEIVER D0..D7"
- note added: "RS-232 LEVEL CONDITIONING"
- title: MPU-65X -> MPX
- moved on the sheet: U1, Y1

Commit message: cleanup and mpx work
Parts:
- removed U10: 74AHCT244, IMNOTWOPR:DIP-20N, symbol 74xx:74AHCT244
- removed Y1: 1Mhz, Oscillator:Oscillator_DIP-14, symbol Oscillator:ACO-xxxMHz
- added C2, C3, C4, C5: 1µF, IMNOTWOPR:C_Rect_P200mil, symbol IMNOTWOPR:C
- added C6: 20pF, IMNOTWOPR:C_Rect_P200mil, symbol IMNOTWOPR:C
- added J1: SERIALA, IMNOTWOPR:DE-9_IDC_Header_Straight-Through, symbol Connector:DE9_Socket
- added J3: Conn_02x10_Odd_Even, Connector_PinHeader_2.54mm:PinHeader_2x10_P2.54mm_Vertical, symbol Connector_Generic:Conn_02x10_Odd_Even
- added R1: 1MΩ, IMNOTWOPR:R_Axial_DIN0207_P400mil, symbol IMNOTWOPR:R
- added R2: 10kΩ, IMNOTWOPR:R_Axial_DIN0207_P400mil, symbol IMNOTWOPR:R
- added U10, U16: 74AHCT541, IMNOTWOPR:DIP-20N, symbol 74xx:74AHCT541
- added U15: 74HC20, IMNOTWOPR:DIP-14N, symbol 74xx:74LS20
- added Y2: 1.8432Mhz, Crystal:Crystal_HC49-U_Vertical, symbol Device:Crystal
Connections:
- net +5V: now also R2.1, U10.20 (VCC), U15.5, U16.20 (VCC)
- net D0: now also U4.33 (D_{0}), U5.18 (D_{0})
- net D1: now also U4.32 (D_{1}), U5.19 (D_{1})
- net D2: now also U4.31 (D_{2}), U5.20 (D_{2})
- net D3: now also U4.30 (D_{3}), U5.21 (D_{3})
- net D4: now also U4.29 (D_{4}), U5.22 (D_{4})
- net D5: now also U4.28 (D_{5}), U5.23 (D_{5})
- net D6: now also U4.27 (D_{6}), U5.24 (D_{6})
- net D7: now also U4.26 (D_{7}), U5.25 (D_{7})
- net GND: now also C4.2, C5.2, C6.2, J1.5, U10.10 (GND), U10.8 (A6), U10.9 (A7), U16.10 (GND)
- net R_{X}1: now also J1.3
- net T_{X}1: now also J1.2
- net VPB: now reaches U1.1 (VPB)
- net VPB: now also U10.6 (A4)
- net READY: now reaches U1.2 (READY)
- net PHI1O: now reaches U1.3 (ϕ_{1}OUT)
- net R~{W}: now reaches U1.34 (R~{W})
- net R~{W}: now also U4.22 (~{RW}), U5.28 (~{RW}), U10.3 (A1)
- net BE: now reaches U1.36 (BE)
- net PHI2: now reaches U1.37 (ϕ_{2}IN)
- net PHI2: now also U4.25 (Φ_{2}), U5.27 (Φ_{2}), U10.2 (A0)
- net ~{SO}: now reaches U1.38 (~{SO})
- net PHI20: now reaches U1.39 (ϕ_{2}OUT)
- net at U1.4 (~{IRQ}): now also R2.2, U15.6
- net ~{RESET}: now reaches U1.40 (~{RES})
- net MLB: now reaches U1.5 (MLB)
- net MLB: now also U10.7 (A5)
- net ~{NMI}: now reaches U1.6 (~{NMI})
- net SYNC: now reaches U1.7 (SYNC)
- net SYNC: now also U10.5 (A3)
- net at U4.10 (PB_{0}): now also J3.2 (Pin_2)
- net at U4.11 (PB_{1}): now also J3.4 (Pin_4)
- net at U4.12 (PB_{2}): now also J3.6 (Pin_6)
- net at U4.13 (PB_{3}): now also J3.8 (Pin_8)
- net at U4.14 (PB_{4}): now also J3.10 (Pin_10)
- net at U4.15 (PB_{5}): now also J3.12 (Pin_12)
- net at U4.16 (PB_{6}): now also J3.14 (Pin_14)
- net at U4.17 (PB_{7}): now also J3.16 (Pin_16)
- net at U4.18 (CB_{1}): now also J3.18 (Pin_18)
- net at U4.19 (CB_{2}): now also J3.20 (Pin_20)
- net at U4.2 (PA_{0}): now also J3.1 (Pin_1)
- net at U4.21 (~{IRQ}): now also U15.2
- net at U4.3 (PA_{1}): now also J3.3 (Pin_3)
- net at U4.39 (CA_{2}): now also J3.19 (Pin_19)
- net at U4.4 (PA_{2}): now also J3.5 (Pin_5)
- net at U4.40 (CA_{1}): now also J3.17 (Pin_17)
- net at U4.5 (PA_{3}): now also J3.7 (Pin_7)
- net at U4.6 (PA_{4}): now also J3.9 (Pin_9)
- net at U4.7 (PA_{5}): now also J3.11 (Pin_11)
- net at U4.8 (PA_{6}): now also J3.13 (Pin_13)
- net at U4.9 (PA_{7}): now also J3.15 (Pin_15)
- net at U6.1 (C1+): now also C2.1
- net at U6.11 (T1IN): now also U5.10 (TX_{D})
- net at U6.12 (R1OUT): now also U5.12 (R_{X}D)
- net at U6.2 (VS+): now also C4.1
- net at U6.3 (C1-): now also C2.2
- net at U6.4 (C2+): now also C3.1
- net at U6.5 (C2-): now also C3.2
- net at U6.6 (VS-): now also C5.1
- net at U5.26 (~{IRQ}): now also U15.1
- net at U5.6 (XTLI): now also C6.1, R1.2, Y2.1
- net at U5.7 (XTLO): now also R1.1, Y2.2
- new net BMLB: U10.13 (Y5)
- new net BPHI2: U10.18 (Y0)
- new net BR~{W}: U10.17 (Y1)
- new net BSYNC: U10.15 (Y3)
- new net BVALID: U10.16 (Y2)
- new net BVPB: U10.14 (Y4)
- new net VALID: U10.4 (A2)
- new net ~{IRQ}: U15.4
- no-connect marks 7 -> 24
Other:
- note added: "CONTROL SIGNAL IN BUFFERING"
- note added: "CONTROL SIGNAL OUT BUFFERING"
- note added: "RESERVED FOR FUTURE EXPANSION"
- note removed: "CONTROL SIGNAL BUFFERING"
- moved on the sheet: RN1A, RN1B, RN1C, RN1D, RN1E, RN1F, RN1G, RN1H, SW1, U1, U12, U14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

Commit message: sync
Parts:
- removed C2, C3, C4, C5: 1µF, IMNOTWOPR:C_Rect_P200mil, symbol IMNOTWOPR:C
- removed U6: MAX232, IMNOTWOPR:DIP-16N, symbol IMNOTWOPR:MAX232
- added U11: MC1488, IMNOTWOPR:DIP-14N, symbol IMNOTWOPR:MC1488
- added U13: MC1489, IMNOTWOPR:DIP-14N, symbol IMNOTWOPR:MC1489
Connections:
- net R_{X}1 is gone; now on net TXD: J1.3
- net T_{X}1 is gone; now on net RXD: J1.2
- net +5V: now also U11.10 (3B), U11.5 (2B), U13.14 (V_{CC})
- net GND: now also U11.12 (4A), U11.13 (4B), U11.7 (GND), U13.7 (GND)
- net DCD: now reaches J1.1
- net DCD: now also U5.16 (~{DCD}), U13.1 (1A), U13.3 (1Y)
- net DTR: now reaches J1.4
- net DTR: now also U5.11 (~{DTR}), U11.8 (3Y), U11.9 (3A)
- net DSR: now reaches J1.6
- net DSR: now also U5.17 (~{DSR}), U13.4 (2A), U13.6 (2Y)
- net RTS: now reaches J1.7
- net RTS: now also U5.8 (~{RTS}), U11.2 (1A), U11.3 (1Y)
- net CTS: now reaches J1.8
- net CTS: now also U5.9 (~{CTS}), U13.11 (4Y), U13.13 (4A)
- net RI: now reaches J1.9
- net TXD: now reaches U5.10 (TX_{D})
- net TXD: now also U11.4 (2A), U11.6 (2Y)
- net RXD: now reaches U5.12 (R_{X}D)
- net RXD: now also U13.10 (3A), U13.8 (3Y)
- new net +12V: U11.14 (V_{CC}+)
- new net -12V: U11.1 (V_{CC}-)
- no-connect marks 24 -> 15
Other:
- note removed: "RS-232 LEVEL CONDITIONING"
- moved on the sheet: J1
