File: modules/PSG/PSG.kicad_pcb (KiCad board)
At the start: 2 copper layers, 160 x 100 mm, 45 parts, among them J1 CardConnector, J2 MonoJack, J3 PG SEL, P1 10kΩ, SW1 PAGE SELECT, U1 AY-3-8910, U12 74HC138, U14 74HC688, U2 LM386N-4, U3 TL072, U7 74AHCT541, U8 74AHCT541, U9 74AHCT245, Y1 2Mhz

Commit message: sync
Parts:
- removed REF**: PageSelectLabel, IMNOTWOPR:PageSelectLabel
- added C14: 100nF, IMNOTWOPR:C_Rect_P200mil, F.Cu at (174.1, 74.7)
- added C15: 100nF, IMNOTWOPR:C_Rect_P200mil, F.Cu at (183.0, 82.3)
- added C16: 100nF, IMNOTWOPR:C_Rect_P200mil, F.Cu at (195.7, 82.3)
- added C17: 100nF, IMNOTWOPR:C_Rect_P200mil, F.Cu at (167.2, 49.3)
- added C18: 100nF, IMNOTWOPR:C_Rect_P200mil, F.Cu at (183.0, 54.4)
- added C19: 10µF, IMNOTWOPR:CP_Radial_Tantal_P100mil, F.Cu at (81.4, 125.5)
- added C20: 100nF, IMNOTWOPR:C_Rect_P200mil, F.Cu at (195.7, 54.4)
- added J4: IO PORTS, Connector_PinHeader_2.54mm:PinHeader_2x10_P2.54mm_Vertical, F.Cu at (125.9, 84.8)
- added SW2: SPEAKER ON, IMNOTWOPR:PanelConnector_1x03, F.Cu at (71.9, 128.0)
- added U4: 74HC00, IMNOTWOPR:DIP-14N, F.Cu at (167.2, 59.4)
- J3: value PG SEL -> BASE ADDR
- JP1: value AMP VSEL -> VSEL
- R11: value 1kΩ -> 470Ω
- moved C3 85.3 mm to (197.6, 133.1), turned to 90 degrees
- moved C13 69.6 mm to (75.7, 71.5), turned to -90 degrees
- moved C4 62.9 mm to (91.0, 69.0), turned to -90 degrees
- moved C10 56.5 mm to (111.3, 113.4), turned to 180 degrees
- moved C2 54.0 mm to (151.9, 95.0), turned to -90 degrees
- moved C1 53.6 mm to (89.0, 109.0), turned to 180 degrees
- moved C12 52.2 mm to (85.9, 81.0), turned to 180 degrees
- moved R12 49.0 mm to (71.3, 84.2), turned to 90 degrees
- moved JP1 48.2 mm to (89.0, 102.6), turned to 90 degrees
- moved J3 48.1 mm to (156.4, 74.7)
- moved R10 47.8 mm to (88.4, 62.0), turned to 180 degrees
- moved U12 44.8 mm to (167.2, 81.0)
- moved R11 43.1 mm to (75.7, 84.2), turned to 90 degrees
- moved R6 43.0 mm to (88.4, 51.8)
- moved J2 40.3 mm to (64.9, 81.0)
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Connections:
- net ~{BRESET} renamed ~{RESET}
- net Φ_{2} renamed /PSG/PHI2
- C12 pad 2: Net-(C12-Pad2) -> Net-(SW2-A)
- J1 pad a1: unconnected-(J1A-+5V-Pada1) -> +5V
- J1 pad a10: A6 -> Net-(J1A-A_{6})
- J1 pad a11: A7 -> Net-(J1A-A_{7})
- J1 pad a12: A8 -> Net-(J1A-A_{8})
- J1 pad a13: A9 -> Net-(J1A-A_{9})
- J1 pad a14: A10 -> Net-(J1A-A_{10})
- J1 pad a15: A11 -> Net-(J1A-A_{11})
- J1 pad a16: A12 -> Net-(J1A-A_{12})
- J1 pad a17: A13 -> Net-(J1A-A_{13})
- J1 pad a18: A14 -> Net-(J1A-A_{14})
- J1 pad a19: A15 -> Net-(J1A-A_{15})
- J1 pad a2: unconnected-(J1A-+5V-Pada2) -> +5V
- J1 pad a30: unconnected-(J1A-+12V-Pada30) -> +12V
- J1 pad a31: unconnected-(J1A-+5V-Pada31) -> +5V
- J1 pad a32: unconnected-(J1A-+5V-Pada32) -> +5V
- J1 pad a4: A0 -> Net-(J1A-A_{0})
- J1 pad a5: A1 -> Net-(J1A-A_{1})
- J1 pad a6: A2 -> Net-(J1A-A_{2})
- J1 pad a7: A3 -> Net-(J1A-A_{3})
- J1 pad a8: A4 -> Net-(J1A-A_{4})
- J1 pad a9: A5 -> Net-(J1A-A_{5})
- J1 pad b10: D6 -> Net-(J1B-D_{6})
- J1 pad b11: D7 -> Net-(J1B-D_{7})
- J1 pad b13: R~{W} -> /PSG/RW
- J1 pad b30: unconnected-(J1B--12V-Padb30) -> -12V
- J1 pad b31: unconnected-(J1B-GND-Padb31) -> GND
- J1 pad b32: unconnected-(J1B-+5V-Padb32) -> +5V
- J1 pad b4: D0 -> Net-(J1B-D_{0})
- J1 pad b5: D1 -> Net-(J1B-D_{1})
- J1 pad b6: D2 -> Net-(J1B-D_{2})
- J1 pad b7: D3 -> Net-(J1B-D_{3})
- J1 pad b8: D4 -> Net-(J1B-D_{4})
- J1 pad b9: D5 -> Net-(J1B-D_{5})
- J1 pad c18: unconnected-(J1C-GND-Padc18) -> GND
- J1 pad c2: unconnected-(J1C-GND-Padc2) -> GND
- J1 pad c24: unconnected-(J1C-GND-Padc24) -> GND
- J1 pad c31: unconnected-(J1C-GND-Padc31) -> GND
- J1 pad c32: unconnected-(J1C-GND-Padc32) -> GND
- J1 pad c6: unconnected-(J1C-GND-Padc6) -> GND
- J3 pad 1: Net-(J3-Pin_1) -> /PSG/PG_SEL
- J3 pad 11: Net-(J3-Pin_11) -> /PSG/PG_SEL
- J3 pad 12: Net-(J3-Pin_10) -> Net-(J3-Pin_12)
- J3 pad 13: Net-(J3-Pin_13) -> /PSG/PG_SEL
- J3 pad 14: Net-(J3-Pin_10) -> Net-(J3-Pin_14)
- J3 pad 15: Net-(J3-Pin_15) -> /PSG/PG_SEL
- J3 pad 16: Net-(J3-Pin_10) -> Net-(J3-Pin_16)
- J3 pad 2: Net-(J3-Pin_10) -> Net-(J3-Pin_2)
- J3 pad 3: Net-(J3-Pin_3) -> /PSG/PG_SEL
- J3 pad 4: Net-(J3-Pin_10) -> Net-(J3-Pin_4)
- J3 pad 5: Net-(J3-Pin_5) -> /PSG/PG_SEL
- J3 pad 6: Net-(J3-Pin_10) -> Net-(J3-Pin_6)
- J3 pad 7: Net-(J3-Pin_7) -> /PSG/PG_SEL
- J3 pad 8: Net-(J3-Pin_10) -> Net-(J3-Pin_8)
- J3 pad 9: Net-(J3-Pin_9) -> /PSG/PG_SEL
- P1 pad 3: Net-(C12-Pad2) -> Net-(SW2-B)
- R11 pad 2: Net-(C12-Pad2) -> Net-(SW2-A)
- U1 pad 10: unconnected-(U1-IOB_{3}-Pad10) -> Net-(J4-Pin_8)
- U1 pad 11: unconnected-(U1-IOB_{2}-Pad11) -> Net-(J4-Pin_6)
- U1 pad 12: unconnected-(U1-IOB_{1}-Pad12) -> Net-(J4-Pin_4)
- U1 pad 13: unconnected-(U1-IOB_{0}-Pad13) -> Net-(J4-Pin_2)
- U1 pad 14: unconnected-(U1-IOA_{7}-Pad14) -> Net-(J4-Pin_15)
- U1 pad 15: unconnected-(U1-IOA_{6}-Pad15) -> Net-(J4-Pin_13)
- U1 pad 16: unconnected-(U1-IOA_{5}-Pad16) -> Net-(J4-Pin_11)
- U1 pad 17: unconnected-(U1-IOA_{4}-Pad17) -> Net-(J4-Pin_9)
- U1 pad 18: unconnected-(U1-IOA_{3}-Pad18) -> Net-(J4-Pin_7)
- U1 pad 19: unconnected-(U1-IOA_{2}-Pad19) -> Net-(J4-Pin_5)
- U1 pad 20: unconnected-(U1-IOA_{1}-Pad20) -> Net-(J4-Pin_3)
- U1 pad 21: unconnected-(U1-IOA_{0}-Pad21) -> Net-(J4-Pin_1)
- U1 pad 24: unconnected-(U1-~{A_{9}}-Pad24) -> GND
- U1 pad 25: unconnected-(U1-A_{8}-Pad25) -> +5V
- U1 pad 28: /PSG/BC2 -> /PSG/SEL
- U1 pad 29: /PSG/A1 -> /PSG/BC1
- U1 pad 30: D7 -> /PSG/D7
- U1 pad 31: D6 -> /PSG/D6
- U1 pad 32: D5 -> /PSG/D5
- U1 pad 33: D4 -> /PSG/D4
- U1 pad 34: D3 -> /PSG/D3
- U1 pad 35: D2 -> /PSG/D2
- U1 pad 36: D1 -> /PSG/D1
- U1 pad 37: D0 -> /PSG/D0
- U1 pad 6: unconnected-(U1-IOB_{7}-Pad6) -> Net-(J4-Pin_16)
- U1 pad 7: unconnected-(U1-IOB_{6}-Pad7) -> Net-(J4-Pin_14)
- U1 pad 8: unconnected-(U1-IOB_{5}-Pad8) -> Net-(J4-Pin_12)
- U1 pad 9: unconnected-(U1-IOB_{4}-Pad9) -> Net-(J4-Pin_10)
- U12 pad 10: Net-(J3-Pin_11) -> Net-(J3-Pin_12)
- U12 pad 11: Net-(J3-Pin_9) -> Net-(J3-Pin_10)
- U12 pad 12: Net-(J3-Pin_7) -> Net-(J3-Pin_8)
- U12 pad 13: Net-(J3-Pin_5) -> Net-(J3-Pin_6)
- U12 pad 14: Net-(J3-Pin_3) -> Net-(J3-Pin_4)
- U12 pad 15: Net-(J3-Pin_1) -> Net-(J3-Pin_2)
- U12 pad 7: Net-(J3-Pin_15) -> Net-(J3-Pin_16)
- U12 pad 9: Net-(J3-Pin_13) -> Net-(J3-Pin_14)
- U2 pad 7: unconnected-(U2-BYPASS-Pad7) -> Net-(U2-BYPASS)
- U7 pad 1: unconnected-(U7-G1-Pad1) -> GND
- U7 pad 11: unconnected-(U7-Y7-Pad11) -> /PSG/A7
- U7 pad 12: unconnected-(U7-Y6-Pad12) -> /PSG/A6
- U7 pad 13: unconnected-(U7-Y5-Pad13) -> /PSG/A5
- U7 pad 14: unconnected-(U7-Y4-Pad14) -> /PSG/A4
- U7 pad 17: unconnected-(U7-Y1-Pad17) -> /PSG/A1
- U7 pad 19: unconnected-(U7-G2-Pad19) -> GND
- U7 pad 2: unconnected-(U7-A0-Pad2) -> Net-(J1A-A_{0})
- U7 pad 3: unconnected-(U7-A1-Pad3) -> Net-(J1A-A_{1})
- U7 pad 4: unconnected-(U7-A2-Pad4) -> Net-(J1A-A_{2})
- U7 pad 5: unconnected-(U7-A3-Pad5) -> Net-(J1A-A_{3})
- U7 pad 6: unconnected-(U7-A4-Pad6) -> Net-(J1A-A_{4})
- U7 pad 7: unconnected-(U7-A5-Pad7) -> Net-(J1A-A_{5})
- U7 pad 8: unconnected-(U7-A6-Pad8) -> Net-(J1A-A_{6})
- U7 pad 9: unconnected-(U7-A7-Pad9) -> Net-(J1A-A_{7})
- U8 pad 1: unconnected-(U8-G1-Pad1) -> GND
- U8 pad 11: unconnected-(U8-Y7-Pad11) -> /PSG/A15
- U8 pad 12: unconnected-(U8-Y6-Pad12) -> /PSG/A14
- U8 pad 13: unconnected-(U8-Y5-Pad13) -> /PSG/A13
- U8 pad 14: unconnected-(U8-Y4-Pad14) -> /PSG/A12
- U8 pad 15: unconnected-(U8-Y3-Pad15) -> /PSG/A11
- U8 pad 16: unconnected-(U8-Y2-Pad16) -> /PSG/A10
- U8 pad 17: unconnected-(U8-Y1-Pad17) -> /PSG/A9
- U8 pad 18: unconnected-(U8-Y0-Pad18) -> /PSG/A8
- U8 pad 19: unconnected-(U8-G2-Pad19) -> GND
- U8 pad 2: unconnected-(U8-A0-Pad2) -> Net-(J1A-A_{8})
- U8 pad 3: unconnected-(U8-A1-Pad3) -> Net-(J1A-A_{9})
- U8 pad 4: unconnected-(U8-A2-Pad4) -> Net-(J1A-A_{10})
- U8 pad 5: unconnected-(U8-A3-Pad5) -> Net-(J1A-A_{11})
- U8 pad 6: unconnected-(U8-A4-Pad6) -> Net-(J1A-A_{12})
- U8 pad 7: unconnected-(U8-A5-Pad7) -> Net-(J1A-A_{13})
- U8 pad 8: unconnected-(U8-A6-Pad8) -> Net-(J1A-A_{14})
- U8 pad 9: unconnected-(U8-A7-Pad9) -> Net-(J1A-A_{15})
- U9 pad 1: R~{W} -> /PSG/BDIR
- U9 pad 11: unconnected-(U9-B7-Pad11) -> /PSG/D7
- U9 pad 12: unconnected-(U9-B6-Pad12) -> /PSG/D6
- U9 pad 13: unconnected-(U9-B5-Pad13) -> /PSG/D5
- U9 pad 14: unconnected-(U9-B4-Pad14) -> /PSG/D4
- U9 pad 15: unconnected-(U9-B3-Pad15) -> /PSG/D3
- U9 pad 16: unconnected-(U9-B2-Pad16) -> /PSG/D2
- U9 pad 17: unconnected-(U9-B1-Pad17) -> /PSG/D1
- U9 pad 18: unconnected-(U9-B0-Pad18) -> /PSG/D0
- U9 pad 19: ~{PG_SEL} -> /PSG/PG_SEL
- U9 pad 2: unconnected-(U9-A0-Pad2) -> Net-(J1B-D_{0})
- U9 pad 3: unconnected-(U9-A1-Pad3) -> Net-(J1B-D_{1})
- U9 pad 4: unconnected-(U9-A2-Pad4) -> Net-(J1B-D_{2})
- U9 pad 5: unconnected-(U9-A3-Pad5) -> Net-(J1B-D_{3})
- U9 pad 6: unconnected-(U9-A4-Pad6) -> Net-(J1B-D_{4})
- U9 pad 7: unconnected-(U9-A5-Pad7) -> Net-(J1B-D_{5})
- U9 pad 8: unconnected-(U9-A6-Pad8) -> Net-(J1B-D_{6})
- U9 pad 9: unconnected-(U9-A7-Pad9) -> Net-(J1B-D_{7})
Routing:
- net GND: track 0.00 -> 483.2 mm
- net +5V: track 0.00 -> 296.0 mm
- net /PSG/PG_SEL: track 0.00 -> 80.3 mm, vias 0 -> 2
- net /PSG/BDIR: track 0.00 -> 67.0 mm, vias 0 -> 2
- net Net-(SW2-A): track 0.00 -> 65.6 mm
- net /PSG/SEL: track 0.00 -> 54.9 mm, vias 0 -> 2
- net /PSG/BC1: track 0.00 -> 47.5 mm, vias 0 -> 2
- net CHC: track 0.00 -> 45.1 mm
- net /PSG/A1: track 0.00 -> 45.0 mm
- net /PSG/PHI2: track 0.00 -> 44.1 mm
- net Net-(U2-+): track 0.00 -> 43.0 mm
- net +12V: track 0.00 -> 42.8 mm
- net /PSG/D7: track 0.00 -> 39.8 mm
- net /PSG/D5: track 0.00 -> 39.8 mm
- net /PSG/D6: track 0.00 -> 39.8 mm
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