File: modules/PSG/PSG.kicad_sch (KiCad schematic)
At the start: 8 parts, among them J3 PG SEL, SW1 PAGE SELECT, U1 AY-3-8910, U12 74HC138, U14 74HC688, U4 74HC00, Y1 2Mhz

Commit message: sync
Parts:
- added C13, C14, C15, C16, C17, C18, C2, C20, C4: 100nF, IMNOTWOPR:C_Rect_P200mil, symbol IMNOTWOPR:C
- added C3: 47µF, IMNOTWOPR:CP_Radial_Tantal_P100mil, symbol IMNOTWOPR:C_Polarized
- added J1: CardConnector, IMNOTWOPR:SystemConector_Male, symbol IMNOTWOPR:CardConnector
- added J4: IO PORTS, Connector_PinHeader_2.54mm:PinHeader_2x10_P2.54mm_Vertical, symbol Connector_Generic:Conn_02x10_Odd_Even
- added MH1: CardBracket, IMNOTWOPR:CardBracket, symbol IMNOTWOPR:CardBracket
- added U3: TL072, IMNOTWOPR:DIP-8N, symbol Amplifier_Operational:TL072
- added unit 5 of U4
- added unit 4 of U4
- added unit 3 of U4
- added U7, U8: 74AHCT541, IMNOTWOPR:DIP-20N, symbol 74xx:74AHCT541
- added U9: 74AHCT245, IMNOTWOPR:DIP-20N, symbol 74xx:74HC245
- J3: value PG SEL -> BASE ADDR
- U12: symbol 74xx:74HC138 -> IMNOTWOPR:74HC138
- U4: footprint (none) -> IMNOTWOPR:DIP-14N
Connections:
- net +5V: now also U1.25 (A_{8}), C14.1, C15.1, C16.1, C17.1, C18.1, C2.1, C20.1, C3.1, J1.a1 (+5V), J1.a2 (+5V), J1.a31 (+5V), J1.a32 (+5V), J1.b1 (+5V), J1.b32 (+5V), J4.17 (Pin_17), J4.19 (Pin_19), U4.14 (VCC), U7.20 (VCC), U8.20 (VCC), U9.20 (VCC)
- net A1: now also U4.1, U4.2, U7.17 (Y1); no longer U1.29 (BC_{1})
- net A10: now also U8.16 (Y2)
- net A11: now also U8.15 (Y3)
- net A12: now also U8.14 (Y4)
- net A13: now also U8.13 (Y5)
- net A14: now also U8.12 (Y6)
- net A15: now also U8.11 (Y7)
- net A4: now also U7.14 (Y4)
- net A5: now also U7.13 (Y5)
- net A6: now also U7.12 (Y6)
- net A7: now also U7.11 (Y7)
- net A8: now also U8.18 (Y0)
- net A9: now also U8.17 (Y1)
- net BDIR: now also U4.8, U9.1 (A->B); no longer U4.6
- net D0: now also U9.18 (B0)
- net D1: now also U9.17 (B1)
- net D2: now also U9.16 (B2)
- net D3: now also U9.15 (B3)
- net D4: now also U9.14 (B4)
- net D5: now also U9.13 (B5)
- net D6: now also U9.12 (B6)
- net D7: now also U9.11 (B7)
- net GND: now also U1.24 (~{A_{9}}), C13.1, C14.2, C15.2, C16.2, C17.2, C18.2, C2.2, C20.2, C3.2, C4.2, J1.b2 (GND), J1.b31 (GND), J1.c18 (GND), J1.c2 (GND), J1.c24 (GND), J1.c31 (GND), J1.c32 (GND), J1.c6 (GND), J4.18 (Pin_18), J4.20 (Pin_20), U4.7 (GND), U7.1 (G1), U7.10 (GND), U7.19 (G2), U8.1 (G1), U8.10 (GND), U8.19 (G2), U9.10 (GND)
- net at U12.15 (~{Y0}): now also J3.2 (Pin_2); no longer J3.1 (Pin_1)
- net at U12.10 (~{Y5}): now also J3.12 (Pin_12); no longer J3.11 (Pin_11)
- net at U12.9 (~{Y6}): now also J3.14 (Pin_14); no longer J3.13 (Pin_13)
- net at U12.7 (~{Y7}): now also J3.16 (Pin_16); no longer J3.15 (Pin_15)
- net at U12.14 (~{Y1}): now also J3.4 (Pin_4); no longer J3.3 (Pin_3)
- net at U12.13 (~{Y2}): now also J3.6 (Pin_6); no longer J3.5 (Pin_5)
- net at U12.12 (~{Y3}): now also J3.8 (Pin_8); no longer J3.7 (Pin_7)
- net at U12.11 (~{Y4}): now also J3.10 (Pin_10); no longer J3.9 (Pin_9)
- net at U1.10 (IOB_{3}): now also J4.8 (Pin_8)
- net at U1.11 (IOB_{2}): now also J4.6 (Pin_6)
- net at U1.12 (IOB_{1}): now also J4.4 (Pin_4)
- net at U1.13 (IOB_{0}): now also J4.2 (Pin_2)
- net at U1.14 (IOA_{7}): now also J4.15 (Pin_15)
- net at U1.15 (IOA_{6}): now also J4.13 (Pin_13)
- net at U1.16 (IOA_{5}): now also J4.11 (Pin_11)
- net at U1.17 (IOA_{4}): now also J4.9 (Pin_9)
- net at U1.18 (IOA_{3}): now also J4.7 (Pin_7)
- net at U1.19 (IOA_{2}): now also J4.5 (Pin_5)
- net at U1.20 (IOA_{1}): now also J4.3 (Pin_3)
- net at U1.21 (IOA_{0}): now also J4.1 (Pin_1)
- net at U1.6 (IOB_{7}): now also J4.16 (Pin_16)
- net at U1.7 (IOB_{6}): now also J4.14 (Pin_14)
- net at U1.8 (IOB_{5}): now also J4.12 (Pin_12)
- net at U1.9 (IOB_{4}): now also J4.10 (Pin_10)
- net BC2 renamed SEL
- net SEL: now also U4.6, U4.13, U4.9; no longer U4.3
- net R~{W} renamed PG_SEL
- net PG_SEL: now also J3.1 (Pin_1), J3.11 (Pin_11), J3.13 (Pin_13), J3.15 (Pin_15), J3.3 (Pin_3), J3.5 (Pin_5), J3.7 (Pin_7), J3.9 (Pin_9), U9.19 (CE)
- net ~{BRESET} renamed ~{RESET}
- net ~{RESET}: now also J1.b15 (~{RESET})
- net Φ_{2} renamed PHI2
- net PHI2: now also J1.b12 (Φ_{2})
- new net: J1.a4 (A_{0}), U7.2 (A0)
- new net: J1.a5 (A_{1}), U7.3 (A1)
- new net: J1.a6 (A_{2}), U7.4 (A2)
- new net: J1.a7 (A_{3}), U7.5 (A3)
- new net: J1.a8 (A_{4}), U7.6 (A4)
- new net: J1.a9 (A_{5}), U7.7 (A5)
- new net: J1.a10 (A_{6}), U7.8 (A6)
- new net: J1.a11 (A_{7}), U7.9 (A7)
- new net: J1.a12 (A_{8}), U8.2 (A0)
- new net: J1.a13 (A_{9}), U8.3 (A1)
- new net: J1.a14 (A_{10}), U8.4 (A2)
- new net: J1.a15 (A_{11}), U8.5 (A3)
- new net: J1.a16 (A_{12}), U8.6 (A4)
- new net: J1.a17 (A_{13}), U8.7 (A5)
- new net: J1.a18 (A_{14}), U8.8 (A6)
- new net: J1.a19 (A_{15}), U8.9 (A7)
- new net: J1.b10 (D_{6}), U9.8 (A6)
- new net: J1.b11 (D_{7}), U9.9 (A7)
- new net: J1.b4 (D_{0}), U9.2 (A0)
- new net: J1.b5 (D_{1}), U9.3 (A1)
- new net: J1.b6 (D_{2}), U9.4 (A2)
- new net: J1.b7 (D_{3}), U9.5 (A3)
- new net: J1.b8 (D_{4}), U9.6 (A4)
- new net: J1.b9 (D_{5}), U9.7 (A5)
- new net +12V: C4.1, J1.a3 (+12V), J1.a30 (+12V), U3.8 (V+)
- new net -12V: C13.2, J1.b3 (-12V), J1.b30 (-12V), U3.4 (V-)
- new net BC1: U1.29 (BC_{1}), U4.11
- new net RW: J1.b13 (R~{W}), U4.10
- new net /A1: U4.12, U4.3
- no-connect marks 22 -> 57
Other:
- note added: "BASE ADDRESS"
- note added: "DECOUPLING CAPACITORS"
- note added: "PAGE SELECT"
- note removed: "ADDRESS DECODING"
- moved on the sheet: J3, RN1A, RN1B, RN1C, RN1D, RN1E, RN1F, RN1G, RN1H, SW1, U1, U12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
