File: modules/PSG/system.kicad_sch (KiCad schematic)
At the start: 11 parts, among them J1 CardConnector, U3 TL072, U4 74HC00, U7 74AHCT541, U8 74AHCT541, U9 74AHCT245

Commit message: sync
Parts:
- removed C13, C2, C4: 100nF, IMNOTWOPR:C_Rect_P200mil, symbol IMNOTWOPR:C
- removed C3: 47µF, IMNOTWOPR:CP_Radial_Tantal_P100mil, symbol IMNOTWOPR:C_Polarized
- removed J1: CardConnector, IMNOTWOPR:SystemConector_Male, symbol IMNOTWOPR:CardConnector
- removed MH1: CardBracket, IMNOTWOPR:CardBracket, symbol IMNOTWOPR:CardBracket
- removed U3: TL072, IMNOTWOPR:DIP-8N, symbol Amplifier_Operational:TL072
- removed U4: 74HC00, symbol 74xx:74HC00
- removed U7, U8: 74AHCT541, IMNOTWOPR:DIP-20N, symbol 74xx:74AHCT541
- removed U9: 74AHCT245, IMNOTWOPR:DIP-20N, symbol 74xx:74HC245
Connections:
- no-connect marks 67 -> 0
