File: modules/RAM-1/RAM-1.kicad_sch (KiCad schematic)
At the start: 8 parts, among them U1 2102, U2 2102, U3 2102, U4 2102, U5 2102, U6 2102, U7 2102, U8 2102

Commit message: 1k RAM work
Parts:
- added J1: CardConnector, IMNOTWOPR:SystemConector_Male, symbol IMNOTWOPR:CardConnector
- added RN1: 10k, Resistor_THT:R_Array_SIP7, symbol Device:R_Network06
- added SW1: SW_DIP_x06, Button_Switch_THT:SW_DIP_SPSTx06_Slide_9.78x17.42mm_W7.62mm_P2.54mm, symbol Switch:SW_DIP_x06
- added U10, U9: 74AHCT541, IMNOTWOPR:DIP-20N, symbol 74xx:74AHCT541
- added U11: 74HCT32, IMNOTWOPR:DIP-14N, symbol 74xx:74LS32
- added U12, U15: 74AHCT244, IMNOTWOPR:DIP-20N, symbol 74xx:74AHC244
- added U13: 74HCT00, IMNOTWOPR:DIP-14N, symbol 74xx:74HC00
- added U14: 74HC688, IMNOTWOPR:DIP-20N, symbol 74xx:74HC688
Connections:
- net A0: now also U9.18 (Y0)
- net A1: now also U9.17 (Y1)
- net A2: now also U9.16 (Y2)
- net A3: now also U9.15 (Y3)
- net A4: now also U9.14 (Y4)
- net A5: now also U9.13 (Y5)
- net A6: now also U9.12 (Y6)
- net A7: now also U9.11 (Y7)
- net A8: now also U10.18 (Y0)
- net A9: now also U10.17 (Y1)
- net DI0: now also U15.18 (1Y0)
- net DI1: now also U15.16 (1Y1)
- net DI2: now also U15.14 (1Y2)
- net DI3: now also U15.12 (1Y3)
- net DI4: now also U15.3 (2Y0)
- net DI5: now also U15.5 (2Y1)
- net DI6: now also U15.7 (2Y2)
- net DI7: now also U15.9 (2Y3)
- net DO0: now also U12.2 (1A0)
- net DO1: now also U12.4 (1A1)
- net DO2: now also U12.6 (1A2)
- net DO4: now also U12.17 (2A0); no longer U4.11 (D_{OUT})
- net DO5: now also U12.15 (2A1)
- net DO6: now also U12.13 (2A2)
- net DO7: now also U12.11 (2A3)
- net R~{W}: now also J1.b13 (R~{W}), U11.4, U13.10, U13.4, U13.9; no longer U1.3 (R/~{W}), U2.3 (R/~{W}), U3.3 (R/~{W}), U4.3 (R/~{W}), U5.3 (R/~{W}), U6.3 (R/~{W}), U7.3 (R/~{W}), U8.3 (R/~{W})
- net ~{CE}: now also U11.2, U11.9, U14.19 (P=R)
- new net: U11.6, U15.1 (1OE), U15.19 (2OE)
- new net: RN1.2 (R1), SW1.7, U14.18 (R7)
- new net: RN1.3 (R2), SW1.8, U14.16 (R6)
- new net: RN1.4 (R3), SW1.9, U14.14 (R5)
- new net: RN1.5 (R4), SW1.10, U14.12 (R4)
- new net: RN1.6 (R5), SW1.11, U14.9 (R3)
- new net: RN1.7 (R6), SW1.12, U14.7 (R2)
- new net: U11.10, U13.6
- new net: U11.3, U11.5
- new net: U13.12, U13.8
- new net: U11.8, U12.1 (1OE), U12.19 (2OE)
- new net +5V: J1.a1 (+5V), J1.a2 (+5V), J1.a31 (+5V), J1.a32 (+5V), J1.b1 (+5V), J1.b32 (+5V), SW1.1, SW1.2, SW1.3, SW1.4, SW1.5, SW1.6, U10.20 (VCC), U12.20 (VCC), U14.20 (VCC), U15.20 (VCC), U9.20 (VCC)
- new net A10: U10.16 (Y2), U14.6 (P2)
- new net A11: U10.15 (Y3), U14.8 (P3)
- new net A12: U10.14 (Y4), U14.11 (P4)
- new net A13: U10.13 (Y5), U14.13 (P5)
- new net A14: U10.12 (Y6), U14.15 (P6)
- new net A15: U10.11 (Y7), U14.17 (P7)
- new net DO3: U12.8 (1A3), U4.11 (D_{OUT})
- new net GND: J1.b2 (GND), J1.b31 (GND), RN1.1 (common), U10.1 (G1), U10.10 (GND), U10.19 (G2), U12.10 (GND), U14.1 (G), U14.10 (GND), U14.2 (P0), U14.3 (R0), U14.4 (P1), U14.5 (R1), U15.10 (GND), U9.1 (G1), U9.10 (GND), U9.19 (G2)
- new net PHI2: J1.b12 (Φ_{2}), U13.1, U13.13, U13.2, U13.5
- new net RAM_RW: U1.3 (R/~{W}), U13.11, U2.3 (R/~{W}), U3.3 (R/~{W}), U4.3 (R/~{W}), U5.3 (R/~{W}), U6.3 (R/~{W}), U7.3 (R/~{W}), U8.3 (R/~{W})
- new net SA0: J1.a4 (A_{0}), U9.2 (A0)
- new net SA1: J1.a5 (A_{1}), U9.3 (A1)
- new net SA10: J1.a14 (A_{10}), U10.4 (A2)
- new net SA11: J1.a15 (A_{11}), U10.5 (A3)
- new net SA12: J1.a16 (A_{12}), U10.6 (A4)
- new net SA13: J1.a17 (A_{13}), U10.7 (A5)
- new net SA14: J1.a18 (A_{14}), U10.8 (A6)
- new net SA15: J1.a19 (A_{15}), U10.9 (A7)
- new net SA2: J1.a6 (A_{2}), U9.4 (A2)
- new net SA3: J1.a7 (A_{3}), U9.5 (A3)
- new net SA4: J1.a8 (A_{4}), U9.6 (A4)
- new net SA5: J1.a9 (A_{5}), U9.7 (A5)
- new net SA6: J1.a10 (A_{6}), U9.8 (A6)
- new net SA7: J1.a11 (A_{7}), U9.9 (A7)
- new net SA8: J1.a12 (A_{8}), U10.2 (A0)
- new net SA9: J1.a13 (A_{9}), U10.3 (A1)
- new net SD0: J1.b4 (D_{0}), U12.18 (1Y0), U15.2 (1A0)
- new net SD1: J1.b5 (D_{1}), U12.16 (1Y1), U15.4 (1A1)
- new net SD2: J1.b6 (D_{2}), U12.14 (1Y2), U15.6 (1A2)
- new net SD3: J1.b7 (D_{3}), U12.12 (1Y3), U15.8 (1A3)
- new net SD4: J1.b8 (D_{4}), U12.3 (2Y0), U15.17 (2A0)
- new net SD5: J1.b9 (D_{5}), U12.5 (2Y1), U15.15 (2A1)
- new net SD6: J1.b10 (D_{6}), U12.7 (2Y2), U15.13 (2A2)
- new net SD7: J1.b11 (D_{7}), U12.9 (2Y3), U15.11 (2A3)
- new net ~{PHI}: U11.1, U13.3
- no-connect marks 0 -> 30
Other:
- note added: "PAGE SELECT"
- moved on the sheet: U1A, U2A, U3A, U4A, U5A, U6A, U7A, U8A
