File: modules/RAM-1/system.kicad_sch (KiCad schematic)
At the start: 19 parts, among them J1 CardConnector, U1 2102, U2 2102, U3 2102, U4 2102, U5 2102, U6 2102, U7 2102, U8 2102

Commit message: 1k RAM work
Parts:
- removed unit 2 of J1
- removed unit 1 of J1
- added C10, C11: 100n, IMNOTWOPR:C_Rect_P200mil, symbol IMNOTWOPR:C
- added U11: 74HCT32, IMNOTWOPR:DIP-14N, symbol 74xx:74LS32
- added U13: 74HCT00, IMNOTWOPR:DIP-14N, symbol 74xx:74HC00
Connections:
- net GND: now also C1.2, C2.2, C3.2, C4.2, C5.2, C6.2, C7.2, C8.2, C9.2, U1.9 (GND), U2.9 (GND), U3.9 (GND), U4.9 (GND), U5.9 (GND), U6.9 (GND), U7.9 (GND), U8.9 (GND), C10.2, C11.2, U11.12, U11.13, U11.7 (GND), U13.7 (GND)
- net +5V: now reaches C1.1, C2.1, C3.1, C4.1, C5.1, C6.1, C7.1, C8.1, C9.1, U1.10 (V_{CC}), U2.10 (V_{CC}), U3.10 (V_{CC}), U4.10 (V_{CC}), U5.10 (V_{CC}), U6.10 (V_{CC}), U7.10 (V_{CC}), U8.10 (V_{CC})
- net +5V: now also C10.1, C11.1, U11.14 (VCC), U13.14 (VCC)
- no-connect marks 80 -> 26
Other:
- moved on the sheet: MH1
