File: modules/BTC/system.kicad_sch (KiCad schematic)
At the start: 0 parts

Commit message: lib work and ben wip
Other:
- title: PWR -> BEX
Changed lines of the file:
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@@
 	(paper "A3")
 	(title_block
-		(title "PWR")
-		(rev "B")
+		(title "BEX")
+		(rev "A")
 		(company "THE HOUSE OF GALAHAD")
 		(comment 1 "IMNOTWOPR")
-		(comment 2 "POWER CONTROL")
-		(comment 3 "75-1010-01")
+		(comment 2 "BUS EXERCISER")
+		(comment 3 "75-1098-01")
 	)
 	(sheet_instances
