File: panels/TEMPLATE_8HP/TEMPLATE_8HP.kicad_pcb (KiCad board)
At the start: 2 copper layers, 40.3 x 128.4 mm, 5 parts

Commit message: mega updates.  psg module.  ferrous & example makefiles overhaul
Other:
- board text added: "${TITLE}"
- board text removed: "MOD"
Changed lines of the file:
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@@
 	(paper "USLetter")
 	(title_block
-		(title "TEMPLATE 8HP")
+		(title "8HP")
 		(date "9999-99-99")
 		(rev "A")
@@
 		(comment 2 "mailto:paul.f.burdette@gmail.com")
 		(comment 3 "https://github.com/Desval27/FormantKO/")
-		(comment 4 "No Organic Grounding")
-		(comment 5 "0000-Z")
+		(comment 4 "CURRENT FLOWS WHERE IT WANTS")
+		(comment 5 "75-2002-01")
 	)
 	(layers
@@
 		)
 	)
-	(gr_text "MOD"
+	(gr_text "${TITLE}"
 		(at 86.395894 42.515428 0)
 		(layer "F.SilkS")
@@
 			)
 		)
-		(render_cache "MOD" 0
-			(polygon
-				(pts
-					(xy 83.52598 43.772151) (xy 83.52598 41.638629) (xy 82.291149 43.772151) (xy 81.606597 43.772151)
-					(xy 80.384406 41.638629) (xy 80.384406 43.772151) (xy 79.582252 43.772151) (xy 79.582252 40.94675)
-					(xy 80.938899 40.94675) (xy 81.967833 42.808247) (xy 82.984127 40.94675) (xy 84.332348 40.94675)
-					(xy 84.332348 43.772151)
-				)
-			)
-			(polygon
-				(pts
-					(xy 87.547744 40.939239) (xy 87.869714 40.952627) (xy 88.121374 40.988699) (xy 88.315069 41.042171)
-					(xy 88.461694 41.109083) (xy 88.57045 41.187085) (xy 88.657361 41.287598) (xy 88.73141 41.426208)
-					(xy 88.790574 41.612619) (xy 88.83064 41.858774) (xy 88.845589 42.178467) (xy 88.845589 42.312739)
-					(xy 88.826621 42.777636) (xy 88.777648 43.10783) (xy 88.708792 43.33411) (xy 88.627236 43.482723)
-					(xy 88.53679 43.572507) (xy 88.398432 43.651158) (xy 88.196761 43.716084) (xy 87.912393 43.761417)
-					(xy 87.522648 43.778746) (xy 86.880045 43.791385) (xy 86.611133 43.795598) (xy 86.031545 43.774533)
-					(xy 85.785661 43.758597) (xy 85.583098 43.714321) (xy 85.416481 43.645581) (xy 85.279766 43.554164)
-					(xy 85.169896 43.435325) (xy 85.087853 43.282746) (xy 85.034664 43.088543) (xy 85.015251 42.842135)
-					(xy 85.006824 42.325379) (xy 85.009945 42.251923) (xy 85.86778 42.251923) (xy 85.86778 42.327577)
-					(xy 85.86778 42.440783) (xy 85.881218 42.701212) (xy 85.914194 42.864993) (xy 85.958089 42.961204)
-					(xy 86.008674 43.012321) (xy 86.091205 43.054091) (xy 86.218094 43.083806) (xy 86.40542 43.095476)
-					(xy 86.863192 43.103903) (xy 87.300081 43.09969) (xy 87.54315 43.088684) (xy 87.709576 43.06071)
-					(xy 87.81867 43.02202) (xy 87.881813 42.975255) (xy 87.930333 42.902054) (xy 87.963459 42.79382)
-					(xy 87.976207 42.638071) (xy 87.984633 42.260349) (xy 87.978346 42.074289) (xy 87.961552 41.930988)
-					(xy 87.924128 41.80767) (xy 87.86703 41.729487) (xy 87.783612 41.677701) (xy 87.654905 41.643575)
-					(xy 87.511715 41.627932) (xy 87.35467 41.622509) (xy 86.50617 41.626722) (xy 86.234282 41.643764)
-					(xy 86.065067 41.685523) (xy 85.980009 41.737942) (xy 85.922395 41.818343) (xy 85.890861 41.935201)
-					(xy 85.86778 42.251923) (xy 85.009945 42.251923) (xy 85.026172 41.870025) (xy 85.075643 41.553968)
-					(xy 85.144433 41.34347) (xy 85.225177 41.210166) (xy 85.313776 41.130556) (xy 85.44649 41.060626)
-					(xy 85.637088 41.003002) (xy 85.902545 40.962923) (xy 86.262538 40.947666) (xy 86.867405 40.935026)
-				)
-			)
-			(polygon
-				(pts
-					(xy 92.314571 40.960699) (xy 92.568037 40.998067) (xy 92.76009 41.053097) (xy 92.902839 41.121542)
-					(xy 93.006388 41.201007) (xy 93.08779 41.302658) (xy 93.157846 41.443762) (xy 93.21421 41.634646)
-					(xy 93.252541 41.887789) (xy 93.266873 42.217484) (xy 93.266873 42.378501) (xy 93.266873 42.467528)
-					(xy 93.266873 42.543732) (xy 93.260462 42.823268) (xy 93.212285 43.15153) (xy 93.163694 43.30526)
-					(xy 93.069789 43.448948) (xy 92.922491 43.585855) (xy 92.794736 43.665329) (xy 92.650555 43.723336)
-					(xy 92.487118 43.759508) (xy 92.300954 43.772151) (xy 89.516402 43.772151) (xy 89.516402 43.080455)
-					(xy 90.368932 43.080455) (xy 91.805263 43.080455) (xy 92.012361 43.067612) (xy 92.153411 43.034836)
-					(xy 92.245791 42.988657) (xy 92.302969 42.932078) (xy 92.353314 42.825624) (xy 92.390752 42.647582)
-					(xy 92.405917 42.367877) (xy 92.405917 42.342415) (xy 92.392101 42.061706) (xy 92.358255 41.885597)
-					(xy 92.31341 41.78261) (xy 92.261016 41.728484) (xy 92.171933 41.683638) (xy 92.030853 41.651284)
-					(xy 91.817902 41.638446) (xy 90.368932 41.638446) (xy 90.368932 43.080455) (xy 89.516402 43.080455)
-					(xy 89.516402 40.94675) (xy 91.98588 40.94675)
-				)
-			)
+		(render_cache "8HP" 0
+			(polygon
+				(pts
+					(xy 82.563907 40.959206) (xy 82.803143 40.959206) (xy 83.146462 40.975141) (xy 83.387374 41.016116)
+					(xy 83.550305 41.073651) (xy 83.655672 41.142205) (xy 83.742287 41.239983) (xy 83.806137 41.360486)
+					(xy 83.846899 41.508583) (xy 83.861569 41.690836) (xy 83.845425 41.890433) (xy 83.803403 42.030056)
+					(xy 83.741768 42.125344) (xy 83.653328 42.199782) (xy 83.517679 42.271776) (xy 83.3199 42.339484)
+					(xy 83.518867 42.406757) (xy 83.656878 42.476095) (xy 83.748179 42.54593) (xy 83.813871 42.636009)
+					(xy 83.85762 42.764934) (xy 83.874209 42.946183) (xy 83.863025 43.1912) (xy 83.834275 43.363472)
+					(xy 83.795592 43.46228) (xy 83.731687 43.548699) (xy 83.639003 43.62469) (xy 83.482737 43.706974)
+					(xy 83.347011 43.742659) (xy 83.059415 43.763725) (xy 82.778047 43.767938) (xy 82.206885 43.772151)
+					(xy 81.643966 43.767938) (xy 81.284329 43.750295) (xy 81.020376 43.70402) (xy 80.83137 43.637329)
+					(xy 80.738751 43.57697) (xy 80.664659 43.492197) (xy 80.607878 43.378261) (xy 80.57021 43.227591)
+					(xy 80.556231 43.030447) (xy 80.566998 42.886649) (xy 81.350142 42.886649) (xy 81.359684 42.98823)
+					(xy 81.383664 43.052612) (xy 81.427924 43.101175) (xy 81.503466 43.140906) (xy 81.596005 43.166555)
+					(xy 81.723834 43.185052) (xy 81.980105 43.197692) (xy 82.597429 43.193479) (xy 82.800688 43.178386)
+					(xy 82.946025 43.138891) (xy 83.019334 43.090302) (xy 83.063969 43.016336) (xy 83.080481 42.907531)
+					(xy 83.065598 42.787807) (xy 83.026277 42.70669) (xy 82.964893 42.653275) (xy 82.835187 42.606505)
+					(xy 82.635348 42.588062) (xy 81.778605 42.588062) (xy 81.589389 42.604058) (xy 81.463532 42.644848)
+					(xy 81.403531 42.693118) (xy 81.364917 42.769786) (xy 81.350142 42.886649) (xy 80.566998 42.886649)
+					(xy 80.572935 42.807364) (xy 80.615415 42.65842) (xy 80.675849 42.562783) (xy 80.764794 42.488412)
+					(xy 80.908879 42.410825) (xy 81.127393 42.331057) (xy 80.91778 42.259917) (xy 80.780708 42.187281)
+					(xy 80.696915 42.114902) (xy 80.640871 42.021191) (xy 80.601298 41.875474) (xy 80.592941 41.758613)
+					(xy 81.383664 41.758613) (xy 81.397648 41.861146) (xy 81.435652 41.9342) (xy 81.497054 41.985576)
+					(xy 81.621472 42.031485) (xy 81.795275 42.048774) (xy 82.689936 42.052987) (xy 82.844421 42.036506)
+					(xy 82.960679 41.991621) (xy 83.019198 41.942453) (xy 83.054892 41.875066) (xy 83.067841 41.78316)
+					(xy 83.053234 41.678821) (xy 83.014405 41.609257) (xy 82.952253 41.564623) (xy 82.825541 41.527853)
+					(xy 82.639378 41.513515) (xy 81.824584 41.509485) (xy 81.637631 41.523115) (xy 81.505481 41.558578)
+					(xy 81.438486 41.60185) (xy 81.398332 41.66604) (xy 81.383664 41.758613) (xy 80.592941 41.758613)
+					(xy 80.585723 41.65768) (xy 80.601345 41.465867) (xy 80.643778 41.318064) (xy 80.708778 41.204828)
+					(xy 80.79565 41.119307) (xy 80.94406 41.037641) (xy 81.142362 40.983552) (xy 81.40473 40.963419)
+					(xy 81.917091 40.94675)
+				)
+			)
+			(polygon
+				(pts
+					(xy 88.219289 40.94675) (xy 88.219289 43.772151) (xy 87.362546 43.772151) (xy 87.362546 42.670127)
+					(xy 85.430524 42.670127) (xy 85.430524 43.772151) (xy 84.577995 43.772151) (xy 84.577995 40.94675)
+					(xy 85.430524 40.94675) (xy 85.430524 41.978432) (xy 87.362546 41.978432) (xy 87.362546 40.94675)
+				)
+			)
+			(polygon
+				(pts
+					(xy 91.548422 40.96375) (xy 91.793786 41.008581) (xy 91.97156 41.073696) (xy 92.097072 41.154295)
+					(xy 92.175323 41.239417) (xy 92.241506 41.356471) (xy 92.294125 41.513438) (xy 92.32966 41.720304)
+					(xy 92.342902 41.98869) (xy 92.327431 42.297738) (xy 92.286373 42.530193) (xy 92.226339 42.70163)
+					(xy 92.15166 42.825283) (xy 92.072475 42.902667) (xy 91.961963 42.968091) (xy 91.81209 43.020212)
+					(xy 91.612656 43.055527) (xy 91.351704 43.068732) (xy 91.133167 43.068732) (xy 89.801799 43.068732)
+					(xy 89.801799 43.772151) (xy 88.94927 43.772151) (xy 88.94927 42.377036) (xy 89.801799 42.377036)
+					(xy 91.040843 42.377036) (xy 91.20362 42.367276) (xy 91.312839 42.342576) (xy 91.383028 42.30816)
+					(xy 91.433258 42.253339) (xy 91.467978 42.162157) (xy 91.481763 42.018182) (xy 91.467583 41.865557)
+					(xy 91.431982 41.769202) (xy 91.380829 41.711535) (xy 91.308915 41.675015) (xy 91.196479 41.648811)
+					(xy 91.028204 41.638446) (xy 89.801799 41.638446) (xy 89.801799 42.377036) (xy 88.94927 42.377036)
+					(xy 88.94927 40.94675) (xy 91.217248 40.94675)
+				)
+			)

Commit message: ben schematic
Parts:
- added REF**: Panel_LED_5.0mm_z1, IMNOTWOPR:Panel_LED_5.0mm_z1, F.Cu at (74.7, 67.7)
- added REF**: DB-9 Panel, IMNOTWOPR:DB-9 Panel, F.Cu at (86.7, 99.2)
