File: modules/BEN/BEN.kicad_pcb (KiCad board)
At the start: 2 copper layers, 160 x 100 mm, 6 parts, among them J1 CardConnector, U1 28C256, U2 62256, U3 74HCT541, U4 74HCT541

Commit message: ben schematic wip
Parts:
- added C1: 47u, IMNOTWOPR:CP_Radial_Tantal_P100mil, F.Cu at (193.8, 135.0)
- added C10: 47u, IMNOTWOPR:CP_Radial_Tantal_P100mil, F.Cu at (105.5, 51.0)
- added C11: 47u, IMNOTWOPR:CP_Radial_Tantal_P100mil, F.Cu at (105.5, 59.7)
- added C12: 100n, IMNOTWOPR:C_Rect_P200mil, F.Cu at (117.3, 61.7)
- added C13: 100n, IMNOTWOPR:C_Rect_P200mil, F.Cu at (117.3, 65.0)
- added C14: 100n, IMNOTWOPR:C_Rect_P200mil, F.Cu at (117.3, 68.2)
- added C2: 100n, IMNOTWOPR:C_Rect_P200mil, F.Cu at (78.3, 52.9)
- added C3: 100n, IMNOTWOPR:C_Rect_P200mil, F.Cu at (78.3, 56.1)
- added C4: 100n, IMNOTWOPR:C_Rect_P200mil, F.Cu at (78.3, 59.3)
- added C5: 100n, IMNOTWOPR:C_Rect_P200mil, F.Cu at (78.3, 62.6)
- added C6: 100n, IMNOTWOPR:C_Rect_P200mil, F.Cu at (78.3, 65.8)
- added C7: 100n, IMNOTWOPR:C_Rect_P200mil, F.Cu at (78.3, 69.0)
- added C8: 100n, IMNOTWOPR:C_Rect_P200mil, F.Cu at (117.3, 55.3)
- added C9: 100n, IMNOTWOPR:C_Rect_P200mil, F.Cu at (117.3, 58.5)
- added D1: WP483SEKJ3CGKWT, LED_THT:LED_D5.0mm_FlatTop, F.Cu at (96.2, 50.4)
- added D2: WP483SEKJ3CGKWT, LED_THT:LED_D5.0mm_FlatTop, F.Cu at (96.2, 58.0)
- added D3: WP483SEKJ3CGKWT, LED_THT:LED_D5.0mm_FlatTop, F.Cu at (96.2, 65.6)
- added J2: DE9_Socket, Connector_Dsub:DSUB-9_Socket_Horizontal_P2.77x2.54mm_EdgePinOffset9.40mm, F.Cu at (68.7, 60.2)
- added J3: Conn_02x05_Odd_Even, Connector_IDC:IDC-Header_2x05_P2.54mm_Vertical, F.Cu at (58.6, 68.3)
- added R1: 1k, IMNOTWOPR:R_Axial_DIN0207_P400mil, F.Cu at (129.2, 55.6)
- added R2: 1k, IMNOTWOPR:R_Axial_DIN0207_P400mil, F.Cu at (129.2, 59.6)
- added R3: 1k, IMNOTWOPR:R_Axial_DIN0207_P400mil, F.Cu at (129.2, 63.5)
- added U3: 74AHCT245, IMNOTWOPR:DIP-20N, F.Cu at (184.3, 72.1)
- added U6: W65C22, IMNOTWOPR:DIP-40W, F.Cu at (110.6, 122.3)
- added U7: W65C51, IMNOTWOPR:DIP-28W, F.Cu at (155.1, 122.9)
- added U8: MC1488, FormantKO:DIP-14N, F.Cu at (63.6, 119.1)
- added U9: MC1489, FormantKO:DIP-14N, F.Cu at (76.3, 119.1)
- U1: renamed from U3; value 74HCT541 -> 74AHCT541
- U2: renamed from U4; value 74HCT541 -> 74AHCT541
- moved U1 25.4 mm to (158.9, 72.1)
- moved U4 14.9 mm to (80.2, 95.0), turned to 90 degrees
- moved U5 5.36 mm to (133.5, 95.0), turned to 180 degrees
- moved U2 5.08 mm to (171.6, 92.5)
- renumbered U1 to U4, U2 to U5
Connections:
- net /BEN/D0 renamed /D0
- net /BEN/D1 renamed /D1
- net /BEN/D2 renamed /D2
- net /BEN/D3 renamed /D3
- net /BEN/D4 renamed /D4
- net /BEN/D5 renamed /D5
- net /BEN/D6 renamed /D6
- net /BEN/D7 renamed /D7
- net /BEN/SA0 renamed /BA0
- net /BEN/SA1 renamed /BA1
- net /BEN/SA10 renamed /BA10
- net /BEN/SA11 renamed /BA11
- net /BEN/SA12 renamed /BA12
- net /BEN/SA13 renamed /BA13
- net /BEN/SA14 renamed /BA14
- net /BEN/SA15 renamed /BA15
- net /BEN/SA2 renamed /BA2
- net /BEN/SA3 renamed /BA3
- net /BEN/SA4 renamed /BA4
- net /BEN/SA5 renamed /BA5
- net /BEN/SA6 renamed /BA6
- net /BEN/SA7 renamed /BA7
- net /BEN/SA8 renamed /BA8
- net /BEN/SA9 renamed /BA9
- J1 pad a3: unconnected-(J1A-+12V-Pada3) -> +12V
- J1 pad a30: unconnected-(J1A-+12V-Pada30) -> +12V
- J1 pad b10: unconnected-(J1B-D_{6}-Padb10) -> /BD6
- J1 pad b11: unconnected-(J1B-D_{7}-Padb11) -> /BD7
- J1 pad b13: unconnected-(J1B-R~{W}-Padb13) -> /R~{W}
- J1 pad b14: unconnected-(J1B-~{VALID}-Padb14) -> /~{VALID}
- J1 pad b3: unconnected-(J1B--12V-Padb3) -> -12V
- J1 pad b30: unconnected-(J1B--12V-Padb30) -> -12V
- J1 pad b4: unconnected-(J1B-D_{0}-Padb4) -> /BD0
- J1 pad b5: unconnected-(J1B-D_{1}-Padb5) -> /BD1
- J1 pad b6: unconnected-(J1B-D_{2}-Padb6) -> /BD2
- J1 pad b7: unconnected-(J1B-D_{3}-Padb7) -> /BD3
- J1 pad b8: unconnected-(J1B-D_{4}-Padb8) -> /BD4
- J1 pad b9: unconnected-(J1B-D_{5}-Padb9) -> /BD5
- U1 pad 1: unconnected-(U3A-/OE1-Pad1) -> /~{VALID}
- U1 pad 10: unconnected-(U3B-GND-Pad10) -> GND
- U1 pad 11: unconnected-(U3A-Y7-Pad11) -> /A7
- U1 pad 12: unconnected-(U3A-Y6-Pad12) -> /A6
- U1 pad 13: unconnected-(U3A-Y5-Pad13) -> /A5
- U1 pad 14: unconnected-(U3A-Y4-Pad14) -> /A4
- U1 pad 15: unconnected-(U3A-Y3-Pad15) -> /A3
- U1 pad 16: unconnected-(U3A-Y2-Pad16) -> /A2
- U1 pad 17: unconnected-(U3A-Y1-Pad17) -> /A1
- U1 pad 18: unconnected-(U3A-Y0-Pad18) -> /A0
- U1 pad 19: unconnected-(U3A-/OE2-Pad19) -> /~{VALID}
- U1 pad 20: unconnected-(U3B-VCC-Pad20) -> +5V
- U2 pad 1: unconnected-(U4A-/OE1-Pad1) -> /~{VALID}
- U2 pad 10: unconnected-(U4B-GND-Pad10) -> GND
- U2 pad 11: unconnected-(U4A-Y7-Pad11) -> /A15
- U2 pad 12: unconnected-(U4A-Y6-Pad12) -> /A14
- U2 pad 13: unconnected-(U4A-Y5-Pad13) -> /A13
- U2 pad 14: unconnected-(U4A-Y4-Pad14) -> /A12
- U2 pad 15: unconnected-(U4A-Y3-Pad15) -> /A11
- U2 pad 16: unconnected-(U4A-Y2-Pad16) -> /A10
- U2 pad 17: unconnected-(U4A-Y1-Pad17) -> /A9
- U2 pad 18: unconnected-(U4A-Y0-Pad18) -> /A8
- U2 pad 19: unconnected-(U4A-/OE2-Pad19) -> /~{VALID}
- U2 pad 20: unconnected-(U4B-VCC-Pad20) -> +5V
- U4 pad 1: unconnected-(U1A-A_{14}-Pad1) -> /A14
- U4 pad 10: unconnected-(U1A-A_{0}-Pad10) -> /A0
- U4 pad 14: unconnected-(U1B-GND-Pad14) -> GND
- U4 pad 2: unconnected-(U1A-A_{12}-Pad2) -> /A12
- U4 pad 21: unconnected-(U1A-A_{10}-Pad21) -> /A10
- U4 pad 23: unconnected-(U1A-A_{11}-Pad23) -> /A11
- U4 pad 24: unconnected-(U1A-A_{9}-Pad24) -> /A9
- U4 pad 25: unconnected-(U1A-A_{8}-Pad25) -> /A8
- U4 pad 26: unconnected-(U1A-A_{13}-Pad26) -> /A13
- U4 pad 28: unconnected-(U1B-VCC-Pad28) -> +5V
- U4 pad 3: unconnected-(U1A-A_{7}-Pad3) -> /A7
- U4 pad 4: unconnected-(U1A-A_{6}-Pad4) -> /A6
- U4 pad 5: unconnected-(U1A-A_{5}-Pad5) -> /A5
- U4 pad 6: unconnected-(U1A-A_{4}-Pad6) -> /A4
- U4 pad 7: unconnected-(U1A-A_{3}-Pad7) -> /A3
- U4 pad 8: unconnected-(U1A-A_{2}-Pad8) -> /A2
- U4 pad 9: unconnected-(U1A-A_{1}-Pad9) -> /A1
- U5 pad 1: unconnected-(U2A-A_{14}-Pad1) -> /A14
- U5 pad 10: unconnected-(U2A-A_{0}-Pad10) -> /A0
- U5 pad 14: unconnected-(U2B-GND-Pad14) -> GND
- U5 pad 2: unconnected-(U2A-A_{12}-Pad2) -> /A12
- U5 pad 21: unconnected-(U2A-A_{10}-Pad21) -> /A10
- U5 pad 23: unconnected-(U2A-A_{11}-Pad23) -> /A11
- U5 pad 24: unconnected-(U2A-A_{9}-Pad24) -> /A9
- U5 pad 25: unconnected-(U2A-A_{8}-Pad25) -> /A8
- U5 pad 26: unconnected-(U2A-A_{13}-Pad26) -> /A13
- U5 pad 28: unconnected-(U2B-VCC-Pad28) -> +5V
- U5 pad 3: unconnected-(U2A-A_{7}-Pad3) -> /A7
- U5 pad 4: unconnected-(U2A-A_{6}-Pad4) -> /A6
- U5 pad 5: unconnected-(U2A-A_{5}-Pad5) -> /A5
- U5 pad 6: unconnected-(U2A-A_{4}-Pad6) -> /A4
- U5 pad 7: unconnected-(U2A-A_{3}-Pad7) -> /A3
- U5 pad 8: unconnected-(U2A-A_{2}-Pad8) -> /A2
- U5 pad 9: unconnected-(U2A-A_{1}-Pad9) -> /A1
Routing:
- net GND: track 0.00 -> 49.1 mm
- net /BA6: track 31.3 -> 55.7 mm
- net /BA4: track 31.3 -> 55.7 mm
- net /BA7: track 31.3 -> 55.7 mm
- net /BA5: track 31.3 -> 55.7 mm
- net /BA2: track 31.3 -> 55.7 mm
- net /BA0: track 31.3 -> 55.7 mm
- net /BA3: track 31.3 -> 55.7 mm
- net /BA1: track 31.3 -> 55.7 mm
- net /A9: track 0.00 -> 12.0 mm
- net /A11: track 0.00 -> 12.0 mm
- net /A8: track 0.00 -> 12.0 mm
- net /A15: track 0.00 -> 12.0 mm
- net /A14: track 0.00 -> 12.0 mm
- net /A13: track 0.00 -> 12.0 mm
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Other:
- board text removed: "SA_{0}"
- board text removed: "SA_{1}"
- board text removed: "SA_{2}"
- board text removed: "SA_{3}"
- board text removed: "SA_{4}"
- board text removed: "SA_{5}"
- board text removed: "SA_{6}"

Commit message: lib work and ben wip
Parts:
- removed J3: Conn_02x05_Odd_Even, Connector_IDC:IDC-Header_2x05_P2.54mm_Vertical
- added C15: 100n, IMNOTWOPR:C_Rect_P200mil, F.Cu at (30.0, 62.4)
- added C16: 100n, IMNOTWOPR:C_Rect_P200mil, F.Cu at (30.0, 65.6)
- added C17: 100n, IMNOTWOPR:C_Rect_P200mil, F.Cu at (30.0, 68.9)
- added C18: 100n, IMNOTWOPR:C_Rect_P200mil, F.Cu at (30.0, 72.1)
- added C19: 100n, IMNOTWOPR:C_Rect_P200mil, F.Cu at (30.0, 75.3)
- added C20: 100n, IMNOTWOPR:C_Rect_P200mil, F.Cu at (30.0, 78.6)
- added C21: 100n, IMNOTWOPR:C_Rect_P200mil, F.Cu at (30.0, 81.8)
- added C22: 100n, IMNOTWOPR:C_Rect_P200mil, F.Cu at (30.0, 85.0)
- added D10: LED_G, IMNOTWOPR:LED_G_D5.0mm, F.Cu at (8.32, 41.1)
- added D11: LED_G, IMNOTWOPR:LED_G_D5.0mm, F.Cu at (8.32, 48.6)
- added D12: LED_G, IMNOTWOPR:LED_G_D5.0mm, F.Cu at (15.8, 41.1)
- added D13: LED_G, IMNOTWOPR:LED_G_D5.0mm, F.Cu at (15.8, 48.6)
- added D14: LED_G, IMNOTWOPR:LED_G_D5.0mm, F.Cu at (23.3, 41.1)
- added D15: LED_G, IMNOTWOPR:LED_G_D5.0mm, F.Cu at (23.3, 48.6)
- added D16: SB140, Diode_THT:D_DO-41_SOD81_P10.16mm_Horizontal, F.Cu at (15.8, 54.4)
- added D17: SB140, Diode_THT:D_DO-41_SOD81_P10.16mm_Horizontal, F.Cu at (15.8, 58.7)
- added D4: WP483SEKJ3CGKWT, LED_THT:LED_D5.0mm_FlatTop, F.Cu at (28.4, 90.4)
- added D5: WP483SEKJ3CGKWT, LED_THT:LED_D5.0mm_FlatTop, F.Cu at (28.4, 98.0)
- added D6: WP483SEKJ3CGKWT, LED_THT:LED_D5.0mm_FlatTop, F.Cu at (28.4, 105.6)
- added D7: WP483SEKJ3CGKWT, LED_THT:LED_D5.0mm_FlatTop, F.Cu at (28.4, 113.1)
- added D8: LED_G, IMNOTWOPR:LED_G_D5.0mm, F.Cu at (0.84, 41.1)
- added D9: LED_G, IMNOTWOPR:LED_G_D5.0mm, F.Cu at (0.84, 48.6)
- added R10: 1k, IMNOTWOPR:R_Axial_DIN0207_P400mil, F.Cu at (6.14, 77.9)
- added R11: 1k, IMNOTWOPR:R_Axial_DIN0207_P400mil, F.Cu at (6.14, 81.8)
- added R12: 1k, IMNOTWOPR:R_Axial_DIN0207_P400mil, F.Cu at (6.14, 85.8)
- added R13: 1k, IMNOTWOPR:R_Axial_DIN0207_P400mil, F.Cu at (6.14, 89.7)
- added R14: 1k, IMNOTWOPR:R_Axial_DIN0207_P400mil, F.Cu at (6.14, 93.7)
- added R15: 1k, IMNOTWOPR:R_Axial_DIN0207_P400mil, F.Cu at (6.14, 97.6)
- added R16: 10k, IMNOTWOPR:R_Axial_DIN0207_P400mil, F.Cu at (6.14, 101.5)
- added R17: 10k, IMNOTWOPR:R_Axial_DIN0207_P400mil, F.Cu at (6.14, 105.5)
- added R18: 10k, IMNOTWOPR:R_Axial_DIN0207_P400mil, F.Cu at (6.14, 109.4)
- added R19: 10k, IMNOTWOPR:R_Axial_DIN0207_P400mil, F.Cu at (6.14, 113.4)
- added R20: 10k, IMNOTWOPR:R_Axial_DIN0207_P400mil, F.Cu at (6.14, 117.3)
- added R21: 10k, IMNOTWOPR:R_Axial_DIN0207_P400mil, F.Cu at (6.14, 121.2)
- added R22: 10k, IMNOTWOPR:R_Axial_DIN0207_P400mil, F.Cu at (6.14, 125.2)
- added R23: 10k, IMNOTWOPR:R_Axial_DIN0207_P400mil, F.Cu at (6.14, 129.1)
- added R24: 1M, IMNOTWOPR:R_Axial_DIN0207_P400mil, F.Cu at (6.14, 133.1)
- added R4: 1k, IMNOTWOPR:R_Axial_DIN0207_P400mil, F.Cu at (6.14, 54.3)
- added R5: 1k, IMNOTWOPR:R_Axial_DIN0207_P400mil, F.Cu at (6.14, 58.2)
- added R6: 1k, IMNOTWOPR:R_Axial_DIN0207_P400mil, F.Cu at (6.14, 62.1)
- added R7: 1k, IMNOTWOPR:R_Axial_DIN0207_P400mil, F.Cu at (6.14, 66.1)
- added R8: 1k, IMNOTWOPR:R_Axial_DIN0207_P400mil, F.Cu at (6.14, 70.0)
- added R9: 1k, IMNOTWOPR:R_Axial_DIN0207_P400mil, F.Cu at (6.14, 74.0)
- added SW1: 2MS1T1B1M1QES, IMNOTWOPR:PanelConnector_1x03, F.Cu at (19.9, 65.2)
- added SW2: SW_SPST, IMNOTWOPR:PanelConnector_1x03, F.Cu at (19.9, 73.0)
- added SW3: 2MS1T1B1M1QES, IMNOTWOPR:PanelConnector_1x03, F.Cu at (19.9, 80.8)
- added SW4: 2MS1T1B1M1QES, IMNOTWOPR:PanelConnector_1x03, F.Cu at (19.9, 88.6)
- added SW5: 2MS1T1B1M1QES, IMNOTWOPR:PanelConnector_1x03, F.Cu at (19.9, 96.4)
- added SW6: 2MS1T1B1M1QES, IMNOTWOPR:PanelConnector_1x03, F.Cu at (19.9, 104.2)
- added SW7: 2MS1T1B1M1QES, IMNOTWOPR:PanelConnector_1x03, F.Cu at (19.9, 112.0)
- added SW8: 2MS1T1B1M1QES, IMNOTWOPR:PanelConnector_1x03, F.Cu at (19.9, 119.8)
- added SW9: 2MS1T1B1M1QES, IMNOTWOPR:PanelConnector_1x03, F.Cu at (19.9, 127.6)
- added Y1: 1.8432Mhz, Crystal:Crystal_HC49-U_Vertical, F.Cu at (87.9, 82.3)
- J2: value DE9_Socket -> IDC DE9 Female; footprint Connector_Dsub:DSUB-9_Socket_Horizontal_P2.77x2.54mm_EdgePinOffset9.40mm -> Connector_PinHeader_2.54mm:PinHeader_2x05_P2.54mm_Vertical
- moved U7 82.8 mm to (92.9, 68.3), turned to 90 degrees
- moved C12 76.8 mm to (45.4, 34.8)
- moved C13 76.8 mm to (45.4, 38.0)
- moved C14 76.8 mm to (45.4, 41.3)
- moved C8 76.8 mm to (45.4, 28.3)
- moved C9 76.8 mm to (45.4, 31.6)
- moved C10 76.8 mm to (33.7, 24.1)
- moved C11 76.8 mm to (33.7, 32.7)
- moved C2 76.8 mm to (6.37, 25.9)
- moved C3 76.8 mm to (6.37, 29.2)
- moved C4 76.8 mm to (6.37, 32.4)
- moved C5 76.8 mm to (6.37, 35.6)
- moved C6 76.8 mm to (6.37, 38.9)
- moved C7 76.8 mm to (6.37, 42.1)
- moved D1 76.8 mm to (24.3, 23.5)
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Connections:
- J1 pad b12: unconnected-(J1B-Φ_{2}-Padb12) -> /PHI2
- J1 pad b15: unconnected-(J1B-~{RESET}-Padb15) -> /~{RESET}
- J1 pad b16: unconnected-(J1B-~{IRQ}-Padb16) -> /~{IRQ}
- J2 pad 1: unconnected-(J2-Pad1) -> /~{DCD}
- J2 pad 2: unconnected-(J2-Pad2) -> /TXD
- J2 pad 3: unconnected-(J2-Pad3) -> /RXD
- J2 pad 4: unconnected-(J2-Pad4) -> /~{DTR}
- J2 pad 5: unconnected-(J2-Pad5) -> GND
- J2 pad 6: unconnected-(J2-Pad6) -> /~{DSR}
- J2 pad 7: unconnected-(J2-Pad7) -> /~{RTS}
- J2 pad 8: unconnected-(J2-Pad8) -> /~{CTS}
- R1 pad 1: Net-(J3-Pin_4) -> /~{RTS}
- R2 pad 1: Net-(J3-Pin_7) -> /~{DTR}
- R3 pad 1: Net-(J3-Pin_5) -> /TXD
- U4 pad 22: unconnected-(U4A-/OE-Pad22) -> /~{VALID}
- U4 pad 27: unconnected-(U4A-/WE-Pad27) -> +5V
- U5 pad 22: unconnected-(U5A-/OE-Pad22) -> /~{VALID}
- U5 pad 27: unconnected-(U5A-/WE-Pad27) -> /R~{W}
- U6 pad 21: unconnected-(U6A-~{IRQ}-Pad21) -> Net-(D16-K)
- U6 pad 22: unconnected-(U6A-~{RW}-Pad22) -> /R~{W}
- U6 pad 25: unconnected-(U6A-Φ_{2}-Pad25) -> /PHI2
- U6 pad 34: unconnected-(U6A-~{RESET}-Pad34) -> /~{RESET}
- U6 pad 35: unconnected-(U6A-RS_{3}-Pad35) -> /A3
- U6 pad 36: unconnected-(U6A-RS_{2}-Pad36) -> /A2
- U6 pad 37: unconnected-(U6A-RS_{1}-Pad37) -> /A1
- U6 pad 38: unconnected-(U6A-RS_{0}-Pad38) -> /A0
- U7 pad 13: unconnected-(U7A-RS_{0}-Pad13) -> /A0
- U7 pad 14: unconnected-(U7A-RS_{1}-Pad14) -> /A1
- U7 pad 26: unconnected-(U7A-~{IRQ}-Pad26) -> Net-(D17-K)
- U7 pad 27: unconnected-(U7A-Φ_{2}-Pad27) -> /PHI2
- U7 pad 28: unconnected-(U7A-~{RW}-Pad28) -> /R~{W}
- U7 pad 4: unconnected-(U7A-~{RESET}-Pad4) -> /~{RESET}
- U7 pad 6: unconnected-(U7A-XTLI-Pad6) -> Net-(U7A-XTLI)
- U7 pad 7: unconnected-(U7A-XTLO-Pad7) -> Net-(U7A-XTLO)
- U8 pad 10: (no net) -> Net-(U7A-~{RTS})
- U8 pad 11: (no net) -> unconnected-(U8D-4Y-Pad11)
- U8 pad 13: (no net) -> GND
- U8 pad 3: Net-(J3-Pin_5) -> /TXD
- U8 pad 6: Net-(J3-Pin_7) -> /~{DTR}
- U8 pad 8: (no net) -> /~{RTS}
- U9 pad 1: Net-(J3-Pin_3) -> /RXD
- U9 pad 10: Net-(J3-Pin_2) -> /~{DSR}
- U9 pad 13: Net-(J3-Pin_6) -> /~{CTS}
- U9 pad 3: (no net) -> Net-(U7A-R_{X}D)
- U9 pad 4: Net-(J3-Pin_1) -> /~{DCD}
- U9 pad 8: (no net) -> Net-(U7A-~{DSR})
Routing:
- net /D4: track 0.00 -> 100.6 mm, vias 0 -> 1
- net /D3: track 0.00 -> 100.6 mm, vias 0 -> 1
- net /D7: track 0.00 -> 99.9 mm, vias 0 -> 2
- net /D6: track 0.00 -> 99.9 mm, vias 0 -> 2
- net /D5: track 0.00 -> 99.9 mm, vias 0 -> 2
- net /D2: track 0.00 -> 78.5 mm, vias 0 -> 1
- net /D1: track 0.00 -> 74.5 mm, vias 0 -> 1
- net /D0: track 0.00 -> 69.4 mm, vias 0 -> 1
- net /BA6: track 55.7 -> 0.00 mm
- net /BA4: track 55.7 -> 0.00 mm
- net /BA7: track 55.7 -> 0.00 mm
- net /BA3: track 55.7 -> 0.00 mm
- net /BA0: track 55.7 -> 0.00 mm
- net /BA5: track 55.7 -> 0.00 mm
- net /BA2: track 55.7 -> 0.00 mm
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Other:
- board text removed: "BUS BUFFER"

Commit message: ben schematic
Parts:
- removed the D1 at (24.3, 23.5)
- removed the D2 at (24.3, 31.1)
- removed the D3 at (24.3, 38.7)
- removed the D4 at (28.4, 90.4)
- removed the D5 at (28.4, 98.0)
- removed the D6 at (28.4, 105.6)
- removed the D7 at (28.4, 113.1)
- removed R10, R11, R12, R13, R14, R15: 1k, IMNOTWOPR:R_Axial_DIN0207_P400mil
- removed R16, R17, R18, R19, R20, R21, R22, R23: 10k, IMNOTWOPR:R_Axial_DIN0207_P400mil
- removed the R9 at (6.14, 74.0)
- removed the SW2 at (19.9, 73.0)
- added C15: 100n, IMNOTWOPR:C_Rect_P200mil, F.Cu at (138.6, 107.7)
- added C16: 100n, IMNOTWOPR:C_Rect_P200mil, F.Cu at (22.4, 144.9)
- added C17: 100n, IMNOTWOPR:C_Rect_P200mil, F.Cu at (22.4, 148.1)
- added C26: 30pF, IMNOTWOPR:C_Rect_P200mil, F.Cu at (22.4, 141.6)
- added D11: LED_R, IMNOTWOPR:LED_D5.0mm_Horizontal_O1.27mm_Z3.0mm, F.Cu at (51.2, 100.1)
- added D12: LED_R, IMNOTWOPR:LED_D5.0mm_Horizontal_O1.27mm_Z3.0mm, F.Cu at (51.2, 107.7)
- added D13: LED_R, IMNOTWOPR:LED_D5.0mm_Horizontal_O1.27mm_Z3.0mm, F.Cu at (51.2, 115.3)
- added D14: LED_R, IMNOTWOPR:LED_D5.0mm_Horizontal_O1.27mm_Z3.0mm, F.Cu at (51.2, 122.9)
- added D15: LED_R, IMNOTWOPR:LED_D5.0mm_Horizontal_O3.81mm_Z9.0mm, F.Cu at (51.2, 103.9)
- added D16: LED_R, IMNOTWOPR:LED_D5.0mm_Horizontal_O3.81mm_Z9.0mm, F.Cu at (51.2, 111.5)
- added D17: LED_R, IMNOTWOPR:LED_D5.0mm_Horizontal_O3.81mm_Z9.0mm, F.Cu at (51.2, 119.1)
- added D18: LED_R, IMNOTWOPR:LED_D5.0mm_Horizontal_O3.81mm_Z9.0mm, F.Cu at (51.2, 126.8)
- added J2: Conn_01x04, Connector_PinSocket_2.54mm:PinSocket_1x04_P2.54mm_Vertical, F.Cu at (43.9, 72.7)
- added RN1: 10kΩ, Resistor_THT:R_Array_SIP9, F.Cu at (40.8, 176.3)
- added RN2: 1k, Resistor_THT:R_Array_SIP9, F.Cu at (65.4, 84.8)
- added RN3: 10k, Resistor_THT:R_Array_SIP9, F.Cu at (70.6, 105.8)
- added RN4: 1k5, Resistor_THT:R_Array_SIP9, F.Cu at (66.2, 106.4)
- added SW1: PAGE SELECT, Button_Switch_THT:SW_DIP_SPSTx08_Slide_9.78x22.5mm_W7.62mm_P2.54mm, F.Cu at (43.3, 191.5)
- added U1: 74HCT13, FormantKO:DIP-14N, F.Cu at (92.9, 87.4)
- added U11: 74HC688, IMNOTWOPR:DIP-20N, F.Cu at (120.8, 89.9)
- added U14: 74HC138, IMNOTWOPR:DIP-16N, F.Cu at (122.1, 111.5)
- added U3: 74HCT32, IMNOTWOPR:DIP-14N, F.Cu at (230.0, 97.5)
- added U5: 74HCT00, IMNOTWOPR:DIP-14N, F.Cu at (96.7, 102.6)
- D1: renamed from D16; value SB140 -> 1N5817
- D10: renamed from D13; footprint IMNOTWOPR:LED_G_D5.0mm -> IMNOTWOPR:LED_D5.0mm_Horizontal_O3.81mm_Z9.0mm
- D2: renamed from D8; footprint IMNOTWOPR:LED_G_D5.0mm -> IMNOTWOPR:LED_D5.0mm_Horizontal_O1.27mm_Z3.0mm
- D3: renamed from D9; footprint IMNOTWOPR:LED_G_D5.0mm -> IMNOTWOPR:LED_D5.0mm_Horizontal_O1.27mm_Z3.0mm
- D4: renamed from D10; footprint IMNOTWOPR:LED_G_D5.0mm -> IMNOTWOPR:LED_D5.0mm_Horizontal_O1.27mm_Z3.0mm
- D5: renamed from D11; footprint IMNOTWOPR:LED_G_D5.0mm -> IMNOTWOPR:LED_D5.0mm_Horizontal_O1.27mm_Z3.0mm
- D6: renamed from D17; value SB140 -> 1N5817
- D7: renamed from D14; footprint IMNOTWOPR:LED_G_D5.0mm -> IMNOTWOPR:LED_D5.0mm_Horizontal_O3.81mm_Z9.0mm
- D8: renamed from D15; footprint IMNOTWOPR:LED_G_D5.0mm -> IMNOTWOPR:LED_D5.0mm_Horizontal_O3.81mm_Z9.0mm
- D9: renamed from D12; footprint IMNOTWOPR:LED_G_D5.0mm -> IMNOTWOPR:LED_D5.0mm_Horizontal_O3.81mm_Z9.0mm
- U9: renamed from U3; value 74AHCT245 -> 74AHCT245_Slave
- moved C8 202.7 mm to (197.0, 101.3), turned to 180 degrees
- moved C2 193.3 mm to (197.0, 58.2), turned to 180 degrees
- moved C5 185.9 mm to (185.6, 78.5), turned to 180 degrees
- moved D6 152.0 mm to (21.7, 210.6)
- moved R4 140.5 mm to (84.0, 171.2)
- moved R5 140.5 mm to (84.0, 175.1)
- moved R6 140.5 mm to (84.0, 179.1)
- moved R7 140.5 mm to (84.0, 183.0)
- moved R8 140.5 mm to (84.0, 187.0)
- moved D1 139.8 mm to (117.0, 150.9)
- moved R1 133.4 mm to (84.0, 159.4)
- moved R2 133.4 mm to (84.0, 163.3)
- moved R3 133.4 mm to (84.0, 167.3)
- moved C10 126.7 mm to (132.2, 53.1), turned to -90 degrees
- moved C9 125.4 mm to (113.2, 101.3), turned to -90 degrees
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- renumbered C6 to C10, C7 to C11, C8 to C12, C9 to C13, C15 to C18, C16 to C19, C17 to C20, C18 to C21, C19 to C22, C20 to C23, C21 to C24, C22 to C25, C10 to C3, C11 to C4, C3 to C5, C12 to C6, C13 to C7, C4 to C8, C5 to C9, J2 to J3, R24 to R9, SW1 to SW2, U6 to U10, U7 to U12, U9 to U13, U4 to U2, U5 to U4, U8 to U6, U1 to U7, U2 to U8
Connections:
- C18 pad 1: /PB0 -> Net-(RN3A-R1.2)
- C19 pad 1: /PB1 -> Net-(RN3B-R2.2)
- C20 pad 1: /PB2 -> Net-(RN3C-R3.2)
- C21 pad 1: /PB3 -> Net-(RN3D-R4.2)
- C22 pad 1: /PB4 -> Net-(RN3E-R5.2)
- C23 pad 1: /PB5 -> Net-(RN3F-R6.2)
- C24 pad 1: /PB6 -> Net-(RN3G-R7.2)
- C25 pad 1: /PB7 -> Net-(RN3H-R8.2)
- D2 pad 2: Net-(D8-A) (its old number) -> Net-(D2-A)
- J1 pad b10: /BD6 -> unconnected-(J1B-READY-Padb10)
- J1 pad b11: /BD7 -> unconnected-(J1B-BE-Padb11)
- J1 pad b12: /PHI2 -> unconnected-(J1B-SYNC-Padb12)
- J1 pad b13: /R~{W} -> unconnected-(J1B-VPB-Padb13)
- J1 pad b14: /~{VALID} -> unconnected-(J1B-MLB-Padb14)
- J1 pad b15: /~{RESET} -> unconnected-(J1B-VDA-Padb15)
- J1 pad b16: /~{IRQ} -> unconnected-(J1B-VPA-Padb16)
- J1 pad b22: unconnected-(J1B-~{BUSGNT1}-Padb22) -> /BD0
- J1 pad b23: unconnected-(J1B-BE-Padb23) -> /BD1
- J1 pad b24: unconnected-(J1B-SYNC-Padb24) -> /BD2
- J1 pad b25: unconnected-(J1B-VPB-Padb25) -> /BD3
- J1 pad b26: unconnected-(J1B-MLB-Padb26) -> /BD4
- J1 pad b27: unconnected-(J1B-VDA-Padb27) -> /BD5
- J1 pad b28: unconnected-(J1B-VPA-Padb28) -> /BD6
- J1 pad b29: unconnected-(J1B-RESERVED-Padb29) -> /BD7
- J1 pad b4: /BD0 -> /~{VALID}
- J1 pad b5: /BD1 -> /PHI2
- J1 pad b6: /BD2 -> /R~{W}
- J1 pad b7: /BD3 -> /~{RESET}
- J1 pad b8: /BD4 -> /~{IRQ}
- J1 pad b9: /BD5 -> unconnected-(J1B-~{NMI}-Padb9)
- J1 pad c6: GND -> unconnected-(J1C-GND-Padc6)
- J3 pad 2: /TXD -> /RXD
- J3 pad 3: /RXD -> /TXD
- R1 pad 1: /~{RTS} -> /PB0
- R1 pad 2: Net-(D1-KA) -> Net-(RN3A-R1.2)
- R2 pad 1: /~{DTR} -> /PB1
- R2 pad 2: Net-(D2-KA) -> Net-(RN3B-R2.2)
- R3 pad 1: /TXD -> /PB2
- R3 pad 2: Net-(D3-KA) -> Net-(RN3C-R3.2)
- R4 pad 1: /~{DSR} -> /PB3
- R4 pad 2: Net-(D4-AK) -> Net-(RN3D-R4.2)
- R5 pad 1: /~{DCD} -> /PB4
- R5 pad 2: Net-(D5-AK) -> Net-(RN3E-R5.2)
- R6 pad 1: /RXD -> /PB5
- R6 pad 2: Net-(D6-AK) -> Net-(RN3F-R6.2)
- R7 pad 1: /~{CTS} -> /PB6
- R7 pad 2: Net-(D7-AK) -> Net-(RN3G-R7.2)
- R8 pad 1: +5V -> /PB7
- R8 pad 2: Net-(D8-A) (its old number) -> Net-(RN3H-R8.2)
- SW2 pad 3: /PB0 -> Net-(RN3A-R1.2)
- SW3 pad 3: /PB1 -> Net-(RN3B-R2.2)
- SW4 pad 3: /PB2 -> Net-(RN3C-R3.2)
- SW5 pad 3: /PB3 -> Net-(RN3D-R4.2)
- SW6 pad 3: /PB4 -> Net-(RN3E-R5.2)
- SW7 pad 3: /PB5 -> Net-(RN3F-R6.2)
- SW8 pad 3: /PB6 -> Net-(RN3G-R7.2)
- SW9 pad 3: /PB7 -> Net-(RN3H-R8.2)
- U10 pad 18: unconnected-(U6A-CB_{1}-Pad18) -> Net-(J2-Pin_3)
- U10 pad 19: unconnected-(U6A-CB_{2}-Pad19) -> Net-(J2-Pin_4)
- U10 pad 23: unconnected-(U6A-~{CS_{2}}-Pad23) -> /~{VIA_CS}
- U10 pad 24: unconnected-(U6A-CS_{1}-Pad24) -> +5V
- U10 pad 39: unconnected-(U6A-CA_{2}-Pad39) -> Net-(J2-Pin_2)
- U10 pad 40: unconnected-(U6A-CA_{1}-Pad40) -> Net-(J2-Pin_1)
- U12 pad 11: Net-(U7A-~{DTR}) -> Net-(D12-K)
- U12 pad 16: Net-(U7A-~{DCD}) -> Net-(D15-K)
- U12 pad 17: Net-(U7A-~{DSR}) -> Net-(D15-K)
- U12 pad 2: unconnected-(U7A-CS_{0}-Pad2) -> +5V
- U12 pad 3: unconnected-(U7A-~{CS_{1}}-Pad3) -> /~{ACIA_CS}
- U12 pad 8: Net-(U7A-~{RTS}) -> Net-(D13-K)
- U12 pad 9: Net-(U7A-~{CTS}) -> Net-(D17-K)
- U13 pad 1: /RXD -> /TXD
- U13 pad 10: /~{DSR} -> /~{RTS}
- U13 pad 11: Net-(U7A-~{CTS}) -> unconnected-(U13D-4Y-Pad11)
- U13 pad 13: /~{CTS} -> GND
- U13 pad 4: /~{DCD} -> /~{DTR}
- U13 pad 6: Net-(U7A-~{DCD}) -> Net-(D15-K)
- U13 pad 8: Net-(U7A-~{DSR}) -> Net-(D17-K)
- U2 pad 20: unconnected-(U4A-~{CS}-Pad20) -> /~{ROM_CS}
- U2 pad 22: /~{VALID} -> /~{OE}
- U4 pad 20: unconnected-(U5A-~{CS}-Pad20) -> /~{RAM_CS}
- U4 pad 22: /~{VALID} -> /~{OE}
- U4 pad 27: /R~{W} -> /~{RAM_WE}
- U6 pad 10: Net-(U7A-~{RTS}) -> Net-(D12-K)
- U6 pad 11: unconnected-(U8D-4Y-Pad11) -> /~{CTS}
- U6 pad 12: GND -> Net-(D13-K)
- U6 pad 13: GND -> Net-(D13-K)
- U6 pad 3: /TXD -> /RXD
- U6 pad 4: Net-(U7A-~{DTR}) -> Net-(D12-K)
- U6 pad 5: Net-(U7A-~{DTR}) -> Net-(D12-K)
- U6 pad 6: /~{DTR} -> /~{DSR}
- U6 pad 8: /~{RTS} -> /~{DCD}
- U6 pad 9: Net-(U7A-~{RTS}) -> Net-(D12-K)
- U7 pad 1: /~{VALID} -> GND
- U7 pad 19: /~{VALID} -> GND
- U8 pad 1: /~{VALID} -> GND
- U8 pad 19: /~{VALID} -> GND
- U9 pad 11: /D7 -> /BD7
- U9 pad 12: /D6 -> /BD6
- U9 pad 13: /D5 -> /BD5
- U9 pad 14: /D4 -> /BD4
- U9 pad 15: /D3 -> /BD3
- U9 pad 16: /D2 -> /BD2
- U9 pad 17: /D1 -> /BD1
- U9 pad 18: /D0 -> /BD0
- U9 pad 19: /~{VALID} -> Net-(U9A-~{OE})
- U9 pad 2: /BD0 -> /D0
- U9 pad 3: /BD1 -> /D1
- U9 pad 4: /BD2 -> /D2
- U9 pad 5: /BD3 -> /D3
- U9 pad 6: /BD4 -> /D4
- U9 pad 7: /BD5 -> /D5
- U9 pad 8: /BD6 -> /D6
- U9 pad 9: /BD7 -> /D7
Routing:
- net GND: track 27.7 -> 244.9 mm, vias 0 -> 2
- net +5V: track 27.7 -> 136.3 mm
- net /A5: track 27.7 -> 121.0 mm, vias 0 -> 1
- net /A7: track 27.7 -> 106.7 mm
- net /A4: track 27.7 -> 106.0 mm
- net /A3: track 54.2 -> 132.2 mm, vias 0 -> 2
- net /A2: track 54.2 -> 131.6 mm, vias 0 -> 2
- net /A1: track 54.2 -> 130.5 mm, vias 0 -> 2
- net /A0: track 54.2 -> 129.4 mm, vias 0 -> 2
- net /A9: track 27.7 -> 100.4 mm, vias 0 -> 1
- net /A8: track 27.7 -> 99.9 mm, vias 0 -> 1
- net -12V: track 0.00 -> 69.6 mm
- net +12V: track 0.00 -> 69.6 mm
- net /A10: track 27.7 -> 97.2 mm, vias 0 -> 1
- net /A13: track 27.7 -> 96.7 mm, vias 0 -> 1
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Other:
- board text added: "BRACKET 2.3mm"
- board text added: "PANEL 1.6MM"

Commit message: ben work; fixed logic issue with pwr; started lightman
Parts:
- U1: footprint FormantKO:DIP-14N -> IMNOTWOPR:DIP-14N
- U11: value 74HC688 -> 74HCT688
- U14: value 74HC138 -> 74HCT138
- moved U3 228.5 mm to (12.8, 26.4), turned to 90 degrees
- moved SW1 215.1 mm to (0.79, -19.3)
- moved RN1 204.8 mm to (28.7, -28.2)
- moved C7 175.8 mm to (-17.0, -8.51), turned to -90 degrees
- moved U5 167.7 mm to (-15.7, -21.8)
- moved U13 162.8 mm to (-3.66, 6.10)
- moved U6 162.8 mm to (-3.66, -9.14)
- moved SW9 129.4 mm to (-4.96, 23.8)
- moved U14 128.3 mm to (42.1, 11.2)
- moved C9 123.1 mm to (29.4, 11.2)
- moved C13 112.5 mm to (54.8, 17.5)
- moved C15 112.5 mm to (53.5, 34.0)
- moved D10 112.5 mm to (-33.9, 11.2)
- moved D11 112.5 mm to (-33.9, 26.4)
- moved D12 112.5 mm to (-33.9, 34.0)
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Connections:
- U1 pad 11: (no net) -> unconnected-(U1C-NC-Pad11)
- U1 pad 3: (no net) -> unconnected-(U1C-NC-Pad3)
Routing:
- net +12V: track 69.6 -> 214.9 mm, vias 0 -> 1
- net -12V: track 69.6 -> 210.9 mm, vias 0 -> 2
- net +5V: track 136.3 -> 267.8 mm, vias 0 -> 1
- net /PHI2: track 0.00 -> 95.0 mm, vias 0 -> 2
- net /R~{W}: track 0.00 -> 92.5 mm, vias 0 -> 2
- net /A6: track 52.3 -> 142.5 mm
- net /~{RESET}: track 0.00 -> 90.0 mm, vias 0 -> 2
- net /~{IRQ}: track 0.00 -> 84.9 mm, vias 0 -> 1
- net /~{VALID}: track 0.00 -> 84.9 mm, vias 0 -> 1
- net /A1: track 130.5 -> 214.5 mm, vias 2 -> 1
- net /A7: track 106.7 -> 174.8 mm, vias 0 -> 1
- net /D3: track 69.6 -> 135.2 mm, vias 2 -> 1
- net /A0: track 129.4 -> 192.6 mm, vias 2 -> 1
- net /A15: track 50.6 -> 107.2 mm
- net /A12: track 94.2 -> 150.7 mm
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