File: modules/BEN/BEN.kicad_sch (KiCad schematic)
At the start: 15 parts, among them J1 CardConnector, U1 74HCT541, U2 74HCT541, U3 74HCT245N, U4 28C256, U5 62256, U6 W65C22

Commit message: ben schematic wip
Parts:
- added C10, C11: 47u, IMNOTWOPR:CP_Radial_Tantal_P100mil, symbol IMNOTWOPR:C_Polarized
- added C12, C13, C14, C8, C9: 100n, IMNOTWOPR:C_Rect_P200mil, symbol IMNOTWOPR:C
- added D1, D2, D3: WP483SEKJ3CGKWT, LED_THT:LED_D5.0mm_FlatTop, symbol IMNOTWOPR:LED_Dual_Bidirectional
- added J2: DE9_Socket, Connector_Dsub:DSUB-9_Socket_Horizontal_P2.77x2.54mm_EdgePinOffset9.40mm, symbol Connector:DE9_Socket
- added J3: Conn_02x05_Odd_Even, Connector_IDC:IDC-Header_2x05_P2.54mm_Vertical, symbol Connector_Generic:Conn_02x05_Odd_Even
- added R1, R2, R3: 1k, IMNOTWOPR:R_Axial_DIN0207_P400mil, symbol IMNOTWOPR:R
- added U7: W65C51, IMNOTWOPR:DIP-28W, symbol IMNOTWOPR:W65C51
- added U8: MC1488, FormantKO:DIP-14N, symbol IMNOTWOPR:MC1488
- added U9: MC1489, FormantKO:DIP-14N, symbol IMNOTWOPR:MC1489
- C2, C3, C4, C5, C6, C7: value C -> 100n
- U1, U2: value 74HCT541 -> 74AHCT541; symbol IMNOTWOPR:74HCT541 -> IMNOTWOPR:74AHCT541
- U3: value 74HCT245N -> 74AHCT245; symbol IMNOTWOPR:74HCT245 -> IMNOTWOPR:74AHCT245
Connections:
- net +5V: now also U3.20 (VCC), C14.1, C8.1, C9.1, U7.15 (V_{DD}), U9.14 (V_{CC+})
- net D0: now also U3.18 (B0), U6.33 (D_{0}), U7.18 (D_{0})
- net D1: now also U3.17 (B1), U6.32 (D_{1}), U7.19 (D_{1})
- net D2: now also U3.16 (B2), U6.31 (D_{2}), U7.20 (D_{2})
- net D3: now also U3.15 (B3), U6.30 (D_{3}), U7.21 (D_{3})
- net D4: now also U3.14 (B4), U6.29 (D_{4}), U7.22 (D_{4})
- net D5: now also U3.13 (B5), U6.28 (D_{5}), U7.23 (D_{5})
- net D6: now also U3.12 (B6), U6.27 (D_{6}), U7.24 (D_{6})
- net D7: now also U3.11 (B7), U6.26 (D_{7}), U7.25 (D_{7})
- net GND: now also U3.10 (GND), C10.2, C11.1, C12.2, C13.1, C14.2, C8.2, C9.2, D1.2 (AK), D2.2 (AK), D3.2 (AK), J3.9 (Pin_9), U7.1 (V_{SS}), U8.12 (4A), U8.4B (13), U8.7 (GND), U9.7 (GND)
- net R~{W}: now reaches J1.b13 (R~{W})
- net R~{W}: now also U3.1 (A->B)
- net ~{VALID}: now reaches J1.b14 (~{VALID})
- net ~{VALID}: now also U1.1 (/OE1), U1.19 (/OE2), U2.1 (/OE1), U2.19 (/OE2), U3.19 (~{OE})
- net -12V: now reaches J1.b3 (-12V)
- net -12V: now also J1.b30 (-12V), C11.2, C13.2, U8.1 (V_{CC-})
- net +12V: now reaches J1.a3 (+12V)
- net +12V: now also J1.a30 (+12V), C10.1, C12.1, U8.14 (V_{CC+})
- net A7: now reaches U1.11 (Y7)
- net A7: now also U4.3 (A_{7}), U5.3 (A_{7})
- net A6: now reaches U1.12 (Y6)
- net A6: now also U4.4 (A_{6}), U5.4 (A_{6})
- net A5: now reaches U1.13 (Y5)
- net A5: now also U4.5 (A_{5}), U5.5 (A_{5})
- net A4: now reaches U1.14 (Y4)
- net A4: now also U4.6 (A_{4}), U5.6 (A_{4})
- net A3: now reaches U1.15 (Y3)
- net A3: now also U4.7 (A_{3}), U5.7 (A_{3})
- net A2: now reaches U1.16 (Y2)
- net A2: now also U4.8 (A_{2}), U5.8 (A_{2})
- net A1: now reaches U1.17 (Y1)
- net A1: now also U4.9 (A_{1}), U5.9 (A_{1})
- net A0: now reaches U1.18 (Y0)
- net A0: now also U4.10 (A_{0}), U5.10 (A_{0})
- net A15: now reaches U2.11 (Y7)
- net A14: now reaches U2.12 (Y6)
- net A14: now also U4.1 (A_{14}), U5.1 (A_{14})
- net A13: now reaches U2.13 (Y5)
- net A13: now also U4.26 (A_{13}), U5.26 (A_{13})
- net A12: now reaches U2.14 (Y4)
- net A12: now also U4.2 (A_{12}), U5.2 (A_{12})
- net A11: now reaches U2.15 (Y3)
- net A11: now also U4.23 (A_{11}), U5.23 (A_{11})
- net A10: now reaches U2.16 (Y2)
- net A10: now also U4.21 (A_{10}), U5.21 (A_{10})
- net A9: now reaches U2.17 (Y1)
- net A9: now also U4.24 (A_{9}), U5.24 (A_{9})
- net A8: now reaches U2.18 (Y0)
- net A8: now also U4.25 (A_{8}), U5.25 (A_{8})
- net PB0: now reaches U6.10 (PB_{0})
- net PB1: now reaches U6.11 (PB_{1})
- net PB2: now reaches U6.12 (PB_{2})
- net PB3: now reaches U6.13 (PB_{3})
- net PB4: now reaches U6.14 (PB_{4})
- net PB5: now reaches U6.15 (PB_{5})
- net PB6: now reaches U6.16 (PB_{6})
- net PB7: now reaches U6.17 (PB_{7})
- net PA0: now reaches U6.2 (PA_{0})
- net PA1: now reaches U6.3 (PA_{1})
- net PA2: now reaches U6.4 (PA_{2})
- net PA3: now reaches U6.5 (PA_{3})
- net PA4: now reaches U6.6 (PA_{4})
- net PA5: now reaches U6.7 (PA_{5})
- net PA6: now reaches U6.8 (PA_{6})
- net PA7: now reaches U6.9 (PA_{7})
- net SA0 renamed BA0
- net SA1 renamed BA1
- net SA10 renamed BA10
- net SA11 renamed BA11
- net SA12 renamed BA12
- net SA13 renamed BA13
- net SA14 renamed BA14
- net SA15 renamed BA15
- net SA2 renamed BA2
- net SA3 renamed BA3
- net SA4 renamed BA4
- net SA5 renamed BA5
- net SA6 renamed BA6
- net SA7 renamed BA7
- net SA8 renamed BA8
- net SA9 renamed BA9
- net SD_{0} renamed BD0
- net SD_{1} renamed BD1
- net SD_{2} renamed BD2
- net SD_{3} renamed BD3
- net SD_{4} renamed BD4
- net SD_{5} renamed BD5
- net SD_{6} renamed BD6
- net SD_{7} renamed BD7
- new net: J3.5 (Pin_5), R3.1, U8.3 (1Y)
- new net: D3.1 (KA), R3.2
- new net: J3.1 (Pin_1), U9.4 (2A)
- new net: J3.2 (Pin_2), U9.10 (3A)
- new net: J3.3 (Pin_3), U9.1 (1A)
- new net: J3.4 (Pin_4), R1.1, U8.3Y (8)
- new net: J3.6 (Pin_6), U9.13 (4A)
- new net: J3.7 (Pin_7), R2.1, U8.6 (2Y)
- new net: D1.1 (KA), R1.2
- new net: U7.11 (~{DTR}), U8.4 (2A), U8.5 (2B)
- new net: U7.17 (~{DSR}), U9.3Y (8)
- new net: U7.10 (TX_{D}), U8.2 (1A)
- new net: D2.1 (KA), R2.2
- new net: U7.16 (~{DCD}), U9.6 (2Y)
- new net: U7.12 (R_{X}D), U9.1Y (3)
- new net: U7.8 (~{RTS}), U8.3B (10), U8.9 (3A)
- new net: U7.9 (~{CTS}), U9.11 (4Y)
Other:
- moved on the sheet: C1, C2, C3, C4, C5, C6, C7, J1A, MH1

Commit message: lib work and ben wip
Parts:
- removed J2: DE9_Socket, Connector_Dsub:DSUB-9_Socket_Horizontal_P2.77x2.54mm_EdgePinOffset9.40mm, symbol Connector:DE9_Socket
- removed J3: Conn_02x05_Odd_Even, Connector_IDC:IDC-Header_2x05_P2.54mm_Vertical, symbol Connector_Generic:Conn_02x05_Odd_Even
- added C15, C16, C17, C18, C19, C20, C21, C22: 100n, IMNOTWOPR:C_Rect_P200mil, symbol IMNOTWOPR:C
- added D10, D11, D12, D13, D14, D15, D8, D9: LED_G, IMNOTWOPR:LED_G_D5.0mm, symbol IMNOTWOPR:LED_G
- added D16, D17: SB140, Diode_THT:D_DO-41_SOD81_P10.16mm_Horizontal, symbol Diode:SB140
- added D4, D5, D6, D7: WP483SEKJ3CGKWT, LED_THT:LED_D5.0mm_FlatTop, symbol IMNOTWOPR:LED_Dual_Bidirectional
- added J2: IDC DE9 Female, Connector_PinHeader_2.54mm:PinHeader_2x05_P2.54mm_Vertical, symbol IMNOTWOPR:DE-9_IDC_DCE
- added R10, R11, R12, R13, R14, R15, R4, R5, R6, R7, R8, R9: 1k, IMNOTWOPR:R_Axial_DIN0207_P400mil, symbol IMNOTWOPR:R
- added R16, R17, R18, R19, R20, R21, R22, R23: 10k, IMNOTWOPR:R_Axial_DIN0207_P400mil, symbol IMNOTWOPR:R
- added R24: 1M, IMNOTWOPR:R_Axial_DIN0207_P400mil, symbol IMNOTWOPR:R_Vertical
- added SW1, SW3, SW4, SW5, SW6, SW7, SW8, SW9: 2MS1T1B1M1QES, IMNOTWOPR:PanelConnector_1x03, symbol IMNOTWOPR:SW_SPST
- added SW2: SW_SPST, IMNOTWOPR:PanelConnector_1x03, symbol IMNOTWOPR:SW_SPST
- added Y1: 1.8432Mhz, Crystal:Crystal_HC49-U_Vertical, symbol Device:Crystal
Connections:
- net +5V: now also U4.27 (~{WE}), R10.1, R11.1, R12.1, R13.1, R14.1, R15.1, R16.1, R17.1, R18.1, R19.1, R20.1, R21.1, R22.1, R23.1, R8.1, R9.1
- net A0: now also U6.38 (RS_{0}), U7.13 (RS_{0})
- net A1: now also U6.37 (RS_{1}), U7.14 (RS_{1})
- net A2: now also U6.36 (RS_{2})
- net A3: now also U6.35 (RS_{3})
- net GND: now also U8.13 (4B), C15.2, C16.2, C17.2, C18.2, C19.2, C20.2, C21.2, C22.2, D4.1 (KA), D5.1 (KA), D6.1 (KA), D7.1 (KA), J2.5 (GND), SW1.2 (B), SW3.2 (B), SW4.2 (B), SW5.2 (B), SW6.2 (B), SW7.2 (B), SW8.2 (B), SW9.2 (B); no longer U8.4B (13)
- net PA0: now also D8.1 (K)
- net PA1: now also D9.1 (K)
- net PA2: now also D10.1 (K)
- net PA3: now also D11.1 (K)
- net PA4: now also D12.1 (K)
- net PA5: now also D13.1 (K)
- net PA6: now also D14.1 (K)
- net PA7: now also D15.1 (K)
- net PB0: now also C15.1, R16.2, SW1.3 (C)
- net PB1: now also C16.1, R17.2, SW3.3 (C)
- net PB2: now also C17.1, R18.2, SW4.3 (C)
- net PB3: now also C18.1, R19.2, SW5.3 (C)
- net PB4: now also C19.1, R20.2, SW6.3 (C)
- net PB5: now also C20.1, R21.2, SW7.3 (C)
- net PB6: now also C21.1, R22.2, SW8.3 (C)
- net PB7: now also C22.1, R23.2, SW9.3 (C)
- net R~{W}: now also U5.27 (~{WE}), U6.22 (~{RW}), U7.28 (~{RW})
- net ~{VALID}: now also U4.22 (~{OE}), U5.22 (~{OE})
- net PHI2: now reaches J1.b12 (Φ_{2})
- net PHI2: now also U6.25 (Φ_{2}), U7.27 (Φ_{2})
- net ~{RESET}: now reaches J1.b15 (~{RESET})
- net ~{RESET}: now also U6.34 (~{RESET}), U7.4 (~{RESET})
- net ~{IRQ}: now reaches J1.b16 (~{MIRQ})
- net ~{IRQ}: now also D16.2 (A), D17.2 (A)
- net TXD: now reaches R3.1, U8.3 (1Y)
- net TXD: now also J2.2 (TXD)
- net ~{DCD}: now reaches U9.4 (2A)
- net ~{DCD}: now also J2.1 (DCD), R5.1
- net ~{DSR}: now reaches U9.10 (3A)
- net ~{DSR}: now also J2.6 (DSR), R4.1
- net RXD: now reaches U9.1 (1A)
- net RXD: now also J2.3 (RXD), R6.1
- net ~{RTS}: now reaches R1.1
- net ~{RTS}: now also U8.8 (3Y), J2.7 (RTS); no longer U8.3Y (8)
- net ~{CTS}: now reaches U9.13 (4A)
- net ~{CTS}: now also J2.8 (CTS), R7.1
- net ~{DTR}: now reaches R2.1, U8.6 (2Y)
- net ~{DTR}: now also J2.4 (DTR)
- net at U7.17 (~{DSR}): now also U9.8 (3Y); no longer U9.3Y (8)
- net at U6.21 (~{IRQ}): now also D16.1 (K)
- net at U7.12 (R_{X}D): now also U9.3 (1Y); no longer U9.1Y (3)
- net at U7.8 (~{RTS}), U8.9 (3A): now also U8.10 (3B); no longer U8.3B (10)
- net at U7.26 (~{IRQ}): now also D17.1 (K)
- net at U7.6 (XTLI): now also R24.1, Y1.1
- net at U7.7 (XTLO): now also R24.2, Y1.2
- new net: D5.2 (AK), R5.2
- new net: D15.2 (A), R15.2
- new net: D13.2 (A), R13.2
- new net: D7.2 (AK), R7.2
- new net: D10.2 (A), R10.2
- new net: D8.2 (A), R8.2
- new net: D14.2 (A), R14.2
- new net: D6.2 (AK), R6.2
- new net: D4.2 (AK), R4.2
- new net: D12.2 (A), R12.2
- new net: D9.2 (A), R9.2
- new net: D11.2 (A), R11.2
- no-connect marks 56 -> 54
Other:
- note added: "DCE"
- moved on the sheet: C1, C10, C11, C12, C13, C14, C2, C3, C4, C5, C6, C7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

Commit message: ben schematic
Parts:
- removed D1, D2, D3, D4, D5, D6, D7: WP483SEKJ3CGKWT, LED_THT:LED_D5.0mm_FlatTop, symbol IMNOTWOPR:LED_Dual_Bidirectional
- removed R1, R10, R11, R12, R13, R14, R15, R2, R3, R4, R5, R6, R7, R8, R9: 1k, IMNOTWOPR:R_Axial_DIN0207_P400mil, symbol IMNOTWOPR:R
- removed R16, R17, R18, R19, R20, R21, R22, R23: 10k, IMNOTWOPR:R_Axial_DIN0207_P400mil, symbol IMNOTWOPR:R
- removed SW2: SW_SPST, IMNOTWOPR:PanelConnector_1x03, symbol IMNOTWOPR:SW_SPST
- added C15, C16, C17: 100n, IMNOTWOPR:C_Rect_P200mil, symbol IMNOTWOPR:C
- added C26: 30pF, IMNOTWOPR:C_Rect_P200mil, symbol IMNOTWOPR:C
- added D11, D12, D13, D14: LED_R, IMNOTWOPR:LED_D5.0mm_Horizontal_O1.27mm_Z3.0mm, symbol IMNOTWOPR:LED_R
- added D15, D16, D17, D18: LED_R, IMNOTWOPR:LED_D5.0mm_Horizontal_O3.81mm_Z9.0mm, symbol IMNOTWOPR:LED_R
- added J2: Conn_01x04, Connector_PinSocket_2.54mm:PinSocket_1x04_P2.54mm_Vertical, symbol Connector_Generic:Conn_01x04
- added R1, R2, R3, R4, R5, R6, R7, R8: 1k, IMNOTWOPR:R_Axial_DIN0207_P400mil, symbol IMNOTWOPR:R_Horizontal
- added RN1: 10kΩ, Resistor_THT:R_Array_SIP9, symbol Device:R_Network08_Split
- added RN2: 1k, Resistor_THT:R_Array_SIP9, symbol Device:R_Network08_Split
- added RN3: 10k, Resistor_THT:R_Array_SIP9, symbol Device:R_Network08_Split
- added RN4: 1k5, Resistor_THT:R_Array_SIP9, symbol Device:R_Network08_Split
- added SW1: PAGE SELECT, symbol Switch:SW_DIP_x08
- added U1: 74HCT13, FormantKO:DIP-14N, symbol 74xx:74LS13
- added U11: 74HC688, symbol 74xx:74HC688
- added U14: 74HC138, symbol 74xx:74HC138
- added U3: 74HCT32, IMNOTWOPR:DIP-14N, symbol IMNOTWOPR:74HCT32
- added U5: 74HCT00, IMNOTWOPR:DIP-14N, symbol IMNOTWOPR:74HCT00
- C1: Voltage 35V -> V
- C3: renamed from C10; Voltage 35V -> V
- C4: renamed from C11; Voltage 35V -> V
- D1: renamed from D16; value SB140 -> 1N5817
- D10: renamed from D13; footprint IMNOTWOPR:LED_G_D5.0mm -> IMNOTWOPR:LED_D5.0mm_Horizontal_O3.81mm_Z9.0mm
- D2: renamed from D8; footprint IMNOTWOPR:LED_G_D5.0mm -> IMNOTWOPR:LED_D5.0mm_Horizontal_O1.27mm_Z3.0mm
- D3: renamed from D9; footprint IMNOTWOPR:LED_G_D5.0mm -> IMNOTWOPR:LED_D5.0mm_Horizontal_O1.27mm_Z3.0mm
- D4: renamed from D10; footprint IMNOTWOPR:LED_G_D5.0mm -> IMNOTWOPR:LED_D5.0mm_Horizontal_O1.27mm_Z3.0mm
- D5: renamed from D11; footprint IMNOTWOPR:LED_G_D5.0mm -> IMNOTWOPR:LED_D5.0mm_Horizontal_O1.27mm_Z3.0mm
- D6: renamed from D17; value SB140 -> 1N5817
- D7: renamed from D14; footprint IMNOTWOPR:LED_G_D5.0mm -> IMNOTWOPR:LED_D5.0mm_Horizontal_O3.81mm_Z9.0mm
- D8: renamed from D15; footprint IMNOTWOPR:LED_G_D5.0mm -> IMNOTWOPR:LED_D5.0mm_Horizontal_O3.81mm_Z9.0mm
- D9: renamed from D12; footprint IMNOTWOPR:LED_G_D5.0mm -> IMNOTWOPR:LED_D5.0mm_Horizontal_O3.81mm_Z9.0mm
- U9: renamed from U3; value 74AHCT245 -> 74AHCT245_Slave; symbol IMNOTWOPR:74AHCT245 -> IMNOTWOPR:74AHCT245_Slave
- Y1: footprint Crystal:Crystal_HC49-U_Vertical -> (none)
- renumbered C6 to C10, C7 to C11, C8 to C12, C9 to C13, C15 to C18, C16 to C19, C17 to C20, C18 to C21, C19 to C22, C20 to C23, C21 to C24, C22 to C25, C3 to C5, C12 to C6, C13 to C7, C4 to C8, C5 to C9, J2 to J3, R24 to R9, SW1 to SW2, U6 to U10, U7 to U12, U9 to U13, U4 to U2, U5 to U4, U8 to U6, U1 to U7, U2 to U8
Connections:
- net +5V: now also U10.24 (CS_{1}), U12.2 (CS_{0}), C15.1, C16.1, C17.1, RN2.1 (R1), RN2.1 (R1), RN2.1 (R1), RN2.1 (R1), RN2.1 (R1), RN2.1 (R1), RN2.1 (R1), RN2.1 (R1), RN3.1 (R1), RN3.1 (R1), RN3.1 (R1), RN3.1 (R1), RN3.1 (R1), RN3.1 (R1), RN3.1 (R1), RN3.1 (R1), RN4.1 (R1), RN4.1 (R1), RN4.1 (R1), RN4.1 (R1), RN4.1 (R1), RN4.1 (R1), RN4.1 (R1), RN4.1 (R1), SW1.1, SW1.2, SW1.3, SW1.4, SW1.5, SW1.6, SW1.7, SW1.8, U1.14 (VCC), U11.20 (VCC), U14.16 (VCC), U3.14 (VCC), U5.14 (VCC)
- net A10: now also U11.14 (R5)
- net A11: now also U11.12 (R4)
- net A12: now also U11.9 (R3)
- net A13: now also U11.7 (R2)
- net A14: now also U11.5 (R1)
- net A15: now also U11.3 (R0), U5.1, U5.2, U5.9
- net A4: now also U14.1 (A0)
- net A5: now also U14.2 (A1)
- net A6: now also U14.3 (A2)
- net A7: now also U14.6 (E2)
- net A8: now also U11.18 (R7)
- net A9: now also U11.16 (R6)
- net BD0: now also J1.b22 (D_{0}), U9.18 (B0); no longer J1.b4 (D_{0}), U9.2 (A0)
- net BD1: now also J1.b23 (D_{1}), U9.17 (B1); no longer J1.b5 (D_{1}), U9.3 (A1)
- net BD2: now also J1.b24 (D_{2}), U9.16 (B2); no longer J1.b6 (D_{2}), U9.4 (A2)
- net BD3: now also J1.b25 (D_{3}), U9.15 (B3); no longer J1.b7 (D_{3}), U9.5 (A3)
- net BD4: now also J1.b26 (D_{4}), U9.14 (B4); no longer J1.b8 (D_{4}), U9.6 (A4)
- net BD5: now also J1.b27 (D_{5}), U9.13 (B5); no longer J1.b9 (D_{5}), U9.7 (A5)
- net BD6: now also J1.b28 (D_{6}), U9.12 (B6); no longer J1.b10 (D_{6}), U9.8 (A6)
- net BD7: now also J1.b29 (D_{7}), U9.11 (B7); no longer J1.b11 (D_{7}), U9.9 (A7)
- net D0: now also U9.2 (A0); no longer U9.18 (B0)
- net D1: now also U9.3 (A1); no longer U9.17 (B1)
- net D2: now also U9.4 (A2); no longer U9.16 (B2)
- net D3: now also U9.5 (A3); no longer U9.15 (B3)
- net D4: now also U9.6 (A4); no longer U9.14 (B4)
- net D5: now also U9.7 (A5); no longer U9.13 (B5)
- net D6: now also U9.8 (A6); no longer U9.12 (B6)
- net D7: now also U9.9 (A7); no longer U9.11 (B7)
- net GND: now also U13.13 (4A), U7.1 (~{OE1}), U7.19 (~{OE2}), U8.1 (~{OE1}), U8.19 (~{OE2}), C15.2, C16.2, C17.2, C26.2, RN1.1 (R1), RN1.1 (R1), RN1.1 (R1), RN1.1 (R1), RN1.1 (R1), RN1.1 (R1), RN1.1 (R1), RN1.1 (R1), U1.7 (GND), U11.1 (G), U11.10 (GND), U14.4 (~{E0}), U14.8 (GND), U3.12, U3.13, U3.7 (GND), U5.7 (GND); no longer J1.c6 (GND), U6.12 (4A), U6.13 (4B)
- net PB0: now also R1.1; no longer C18.1, SW2.3 (C)
- net PB1: now also R2.1; no longer C19.1, SW3.3 (C)
- net PB2: now also R3.1; no longer C20.1, SW4.3 (C)
- net PB3: now also R4.1; no longer C21.1, SW5.3 (C)
- net PB4: now also R5.1; no longer C22.1, SW6.3 (C)
- net PB5: now also R6.1; no longer C23.1, SW7.3 (C)
- net PB6: now also R7.1; no longer C24.1, SW8.3 (C)
- net PB7: now also R8.1; no longer C25.1, SW9.3 (C)
- net PHI2: now also J1.b5 (PHI2); no longer J1.b12 (Φ_{2})
- net RXD: now also J3.2 (RXD), U6.3 (1Y); no longer J3.3 (RXD), U13.1 (1A)
- net R~{W}: now also J1.b6 (R~{W}), U3.1, U5.12, U5.13; no longer J1.b13 (R~{W}), U4.27 (~{WE})
- net TXD: now also J3.3 (TXD), U13.1 (1A); no longer J3.2 (TXD), U6.3 (1Y)
- net ~{CTS}: now also U6.11 (4Y); no longer U13.13 (4A)
- net ~{DCD}: now also U6.8 (3Y); no longer U13.4 (2A)
- net ~{DSR}: now also U6.6 (2Y); no longer U13.10 (3A)
- net ~{DTR}: now also U13.4 (2A); no longer U6.6 (2Y)
- net ~{IRQ}: now also J1.b8 (~{IRQ}); no longer J1.b16 (~{MIRQ})
- net ~{RESET}: now also J1.b7 (~{RESET}); no longer J1.b15 (~{RESET})
- net ~{RTS}: now also U13.10 (3A); no longer U6.8 (3Y)
- net ~{VALID}: now also J1.b4 (~{VALID}), U3.10, U3.2, U3.4; no longer J1.b14 (~{VALID}), U2.22 (~{OE}), U4.22 (~{OE}), U7.1 (/OE1), U7.19 (/OE2), U8.1 (/OE1), U8.19 (/OE2), U9.19 (~{OE})
- net at D8.2 (A): now also RN2.9 (R8.2)
- net at D10.2 (A): now also RN2.7 (R6.2)
- net at D4.2 (A): now also RN2.4 (R3.2)
- net at D2.2 (A): now also RN2.2 (R1.2)
- net at D7.2 (A): now also RN2.8 (R7.2)
- net at U12.11 (~{DTR}), U6.4 (2A), U6.5 (2B): now also U6.10 (3B), U6.9 (3A), D12.1 (K)
- net at U12.17 (~{DSR}): now also U12.16 (~{DCD}), U13.6 (2Y), D15.1 (K), D16.1 (K); no longer U13.8 (3Y)
- net at U12.10 (TX_{D}), U6.2 (1A): now also D11.1 (K)
- net at R9.1, U12.6 (XTLI), Y1.1: now also C26.1
- net ~{ROM_CS}: now reaches U2.20 (~{CS})
- net ~{ROM_CS}: now also U1.2, U5.8
- net at U10.18 (CB_{1}): now also J2.3 (Pin_3)
- net at U10.19 (CB_{2}): now also J2.4 (Pin_4)
- net ~{VIA_CS}: now reaches U10.23 (~{CS_{2}})
- net ~{VIA_CS}: now also U1.4, U14.15 (~{Y0})
- net at U10.39 (CA_{2}): now also J2.2 (Pin_2)
- net at U10.40 (CA_{1}): now also J2.1 (Pin_1)
- net at D9.2 (A): now also RN2.6 (R5.2)
- net at D3.2 (A): now also RN2.3 (R2.2)
- net at D5.2 (A): now also RN2.5 (R4.2)
- net at U12.12 (R_{X}D), U13.3 (1Y): now also D14.1 (K)
- net at U12.9 (~{CTS}): now also U13.8 (3Y), D17.1 (K); no longer U13.11 (4Y)
- net ~{ACIA_CS}: now reaches U12.3 (~{CS_{1}})
- net ~{ACIA_CS}: now also U1.5, U14.14 (~{Y1})
- net ~{RAM_CS}: now reaches U4.20 (~{CS})
- net ~{RAM_CS}: now also U1.1, U5.6
- new net: RN1.4 (R3.2), SW1.14, U11.6 (P2)
- new net: C21.1, R4.2, RN3.5 (R4.2), SW5.3 (C)
- new net: RN1.6 (R5.2), SW1.12, U11.11 (P4)
- new net: D16.2 (A), RN4.7 (R6.2)
- new net: U3.5, U5.11
- new net: D13.1 (K), U12.8 (~{RTS}), U6.12 (4A), U6.13 (4B)
- new net: D13.2 (A), RN4.4 (R3.2)
- new net: C18.1, R1.2, RN3.2 (R1.2), SW2.3 (C)
- new net: D12.2 (A), RN4.3 (R2.2)
- new net: C23.1, R6.2, RN3.7 (R6.2), SW7.3 (C)
- new net: C22.1, R5.2, RN3.6 (R5.2), SW6.3 (C)
- new net: C24.1, R7.2, RN3.8 (R7.2), SW8.3 (C)
- new net: C25.1, R8.2, RN3.9 (R8.2), SW9.3 (C)
- new net: RN1.5 (R4.2), SW1.13, U11.8 (P3)
- new net: D14.2 (A), RN4.5 (R4.2)
- new net: C19.1, R2.2, RN3.3 (R2.2), SW3.3 (C)
- new net: RN1.7 (R6.2), SW1.11, U11.13 (P5)
- new net: C20.1, R3.2, RN3.4 (R3.2), SW4.3 (C)
- new net: D11.2 (A), RN4.2 (R1.2)
- new net: D17.2 (A), RN4.8 (R7.2)
- new net: RN1.2 (R1.2), SW1.16, U11.2 (P0)
- new net: D15.2 (A), RN4.6 (R5.2)
- new net: RN1.8 (R7.2), SW1.10, U11.15 (P6)
- new net: RN1.3 (R2.2), SW1.15, U11.4 (P1)
- new net: RN1.9 (R8.2), SW1.9, U11.17 (P7)
- new net: U5.3, U5.5
- new net: U3.8, U9.19 (~{OE})
- new net: D18.2 (A), RN4.9 (R8.2)
- new net LOCAL: U1.10, U1.12, U1.13, U1.6, U1.9
- new net ~{IO_SELECT}: U11.19 (P=R), U14.5 (~{E1}), U5.10, U5.4
- new net ~{LOCAL}: U1.8, U3.9
- new net ~{OE}: U2.22 (~{OE}), U3.6, U4.22 (~{OE})
- new net ~{RAM_WE}: U3.3, U4.27 (~{WE})
- no-connect marks 54 -> 64
Other:
- note added: "32K RAM EXCLUDING IO REGION"
- note added: "32K ROM"
- note added: "IO ADDRESS DECODING"
- note added: "RESERVED FOR FUTURE EXPANSION"
- moved on the sheet: C1, C10, C11, C12, C13, C14, C18, C19, C2, C20, C21, C22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

Commit message: ben work; fixed logic issue with pwr; started lightman
Parts:
- U1: footprint FormantKO:DIP-14N -> IMNOTWOPR:DIP-14N; symbol 74xx:74LS13 -> IMNOTWOPR:74HCT13; DigiKey (none) -> https://www.digikey.com/en/products/detail/texas-instrument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
- U11: value 74HC688 -> 74HCT688
- U14: value 74HC138 -> 74HCT138
Other:
- moved on the sheet: C17
