File: modules/SCC/SCC.kicad_sch (KiCad schematic)
At the start: 34 parts, among them J1 CardConnector, SW1 1MS2T1B1M1QES, SW2 1MS1T1B1M1QES, U1 74HCT14, U2 74HCT00, U3 555, U4 74HCT390, U5 74HCT390, U6 74HCT390

Commit message: migrated PWR to SCC; updates to MPU, more work pending
Parts:
- added C12, C13, C8: 100n, IMNOTWOPR:C_Rect_P200mil, symbol IMNOTWOPR:C
- added U7: 74AHCT541, IMNOTWOPR:DIP-20N, symbol IMNOTWOPR:74AHCT541
- added Y1: 1Mhz, Oscillator:Oscillator_DIP-14, symbol Oscillator:ACO-xxxMHz
- D1: value PWR OK -> LED_G; Legend (none) -> PWROK
- D3: value PWR STANDBY -> LED_R; Legend (none) -> PWRSTDBY
- D5: Legend (none) -> HEARTBEAT
- MES1: value +5V METER -> Voltmeter_DC; symbol Device:Voltmeter_DC -> IMNOTWOPR:Voltmeter_DC; Legend (none) -> +5V
- MES2: value +12V METER -> Voltmeter_DC; symbol Device:Voltmeter_DC -> IMNOTWOPR:Voltmeter_DC; Legend (none) -> +12V
- MES3: value -12V METER -> Voltmeter_DC; symbol Device:Voltmeter_DC -> IMNOTWOPR:Voltmeter_DC; Legend (none) -> -12V
- MES4: value IMNOTWOPR:Wire_Meter -> Voltmeter_DC; symbol Device:Voltmeter_DC -> IMNOTWOPR:Voltmeter_DC; Legend (none) -> +12V2
- SW1: Legend RESET -> MANUAL RESET
- renumbered C4 to C1, C9 to C10, C10 to C11, C5 to C2, C1 to C3, C6 to C4, C2 to C5, C7 to C6, C3 to C7, C8 to C9
Connections:
- net ~{RESET} is gone; now on net /RESET: J1.b15 (VDA)
- net +5V: now also C12.1, Y1.14 (Vcc)
- net +5VSB: now also C13.1, C8.1, U7.20 (VCC)
- net GND: now also C12.2, C13.2, C8.2, U7.1 (~{OE1}), U7.10 (GND), U7.19 (~{OE2}), Y1.7 (GND)
- net at U5.13 (Q0): now also U6.4 (~{CP1})
- net PHI2_B0: now reaches J1.b4 (~{VALID})
- net PHI2_B0: now also U7.18 (Y0)
- net CLOCK_BUF2 renamed PHI2_B1
- net PHI2_B1: now also U7.17 (Y1)
- net ~{PSON} renamed /PSON
- new net: U7.2 (A0), U7.3 (A1), U7.4 (A2), U7.5 (A3), U7.6 (A4), U7.7 (A5), U7.8 (A6), U7.9 (A7), Y1.8 (OUT)
- new net PHI2_B2: U7.16 (Y2)
- new net PHI2_B3: U7.15 (Y3)
- new net PHI2_B4: U7.14 (Y4)
- new net PHI2_B5: U7.13 (Y5)
- new net PHI2_B6: U7.12 (Y6)
- new net PHI2_B7: U7.11 (Y7)
- no-connect marks 88 -> 87
Other:
- note added: "PHI2_B2..PHI2_B7 CURRENTLY UNUSED"
- note added: "SYSTEM CLOCK"
- title: PWR -> SCC
- moved on the sheet: C1, C10, C11, C2, C3, C4, C5, C6, C7, C9, D1, D2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

Commit message: SCC module revision B
Parts:
- added C14, C16: 47µF, IMNOTWOPR:CP_Radial_Tantal_P100mil, symbol IMNOTWOPR:C_Polarized
- added C15, C17: 100n, IMNOTWOPR:C_Rect_P200mil, symbol IMNOTWOPR:C
- added unit 2 of U7
Connections:
- net +5V: now also C10.1, C11.1, C13.1, C9.1, U4.16 (VCC), U5.16 (VCC), U6.16 (VCC), C14.1, C15.1, C16.1, C17.1, U7.20 (VCC)
- net +5VSB: no longer C10.1, C11.1, C13.1, C9.1, U4.16 (VCC), U5.16 (VCC), U6.16 (VCC), U7.20 (VCC)
- net GND: now also C14.2, C15.2, C16.2, C17.2, U7.10 (GND); no longer U7.10 (GND)
Other:
- moved on the sheet: C1, C10, C11, C13, C2, C4, C6, C9, MES1, MES2, MES3, MES4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
