File: modules/SER-2/SER-2.kicad_sch (KiCad schematic)
At the start: 2 parts, among them J1 CardConnector

Commit message: work on ser-2 board. library cleanup
Parts:
- added C1, C2, C3: 47u, IMNOTWOPR:CP_Radial_Tantal_P100mil, symbol IMNOTWOPR:C_Polarized
- added C10, C11, C12, C13, C14, C15, C16, C17, C18, C4, C5, C6, C7, C8, C9: 100n, IMNOTWOPR:C_Rect_P200mil, symbol IMNOTWOPR:C
- added C19, C20: 20pf, IMNOTWOPR:C_Rect_P200mil, symbol IMNOTWOPR:C
- added D1, D13, D6, D8: LED_G, IMNOTWOPR:LED_D5.0mm_Horizontal_O1.27mm_Z3.0mm, symbol IMNOTWOPR:LED_G
- added D10, D14, D3, D7: LED_R, IMNOTWOPR:LED_D5.0mm_Horizontal_O1.27mm_Z3.0mm, symbol IMNOTWOPR:LED_R
- added D11, D12, D15, D16, D4, D5: LED_R, IMNOTWOPR:LED_D5.0mm_Horizontal_O3.81mm_Z9.0mm, symbol IMNOTWOPR:LED_R
- added D17, D18: 1N4148, FormantKO:DO-35_P400mil, symbol IMNOTWOPR:1N4148
- added D2, D9: LED_G, IMNOTWOPR:LED_D5.0mm_Horizontal_O3.81mm_Z9.0mm, symbol IMNOTWOPR:LED_G
- added J2, J3: DE-9 DTE, IMNOTWOPR:DE-9_IDC_2x05, symbol IMNOTWOPR:DE-9_IDC_DTE
- added R1, R10, R11, R12, R13, R14, R15, R2, R3, R4, R5, R6, R7, R9: 430R, IMNOTWOPR:R_Axial_DIN0207_P400mil, symbol IMNOTWOPR:R_Horizontal
- added R16, R8: 1M, IMNOTWOPR:R_Axial_DIN0207_P400mil, symbol IMNOTWOPR:R_Vertical
- added R17, R18: 680R, IMNOTWOPR:R_Axial_DIN0207_P400mil, symbol IMNOTWOPR:R_Vertical
- added RN1: 10kΩ, Resistor_THT:R_Array_SIP9, symbol Device:R_Network08_Split
- added SW1: PAGE SELECT, Button_Switch_THT:SW_DIP_SPSTx08_Slide_9.78x22.5mm_W7.62mm_P2.54mm, symbol Switch:SW_DIP_x08
- added U1, U3: MC1488, FormantKO:DIP-14N, symbol IMNOTWOPR:MC1488
- added U10: 74HCT688, IMNOTWOPR:DIP-20N, symbol IMNOTWOPR:74HCT688
- added U11, U12: MC1489, FormantKO:DIP-14N, symbol IMNOTWOPR:MC1489
- added U13: 74HCT138, IMNOTWOPR:DIP-16N, symbol IMNOTWOPR:74HCT138
- added U2, U4: 74AHCT541, IMNOTWOPR:DIP-20N, symbol IMNOTWOPR:74AHCT541
- added U5: 74HCT00, IMNOTWOPR:DIP-14N, symbol IMNOTWOPR:74HCT00
- added U6: 74HCT32, IMNOTWOPR:DIP-14N, symbol IMNOTWOPR:74HCT32
- added U7: 74AHCT245, IMNOTWOPR:DIP-20N, symbol IMNOTWOPR:74AHCT245_Slave
- added U8, U9: W65C51, IMNOTWOPR:DIP-28W, symbol IMNOTWOPR:W65C51
- added Y1, Y2: 1.8432Mhz, Crystal:Crystal_HC49-U_Vertical, symbol Device:Crystal
Connections:
- net +12V: now also C1.1, C4.1, C7.1, U1.14 (V_{CC+}), U3.14 (V_{CC+})
- net +5V: now also C10.1, C11.1, C12.1, C13.1, C14.1, C15.1, C16.1, C17.1, C18.1, C3.1, C6.1, C9.1, D1.2 (A), D10.2 (A), D11.2 (A), D12.2 (A), D2.2 (A), D3.2 (A), D4.2 (A), D5.2 (A), D8.2 (A), D9.2 (A), SW1.1, SW1.2, SW1.3, SW1.4, SW1.5, SW1.6, SW1.7, SW1.8, U10.20 (V_{CC}), U11.14 (V_{CC}), U12.14 (V_{CC}), U13.16 (V_{CC}), U2.20 (VCC), U4.20 (VCC), U5.14 (VCC), U6.14 (VCC), U7.20 (VCC), U8.15 (V_{DD}), U8.2 (CS_{0}), U9.15 (V_{DD}), U9.2 (CS_{0})
- net -12V: now also C2.2, C5.2, C8.2, U1.1 (V_{CC-}), U3.1 (V_{CC-})
- net GND: now also C1.2, C10.2, C11.2, C12.2, C13.2, C14.2, C15.2, C16.2, C17.2, C18.2, C19.2, C2.1, C20.2, C3.2, C4.2, C5.1, C6.2, C7.2, C8.1, C9.2, D13.1 (K), D14.1 (K), D6.1 (K), D7.1 (K), J2.5 (GND), J3.5 (GND), R17.1, R18.1, RN1.1 (R1), RN1.1 (R1), RN1.1 (R1), RN1.1 (R1), RN1.1 (R1), RN1.1 (R1), RN1.1 (R1), RN1.1 (R1), U1.2 (1A), U1.7 (GND), U10.1 (G), U10.10 (GND), U11.7 (GND), U12.7 (GND), U13.4 (G2A), U13.8 (GND), U2.1 (OE1), U2.10 (GND), U2.19 (OE1), U3.2 (1A), U3.7 (GND), U4.1 (OE1), U4.10 (GND), U4.19 (OE1), U5.10, U5.12, U5.13, U5.7 (GND), U5.9, U6.10, U6.12, U6.13, U6.4, U6.5, U6.7 (GND), U6.9, U7.10 (GND), U8.1 (V_{SS}), U9.1 (V_{SS})
- net SA0: now also U2.2 (A0)
- net SA1: now also U2.3 (A1)
- net SA10: now also U4.4 (A2)
- net SA11: now also U4.5 (A3)
- net SA12: now also U4.6 (A4)
- net SA13: now also U4.7 (A5)
- net SA14: now also U4.8 (A6)
- net SA15: now also U4.9 (A7)
- net SA2: now also U2.4 (A2)
- net SA3: now also U2.5 (A3)
- net SA4: now also U2.6 (A4)
- net SA5: now also U2.7 (A5)
- net SA6: now also U2.8 (A6)
- net SA7: now also U2.9 (A7)
- net SA8: now also U4.2 (A0)
- net SA9: now also U4.3 (A1)
- net SD0: now also U7.18 (B0)
- net SD1: now also U7.17 (B1)
- net SD2: now also U7.16 (B2)
- net SD3: now also U7.15 (B3)
- net SD4: now also U7.14 (B4)
- net SD5: now also U7.13 (B5)
- net SD6: now also U7.12 (B6)
- net SD7: now also U7.11 (B7)
- net ~{VALID}: now reaches J1.b4 (VALID)
- net ~{VALID}: now also U6.2
- net PHI2: now reaches J1.b5 (PHI2)
- net PHI2: now also U8.27 (Φ_{2}), U9.27 (Φ_{2})
- net R/W: now reaches J1.b6 (R/W)
- net R/W: now also U7.1 (A->B), U8.28 (R/W), U9.28 (R/W)
- net ~{RESET}: now reaches J1.b7 (RESET)
- net ~{RESET}: now also U8.4 (RESET), U9.4 (RESET)
- net ~{IRQ}: now reaches J1.b8 (IRQ)
- net ~{IRQ}: now also U8.26 (IRQ), U9.26 (IRQ)
- new net: D5.1 (K), R5.1
- new net: D12.1 (K), R13.1
- new net: R13.2, U12.11 (4Y), U9.9 (CTS)
- new net: D10.1 (K), R11.1
- new net: D4.1 (K), R4.1
- new net: J2.2 (R_{X}D), U11.4 (2A)
- new net: C19.1, R8.1, U8.6 (XTLI), Y1.1
- new net: R8.2, U8.7 (XTLO), Y1.2
- new net: RN1.7 (R6.2), SW1.11, U10.13 (P5)
- new net: D14.2 (A), R15.1
- new net: J2.3 (T_{X}D), U1.6 (2Y)
- new net: R14.2, U3.4 (2A), U3.5 (2B), U9.10 (T_{X}D)
- new net: R9.2, U3.10 (3B), U3.9 (3A), U9.11 (DTR)
- new net: R15.2, U12.6 (2Y), U9.12 (R_{X}D)
- new net: R11.2, U12.3 (1Y), U9.16 (DCD)
- new net: R12.2, U12.8 (3Y), U9.17 (DSR)
- new net: C20.1, R16.1, U9.6 (XTLI), Y2.1
- new net: R16.2, U9.7 (XTLO), Y2.2
- new net: R10.2, U3.12 (4A), U3.13 (4B), U9.8 (RTS)
- new net: D3.1 (K), R3.1
- new net: U5.6, U6.1
- new net: U6.3, U7.19 (~{OE})
- new net: D7.2 (A), R7.1
- new net: RN1.8 (R7.2), SW1.10, U10.15 (P6)
- new net: RN1.6 (R5.2), SW1.12, U10.11 (P4)
- new net: RN1.5 (R4.2), SW1.13, U10.8 (P3)
- new net: RN1.4 (R3.2), SW1.14, U10.6 (P2)
- new net: RN1.3 (R2.2), SW1.15, U10.4 (P1)
- new net: RN1.2 (R1.2), SW1.16, U10.2 (P0)
- new net: RN1.9 (R8.2), SW1.9, U10.17 (P7)
- new net: J2.7 (RTS), U1.11 (4Y)
- new net: D6.2 (A), R6.1
- new net: J3.1 (DCD), U12.1 (1A)
- new net: D15.2 (A), D17.1 (K), J2.9 (RI)
- new net: D15.1 (K), D17.2 (A), R17.2
- new net: J3.7 (RTS), U3.11 (4Y)
- new net: J3.3 (T_{X}D), U3.6 (2Y)
- new net: J3.2 (R_{X}D), U12.4 (2A)
- new net: D11.1 (K), R12.1
- new net: U5.3, U5.4, U5.5
- new net: J3.6 (DSR), U12.10 (3A)
- new net: D8.1 (K), R9.1
- new net: D1.1 (K), R1.1
- new net: J2.1 (DCD), U11.1 (1A)
- new net: D9.1 (K), R10.1
- new net: J3.4 (DTR), U3.8 (3Y)
- new net: J2.4 (DTR), U1.8 (3Y)
- new net: J2.6 (DSR), U11.10 (3A)
- new net: J2.8 (CTS), U11.13 (4A)
- new net: J3.8 (CTS), U12.13 (4A)
- new net: D16.2 (A), D18.1 (K), J3.9 (RI)
- new net: D16.1 (K), D18.2 (A), R18.2
- new net: D2.1 (K), R2.1
- new net: D13.2 (A), R14.1
- new net A0: U2.18 (Y0), U8.13 (RS_{0}), U9.13 (RS_{0})
- new net A1: U2.17 (Y1), U8.14 (RS_{1}), U9.14 (RS_{1})
- new net A10: U10.14 (R5), U4.16 (Y2)
- new net A11: U10.12 (R4), U4.15 (Y3)
- new net A12: U10.9 (R3), U4.14 (Y4)
- new net A13: U10.7 (R2), U4.13 (Y5)
- new net A14: U10.5 (R1), U4.12 (Y6)
- new net A15: U10.3 (R0), U4.11 (Y7)
- new net A2: U2.16 (Y2)
- new net A3: U2.15 (Y3)
- new net A4: U13.1 (A0), U2.14 (Y4)
- new net A5: U13.2 (A1), U2.13 (Y5)
- new net A6: U13.3 (A2), U2.12 (Y6)
- new net A7: U13.6 (G1), U2.11 (Y7)
- new net A8: U10.18 (R7), U4.18 (Y0)
- new net A9: U10.16 (R6), U4.17 (Y1)
- new net D0: U7.2 (A0), U8.18 (D_{0}), U9.18 (D_{0})
- new net D1: U7.3 (A1), U8.19 (D_{1}), U9.19 (D_{1})
- new net D2: U7.4 (A2), U8.20 (D_{2}), U9.20 (D_{2})
- new net D3: U7.5 (A3), U8.21 (D_{3}), U9.21 (D_{3})
- new net D4: U7.6 (A4), U8.22 (D_{4}), U9.22 (D_{4})
- new net D5: U7.7 (A5), U8.23 (D_{5}), U9.23 (D_{5})
- new net D6: U7.8 (A6), U8.24 (D_{6}), U9.24 (D_{6})
- new net D7: U7.9 (A7), U8.25 (D_{7}), U9.25 (D_{7})
- new net RXD_A_LED: R7.2, U11.6 (2Y), U8.12 (R_{X}D)
- new net TXD_A_LED: R6.2, U1.4 (2A), U1.5 (2B), U8.10 (T_{X}D)
- new net ~{ACIA_A_CS}: U13.15 (Y0), U5.1, U8.3 (CS_{1})
- new net ~{ACIA_B_CS}: U13.14 (Y1), U5.2, U9.3 (CS_{1})
- new net ~{CTS_A_LED}: R5.2, U11.11 (4Y), U8.9 (CTS)
- new net ~{DCD_A_LED}: R3.2, U11.3 (1Y), U8.16 (DCD)
- new net ~{DSR_A_LED}: R4.2, U11.8 (3Y), U8.17 (DSR)
- new net ~{DTR_A_LED}: R1.2, U1.10 (3B), U1.9 (3A), U8.11 (DTR)
- new net ~{PAGE_SELECT}: U10.19 (P=R), U13.5 (G2B)
- new net ~{RTS_A_LED}: R2.2, U1.12 (4A), U1.13 (4B), U8.8 (RTS)
- no-connect marks 53 -> 71
Other:
- note added: "FUTURE USE"
- note added: "ONLY ENABLE DATA BUS WHEN EITHER ACIA ARE ENABLED AND IF THE CURRENT CYCLE IS VALID"
- note added: "UNUSED GATES, DRIVERS, AND RECEIVERS"
- moved on the sheet: J1A, MH1
