File: modules/SER-2/system.kicad_sch (KiCad schematic)
At the start: 0 parts

Commit message: work on ser-2 board. library cleanup
Other:
- title: TITLE -> SER-2
Changed lines of the file:
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@@
 	(generator "eeschema")
 	(generator_version "10.0")
-	(paper "A3")
+	(paper "A2")
 	(title_block
-		(title "TITLE")
+		(title "SER-2")
 		(rev "A")
 		(company "THE HOUSE OF GALAHAD")
 		(comment 1 "IMNOTWOPR")
-		(comment 2 "DUAL SERIAL PORT")
-		(comment 3 "75-1000-01")
+		(comment 2 "DUAL SERIAL PORTS")
+		(comment 3 "75-1042-01")
 	)
 	(sheet_instances
