File: modules/CPU/CPU.kicad_pcb (KiCad board)
At the start: 2 copper layers, 160 x 100 mm, 27 parts, among them J1 SERIALA, J2 CardConnector, J3 Conn_02x10_Odd_Even, SW1 PAGE SELECT, U1 W65C02, U10 74AHCT541, U11 MC1488, U12 74HC138, U13 MC1489, U14 74HC688, U15 74HC20, U16 74AHCT541, U2 CY62256-70PC, U3 28C256, U4 W65C22, U5 W65C51, U7 74AHCT541, U8 74AHCT541, U9 74AHCT245, Y1 1Mhz, Y2 1.8432Mhz

Commit message: serial & cpu card
Parts:
- removed J3: Conn_02x10_Odd_Even, Connector_PinHeader_2.54mm:PinHeader_2x10_P2.54mm_Vertical
- removed SW1: PAGE SELECT, Button_Switch_THT:SW_DIP_SPSTx08_Slide_9.78x22.5mm_W7.62mm_P2.54mm
- removed U13: MC1489, IMNOTWOPR:DIP-14N
- removed U14: 74HC688, IMNOTWOPR:DIP-20N
- removed U15: 74HC20, IMNOTWOPR:DIP-14N
- removed U16: 74AHCT541, IMNOTWOPR:DIP-20N
- removed Y1: 1Mhz, Oscillator:Oscillator_DIP-14
- removed Y2: 1.8432Mhz, Crystal:Crystal_HC49-U_Vertical
- added C10: 100n, FormantKO:C_Rect_P200mil, F.Cu at (99.7, 95.0)
- added C2: 100n, FormantKO:C_Rect_P200mil, F.Cu at (195.7, 79.8)
- added C3: 100n, FormantKO:C_Rect_P200mil, F.Cu at (183.1, 82.9)
- added C4: 100n, FormantKO:C_Rect_P200mil, F.Cu at (183.0, 53.1)
- added C5: 100n, FormantKO:C_Rect_P200mil, F.Cu at (195.7, 50.5)
- added C7: 100n, FormantKO:C_Rect_P200mil, F.Cu at (102.3, 119.5)
- added C8: 100n, FormantKO:C_Rect_P200mil, F.Cu at (99.7, 87.5)
- added C9: 100n, FormantKO:C_Rect_P200mil, F.Cu at (99.7, 91.3)
- added R3: 10k, IMNOTWOPR:R_Axial_DIN0207_P400mil, F.Cu at (91.3, 83.7)
- added U6: 74HCT10, IMNOTWOPR:DIP-14N, F.Cu at (91.9, 123.6)
- C1: value 47µF -> 47u
- C6: value 20pF -> 100n; footprint IMNOTWOPR:C_Rect_P200mil -> FormantKO:C_Rect_P200mil
- J1: value SERIALA -> CardConnector; footprint IMNOTWOPR:DE-9_IDC_Header_Straight-Through -> IMNOTWOPR:SystemConector_Male
- J2: value CardConnector -> LOCAL RAM; footprint IMNOTWOPR:SystemConector_Male -> Connector_PinHeader_2.54mm:PinHeader_2x03_P2.54mm_Vertical
- R1: value 1MΩ -> 10k
- R2, RN1: value 10kΩ -> 10k
- U1: value W65C02 -> 74AHCT541; footprint IMNOTWOPR:DIP-40W -> IMNOTWOPR:DIP-20N
- U10: value 74AHCT541 -> 74HCT32; footprint IMNOTWOPR:DIP-20N -> IMNOTWOPR:DIP-14N
- U11: value MC1488 -> 62256; footprint IMNOTWOPR:DIP-14N -> IMNOTWOPR:DIP-28W
- U12: value 74HC138 -> 74HCT02; footprint IMNOTWOPR:DIP-16N -> IMNOTWOPR:DIP-14N
- U2: value CY62256-70PC -> 74AHCT541; footprint IMNOTWOPR:DIP-28W -> IMNOTWOPR:DIP-20N
- U3: value 28C256 -> 74AHCT245; footprint IMNOTWOPR:ZIF-28W -> IMNOTWOPR:DIP-20N
- U4: value W65C22 -> 74AHCT541; footprint IMNOTWOPR:DIP-40W -> IMNOTWOPR:DIP-20N
- U5: value W65C51 -> 74AHCT541; footprint IMNOTWOPR:DIP-28W -> IMNOTWOPR:DIP-20N
- U7: value 74AHCT541 -> W65C02; footprint IMNOTWOPR:DIP-20N -> IMNOTWOPR:DIP-40W
- U8: value 74AHCT541 -> 74HCT151; footprint IMNOTWOPR:DIP-20N -> IMNOTWOPR:DIP-16N
- U9: value 74AHCT245 -> 74HCT32; footprint IMNOTWOPR:DIP-20N -> IMNOTWOPR:DIP-14N
- moved U10 127.7 mm to (81.9, 64.1)
- moved J2 117.5 mm to (97.6, 99.2), turned to 0 degrees
- moved U4 111.8 mm to (195.7, 65.8), turned to 0 degrees
- moved U9 111.1 mm to (70.0, 64.1)
- moved U5 110.6 mm to (195.7, 93.7), turned to 0 degrees
- moved U8 104.4 mm to (89.5, 96.7)
- moved J1 98.5 mm to (215.0, 95.0)
- moved U1 86.4 mm to (170.3, 88.7), turned to 0 degrees
- moved R2 86.2 mm to (91.3, 79.7)
- moved U7 72.3 mm to (127.2, 92.5)
- moved U12 60.8 mm to (93.7, 64.1), turned to 0 degrees
- moved U3 49.6 mm to (183.0, 68.3), turned to 0 degrees
- moved RN1 45.6 mm to (88.1, 111.8)
- moved U11 45.5 mm to (73.8, 92.5), turned to 0 degrees
- moved R1 42.6 mm to (91.3, 75.8), turned to 0 degrees
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Connections:
- C6 pad 1: Net-(U5-XTLI) -> +5V
- R1 pad 1: Net-(U5-XTLO) -> Net-(J2-Pin_2)
- R1 pad 2: Net-(U5-XTLI) -> +5V
- R2 pad 1: +5V -> Net-(J2-Pin_4)
- R2 pad 2: Net-(U1-~{IRQ}) -> +5V
- RN1 pad 1: GND -> +5V
- RN1 pad 2: Net-(RN1A-R1.2) -> //RESET
- RN1 pad 3: Net-(RN1B-R2.2) -> //IRQ
- RN1 pad 4: Net-(RN1C-R3.2) -> //NMI
- RN1 pad 5: Net-(RN1D-R4.2) -> /READY
- RN1 pad 7: Net-(RN1F-R6.2) -> unconnected-(RN1F-R6.2-Pad7)
- RN1 pad 8: Net-(RN1G-R7.2) -> unconnected-(RN1G-R7.2-Pad8)
- RN1 pad 9: Net-(RN1H-R8.2) -> unconnected-(RN1H-R8.2-Pad9)
- U1 pad 1: VPB -> //CPU_GRANT
- U1 pad 10: /MPX/A1 -> GND
- U1 pad 11: /MPX/A2 -> unconnected-(U1A-Y7-Pad11)
- U1 pad 12: /MPX/A3 -> unconnected-(U1A-Y6-Pad12)
- U1 pad 13: /MPX/A4 -> unconnected-(U1A-Y5-Pad13)
- U1 pad 14: /MPX/A5 -> unconnected-(U1A-Y4-Pad14)
- U1 pad 15: /MPX/A6 -> unconnected-(U1A-Y3-Pad15)
- U1 pad 16: /MPX/A7 -> unconnected-(U1A-Y2-Pad16)
- U1 pad 17: /MPX/A8 -> unconnected-(U1A-Y1-Pad17)
- U1 pad 18: /MPX/A9 -> unconnected-(U1A-Y0-Pad18)
- U1 pad 19: /MPX/A10 -> //CPU_GRANT
- U1 pad 2: READY -> unconnected-(U1A-A0-Pad2)
- U1 pad 20: /MPX/A11 -> +5V
- U1 pad 3: PHI1O -> unconnected-(U1A-A1-Pad3)
- U1 pad 4: Net-(U1-~{IRQ}) -> unconnected-(U1A-A2-Pad4)
- U1 pad 5: MLB -> unconnected-(U1A-A3-Pad5)
- U1 pad 6: ~{NMI} -> unconnected-(U1A-A4-Pad6)
- U1 pad 7: SYNC -> unconnected-(U1A-A5-Pad7)
- U1 pad 8: +5V -> GND
- U1 pad 9: /MPX/A0 -> GND
- U10 pad 1: unconnected-(U10-G1-Pad1) -> /A14
- U10 pad 10: GND -> unconnected-(U10-Pad10)
- U10 pad 13: BMLB -> unconnected-(U10-Pad13)
- U10 pad 14: BVPB -> +5V
- U10 pad 2: PHI2 -> /A15
- U10 pad 3: R~{W} -> Net-(U8A-I5)
- U10 pad 4: VALID -> unconnected-(U10-Pad4)
- U10 pad 5: SYNC -> unconnected-(U10-Pad5)
- U10 pad 6: VPB -> unconnected-(U10-Pad6)
- U10 pad 7: MLB -> GND
- U10 pad 8: GND -> unconnected-(U10-Pad8)
- U10 pad 9: GND -> unconnected-(U10-Pad9)
- U11 pad 1: -12V -> /A14
- U11 pad 10: +5V -> /A0
- U11 pad 12: GND -> unconnected-(U11A-D_{1}-Pad12)
- U11 pad 13: GND -> unconnected-(U11A-D_{2}-Pad13)
- U11 pad 14: +12V -> unconnected-(U11B-GND-Pad14)
- U11 pad 2: /MPX/RTS -> /A12
- U11 pad 3: /MPX/RTS -> /A7
- U11 pad 4: /MPX/TXD -> /A6
- U11 pad 5: +5V -> /A5
- U11 pad 6: /MPX/TXD -> /A4
- U11 pad 7: GND -> /A3
- U11 pad 8: /MPX/DTR -> /A2
- U11 pad 9: /MPX/DTR -> /A1
- U12 pad 1: /MPX/A4 -> Net-(U11A-~{OE})
- U12 pad 14: ~{ACIA ENABLED} -> unconnected-(U12E-V_{CC}-Pad14)
- U12 pad 2: /MPX/A5 -> /R/W
- U12 pad 3: /MPX/A6 -> /PHI2
- U12 pad 4: Net-(U12-~{G2A}) -> unconnected-(U12-Pad4)
- U12 pad 5: /MPX/A7 -> unconnected-(U12-Pad5)
- U12 pad 6: +5V -> unconnected-(U12-Pad6)
- U12 pad 8: GND -> unconnected-(U12-Pad8)
- U2 pad 1: /MPX/A14 -> //VALID
- U2 pad 10: /MPX/A0 -> GND
- U2 pad 11: /MPX/D0 -> unconnected-(U2A-Y7-Pad11)
- U2 pad 12: /MPX/D1 -> unconnected-(U2A-Y6-Pad12)
- U2 pad 13: /MPX/D2 -> unconnected-(U2A-Y5-Pad13)
- U2 pad 14: GND -> unconnected-(U2A-Y4-Pad14)
- U2 pad 15: /MPX/D3 -> unconnected-(U2A-Y3-Pad15)
- U2 pad 16: /MPX/D4 -> unconnected-(U2A-Y2-Pad16)
- U2 pad 17: /MPX/D5 -> unconnected-(U2A-Y1-Pad17)
- U2 pad 18: /MPX/D6 -> unconnected-(U2A-Y0-Pad18)
- U2 pad 19: /MPX/D7 -> //VALID
- U2 pad 2: /MPX/A12 -> unconnected-(U2A-A0-Pad2)
- U2 pad 20: unconnected-(U2-~{CS}-Pad20) -> +5V
- U2 pad 3: /MPX/A7 -> unconnected-(U2A-A1-Pad3)
- U2 pad 4: /MPX/A6 -> unconnected-(U2A-A2-Pad4)
- U2 pad 5: /MPX/A5 -> unconnected-(U2A-A3-Pad5)
- U2 pad 6: /MPX/A4 -> unconnected-(U2A-A4-Pad6)
- U2 pad 7: /MPX/A3 -> GND
- U2 pad 8: /MPX/A2 -> GND
- U2 pad 9: /MPX/A1 -> GND
- U3 pad 1: /MPX/A14 -> unconnected-(U3A-A->B-Pad1)
- U3 pad 10: /MPX/A0 -> GND
- U3 pad 11: /MPX/D0 -> unconnected-(U3A-B7-Pad11)
- U3 pad 12: /MPX/D1 -> unconnected-(U3A-B6-Pad12)
- U3 pad 13: /MPX/D2 -> unconnected-(U3A-B5-Pad13)
- U3 pad 14: GND -> unconnected-(U3A-B4-Pad14)
- U3 pad 15: /MPX/D3 -> unconnected-(U3A-B3-Pad15)
- U3 pad 16: /MPX/D4 -> unconnected-(U3A-B2-Pad16)
- U3 pad 17: /MPX/D5 -> unconnected-(U3A-B1-Pad17)
- U3 pad 18: /MPX/D6 -> unconnected-(U3A-B0-Pad18)
- U3 pad 19: /MPX/D7 -> //VALID
- U3 pad 2: /MPX/A12 -> unconnected-(U3A-A0-Pad2)
- U3 pad 20: unconnected-(U3-~{CS}-Pad20) -> +5V
- U3 pad 3: /MPX/A7 -> unconnected-(U3A-A1-Pad3)
- U3 pad 4: /MPX/A6 -> unconnected-(U3A-A2-Pad4)
- U3 pad 5: /MPX/A5 -> unconnected-(U3A-A3-Pad5)
- U3 pad 6: /MPX/A4 -> unconnected-(U3A-A4-Pad6)
- U3 pad 7: /MPX/A3 -> unconnected-(U3A-A5-Pad7)
- U3 pad 8: /MPX/A2 -> unconnected-(U3A-A6-Pad8)
- U3 pad 9: /MPX/A1 -> unconnected-(U3A-A7-Pad9)
- U4 pad 1: GND -> unconnected-(U4A-OE1-Pad1)
- U4 pad 10: Net-(J3-Pin_2) -> GND
- U4 pad 11: Net-(J3-Pin_4) -> unconnected-(U4A-Y7-Pad11)
- U4 pad 12: Net-(J3-Pin_6) -> unconnected-(U4A-Y6-Pad12)
- U4 pad 13: Net-(J3-Pin_8) -> unconnected-(U4A-Y5-Pad13)
- U4 pad 14: Net-(J3-Pin_10) -> unconnected-(U4A-Y4-Pad14)
- U4 pad 15: Net-(J3-Pin_12) -> unconnected-(U4A-Y3-Pad15)
- U4 pad 16: Net-(J3-Pin_14) -> unconnected-(U4A-Y2-Pad16)
- U4 pad 17: Net-(J3-Pin_16) -> unconnected-(U4A-Y1-Pad17)
- U4 pad 18: Net-(J3-Pin_18) -> unconnected-(U4A-Y0-Pad18)
- U4 pad 19: Net-(J3-Pin_20) -> unconnected-(U4A-OE1-Pad19)
- U4 pad 2: Net-(J3-Pin_1) -> unconnected-(U4A-A0-Pad2)
- U4 pad 3: Net-(J3-Pin_3) -> unconnected-(U4A-A1-Pad3)
- U4 pad 4: Net-(J3-Pin_5) -> unconnected-(U4A-A2-Pad4)
- U4 pad 5: Net-(J3-Pin_7) -> unconnected-(U4A-A3-Pad5)
- U4 pad 6: Net-(J3-Pin_9) -> unconnected-(U4A-A4-Pad6)
- U4 pad 7: Net-(J3-Pin_11) -> unconnected-(U4A-A5-Pad7)
- U4 pad 8: Net-(J3-Pin_13) -> unconnected-(U4A-A6-Pad8)
- U4 pad 9: Net-(J3-Pin_15) -> unconnected-(U4A-A7-Pad9)
- U5 pad 1: GND -> unconnected-(U5A-OE1-Pad1)
- U5 pad 10: /MPX/TXD -> GND
- U5 pad 11: /MPX/DTR -> unconnected-(U5A-Y7-Pad11)
- U5 pad 12: /MPX/RXD -> unconnected-(U5A-Y6-Pad12)
- U5 pad 13: /MPX/A0 -> unconnected-(U5A-Y5-Pad13)
- U5 pad 14: /MPX/A1 -> unconnected-(U5A-Y4-Pad14)
- U5 pad 15: +5V -> unconnected-(U5A-Y3-Pad15)
- U5 pad 16: /MPX/DCD -> unconnected-(U5A-Y2-Pad16)
- U5 pad 17: /MPX/DSR -> unconnected-(U5A-Y1-Pad17)
- U5 pad 18: /MPX/D0 -> unconnected-(U5A-Y0-Pad18)
- U5 pad 19: /MPX/D1 -> unconnected-(U5A-OE1-Pad19)
- U5 pad 2: +5V -> unconnected-(U5A-A0-Pad2)
- U5 pad 20: /MPX/D2 -> +5V
- U5 pad 3: ~{ACIA ENABLED} -> unconnected-(U5A-A1-Pad3)
- U5 pad 6: Net-(U5-XTLI) -> unconnected-(U5A-A4-Pad6)
- U5 pad 7: Net-(U5-XTLO) -> unconnected-(U5A-A5-Pad7)
- U5 pad 8: /MPX/RTS -> unconnected-(U5A-A6-Pad8)
- U5 pad 9: /MPX/CTS -> unconnected-(U5A-A7-Pad9)
- U7 pad 10: GND -> unconnected-(U7-A_{1}-Pad10)
- U7 pad 11: BA7 -> unconnected-(U7-A_{2}-Pad11)
- U7 pad 12: BA6 -> unconnected-(U7-A_{3}-Pad12)
- U7 pad 13: BA5 -> unconnected-(U7-A_{4}-Pad13)
- U7 pad 14: BA4 -> unconnected-(U7-A_{5}-Pad14)
- U7 pad 15: BA3 -> unconnected-(U7-A_{6}-Pad15)
- U7 pad 16: BA2 -> unconnected-(U7-A_{7}-Pad16)
- U7 pad 17: BA1 -> unconnected-(U7-A_{8}-Pad17)
- U7 pad 18: BA0 -> unconnected-(U7-A_{9}-Pad18)
- U7 pad 2: /MPX/A0 -> unconnected-(U7-READY-Pad2)
- U7 pad 20: +5V -> unconnected-(U7-A_{11}-Pad20)
- U7 pad 3: /MPX/A1 -> unconnected-(U7-ϕ_{1}OUT-Pad3)
- U7 pad 4: /MPX/A2 -> unconnected-(U7-IRQ-Pad4)
- U7 pad 5: /MPX/A3 -> unconnected-(U7-MLB-Pad5)
- U7 pad 6: /MPX/A4 -> unconnected-(U7-NMI-Pad6)
- U7 pad 7: /MPX/A5 -> unconnected-(U7-SYNC-Pad7)
- U7 pad 8: /MPX/A6 -> +5V
- U7 pad 9: /MPX/A7 -> unconnected-(U7-A_{0}-Pad9)
- U8 pad 1: unconnected-(U8-G1-Pad1) -> Net-(U8A-I3)
- U8 pad 10: GND -> Net-(J2-Pin_3)
- U8 pad 11: BA15 -> Net-(J2-Pin_1)
- U8 pad 12: BA14 -> GND
- U8 pad 13: BA13 -> /A15
- U8 pad 14: BA12 -> Net-(U8A-I5)
- U8 pad 15: BA11 -> Net-(U8A-I4)
- U8 pad 16: BA10 -> +5V
- U8 pad 2: /MPX/A8 -> Net-(U8A-I2)
- U8 pad 3: /MPX/A9 -> Net-(U8A-I1)
- U8 pad 4: /MPX/A10 -> +5V
- U8 pad 5: /MPX/A11 -> /LOCAL_RAM
- U8 pad 6: /MPX/A12 -> //LOCAL_RAM
- U8 pad 7: /MPX/A13 -> GND
- U8 pad 8: /MPX/A14 -> GND
- U8 pad 9: /MPX/A15 -> Net-(J2-Pin_5)
- U9 pad 1: unconnected-(U9-A->B-Pad1) -> /A10
- U9 pad 10: GND -> Net-(U8A-I4)
- U9 pad 11: BD7 -> Net-(U8A-I4)
- U9 pad 12: BD6 -> /A13
- U9 pad 13: BD5 -> Net-(U8A-I5)
- U9 pad 14: BD4 -> +5V
- U9 pad 2: /MPX/D0 -> Net-(U8A-I2)
- U9 pad 3: /MPX/D1 -> Net-(U8A-I1)
- U9 pad 4: /MPX/D2 -> /A11
- U9 pad 5: /MPX/D3 -> Net-(U8A-I3)
- U9 pad 6: /MPX/D4 -> Net-(U8A-I2)
- U9 pad 7: /MPX/D5 -> GND
- U9 pad 8: /MPX/D6 -> Net-(U8A-I3)
- U9 pad 9: /MPX/D7 -> /A12
Routing:
- net /MPX/D7: track 203.5 -> 0.00 mm
- net /MPX/D6: track 201.1 -> 0.00 mm
- net /MPX/D0: track 200.6 -> 0.00 mm
- net /MPX/D5: track 200.2 -> 0.00 mm
- net /MPX/D4: track 199.3 -> 0.00 mm
- net /MPX/D1: track 197.0 -> 0.00 mm
- net /MPX/A4: track 195.2 -> 0.00 mm, vias 3 -> 0
- net /MPX/D2: track 193.4 -> 0.00 mm
- net /MPX/A0: track 189.3 -> 0.00 mm, vias 3 -> 0
- net /MPX/A5: track 188.4 -> 0.00 mm, vias 3 -> 0
- net /MPX/A1: track 187.0 -> 0.00 mm, vias 3 -> 0
- net /MPX/A6: track 181.6 -> 0.00 mm, vias 3 -> 0
- net /MPX/A7: track 174.0 -> 0.00 mm, vias 3 -> 0
- net /MPX/D3: track 171.0 -> 0.00 mm
- net /MPX/A2: track 159.3 -> 0.00 mm, vias 1 -> 0
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Other:
- board text added: "${COMPANY} - ${COMMENT1} - ${TITLE} - ${COMMENT2} - REVISION ${REVISION} ${CURRENT_DATE}"
- board text removed: "[ ${COMPANY} | ${COMMENT1} | ${COMMENT4} | ${TITLE} | ${COMMENT2} | REVISION ${REVISION} | ${CURRENT_DATE} ]"
