File: modules/PAR/PAR.kicad_sch (KiCad schematic)
At the start: 2 parts, among them J1 CardConnector

Commit message: par board & schematic wip
Parts:
- added C1: 47µ, IMNOTWOPR:CP_Radial_Tantal_P100mil, symbol IMNOTWOPR:C_Polarized
- added C10, C2, C3, C4, C5, C6, C7, C8, C9: 100n, IMNOTWOPR:C_Rect_P200mil, symbol IMNOTWOPR:C
- added D1, D2: SB140, Diode_THT:D_DO-41_SOD81_P10.16mm_Horizontal, symbol Diode:SB140
- added JP1: PORT1A, IMNOTWOPR:Jumper_1x03, symbol Jumper:Jumper_3_Bridged12
- added JP2: PORT2A, IMNOTWOPR:Jumper_1x03, symbol Jumper:Jumper_3_Bridged12
- added JP3: PORT2B, IMNOTWOPR:Jumper_1x03, symbol Jumper:Jumper_3_Bridged12
- added JP4: PORT1B, IMNOTWOPR:Jumper_1x03, symbol Jumper:Jumper_3_Bridged12
- added R1, R10, R11, R12, R13, R14, R15, R16, R17, R18, R19, R2, R20, R21, R22, R23, R24, R25, R26, R27, R28, R29, R3, R30, R31, R32, R33, R34, R35, R36, R37, R38, R39, R4, R40, R5, R6, R7, R8, R9: 100R, Resistor_THT:R_Axial_DIN0207_L6.3mm_D2.5mm_P2.54mm_Vertical, symbol IMNOTWOPR:R_Horizontal
- added RN1: 10k, Resistor_THT:R_Array_SIP9, symbol Device:R_Network08_Split
- added RN2, RN3, RN4, RN5: 10k, Resistor_THT:R_Array_SIP11, symbol Device:R_Network10
- added SW1: SW_DIP_x08, Button_Switch_THT:SW_DIP_SPSTx08_Slide_9.78x22.5mm_W7.62mm_P2.54mm, symbol Switch:SW_DIP_x08
- added U1, U6: W65C22, IMNOTWOPR:DIP-40W, symbol IMNOTWOPR:W65C22
- added U10, U11: DB-25 VIA, IMNOTWOPR:IDC-Header_2x13_DB-25, symbol IMNOTWOPR:DB-29_IDC_VIA
- added U2: 74HCT30, IMNOTWOPR:DIP-14N, symbol IMNOTWOPR:74HCT30
- added U3: 74HCT00, IMNOTWOPR:DIP-14N, symbol IMNOTWOPR:74HCT00
- added U4, U5: 74AHCT541, IMNOTWOPR:DIP-20N, symbol IMNOTWOPR:74AHCT541
- added U7: 74AHCT245, IMNOTWOPR:DIP-20N, symbol IMNOTWOPR:74AHCT245_Slave
- added U8: 74HCT688, IMNOTWOPR:DIP-20N, symbol IMNOTWOPR:74HCT688
- added U9: 74HCT138, IMNOTWOPR:DIP-16N, symbol IMNOTWOPR:74HCT138
Connections:
- net +5V: now also C1.1, C10.1, C2.1, C3.1, C4.1, C5.1, C6.1, C7.1, C8.1, C9.1, JP1.1 (A), JP2.1 (A), JP3.1 (A), JP4.1 (A), SW1.1, SW1.2, SW1.3, SW1.4, SW1.5, SW1.6, SW1.7, SW1.8, U1.20 (V_{DD}), U1.24 (CS_{1}), U2.14 (V_{CC}), U3.14 (V_{CC}), U4.20 (V_{CC}), U5.20 (V_{CC}), U6.20 (V_{DD}), U6.24 (CS_{1}), U7.20 (V_{CC}), U8.20 (V_{CC}), U9.16 (V_{CC})
- net GND: now also C1.2, C10.2, C2.2, C3.2, C4.2, C5.2, C6.2, C7.2, C8.2, C9.2, JP1.3 (B), JP2.3 (B), JP3.3 (B), JP4.3 (B), RN1.1 (R1), RN1.1 (R1), RN1.1 (R1), RN1.1 (R1), RN1.1 (R1), RN1.1 (R1), RN1.1 (R1), RN1.1 (R1), U1.1 (V_{SS}), U10.11 (GND), U10.12 (GND), U10.13 (GND), U10.24 (GND), U10.25 (GND), U11.11 (GND), U11.12 (GND), U11.13 (GND), U11.24 (GND), U11.25 (GND), U2.7 (GND), U3.10, U3.12, U3.13, U3.7 (GND), U3.9, U4.1 (OE_{1}), U4.10 (GND), U4.19 (OE_{2}), U5.1 (OE_{1}), U5.10 (GND), U5.19 (OE_{2}), U6.1 (V_{SS}), U7.10 (GND), U8.1 (G), U8.10 (GND), U9.4 (G2A), U9.8 (GND)
- net #VALID: now reaches J1.b4 (VALID)
- net #VALID: now also U3.1, U3.2
- net PHI2: now reaches J1.b5 (PHI2)
- net PHI2: now also U1.25 (Φ_{2}), U6.25 (Φ_{2})
- net R/W: now reaches J1.b6 (R/W)
- net R/W: now also U1.22 (R/W), U6.22 (R/W), U7.1 (A->B)
- net #RESET: now reaches J1.b7 (RESET)
- net #RESET: now also U1.34 (RESET), U6.34 (RESET)
- net #IRQ: now reaches J1.b8 (IRQ)
- net #IRQ: now also D1.2 (A), D2.2 (A)
- net +12V: no longer names the net of J1.a3 (+12V)
- net +12V: no longer J1.a30 (+12V)
- net -12V: no longer names the net of J1.b3 (-12V)
- net -12V: no longer J1.b30 (-12V)
- net SA0: no longer names the net of J1.a4 (A_{0})
- net SA0: now also U4.2 (A_{0})
- net SA1: no longer names the net of J1.a5 (A_{1})
- net SA1: now also U4.3 (A_{1})
- net SA10: no longer names the net of J1.a14 (A_{10})
- net SA10: now also U5.4 (A_{2})
- net SA11: no longer names the net of J1.a15 (A_{11})
- net SA11: now also U5.5 (A_{3})
- net SA12: no longer names the net of J1.a16 (A_{12})
- net SA12: now also U5.6 (A_{4})
- net SA13: no longer names the net of J1.a17 (A_{13})
- net SA13: now also U5.7 (A_{5})
- net SA14: no longer names the net of J1.a18 (A_{14})
- net SA14: now also U5.8 (A_{6})
- net SA15: no longer names the net of J1.a19 (A_{15})
- net SA15: now also U5.9 (A_{7})
- net SA2: no longer names the net of J1.a6 (A_{2})
- net SA2: now also U4.4 (A_{2})
- net SA3: no longer names the net of J1.a7 (A_{3})
- net SA3: now also U4.5 (A_{3})
- net SA4: no longer names the net of J1.a8 (A_{4})
- net SA4: now also U4.6 (A_{4})
- net SA5: no longer names the net of J1.a9 (A_{5})
- net SA5: now also U4.7 (A_{5})
- net SA6: no longer names the net of J1.a10 (A_{6})
- net SA6: now also U4.8 (A_{6})
- net SA7: no longer names the net of J1.a11 (A_{7})
- net SA7: now also U4.9 (A_{7})
- net SA8: no longer names the net of J1.a12 (A_{8})
- net SA8: now also U5.2 (A_{0})
- net SA9: no longer names the net of J1.a13 (A_{9})
- net SA9: now also U5.3 (A_{1})
- net SD0: no longer names the net of J1.b22 (D_{0})
- net SD0: now also U7.18 (B0)
- net SD1: no longer names the net of J1.b23 (D_{1})
- net SD1: now also U7.17 (B1)
- net SD2: no longer names the net of J1.b24 (D_{2})
- net SD2: now also U7.16 (B2)
- net SD3: no longer names the net of J1.b25 (D_{3})
- net SD3: now also U7.15 (B3)
- net SD4: no longer names the net of J1.b26 (D_{4})
- net SD4: now also U7.14 (B4)
- net SD5: no longer names the net of J1.b27 (D_{5})
- net SD5: now also U7.13 (B5)
- net SD6: no longer names the net of J1.b28 (D_{6})
- net SD6: now also U7.12 (B6)
- net SD7: no longer names the net of J1.b29 (D_{7})
- net SD7: now also U7.11 (B7)
- new net: JP2.2 (C), RN3.1 (common)
- new net: JP1.2 (C), RN2.1 (common)
- new net: R7.1, U10.7 (PA4)
- new net: R40.2, U10.23 (PB7)
- new net: R31.1, U10.14 (CB1)
- new net: R1.1, U10.1 (CA1)
- new net: R10.2, U10.10 (PA7)
- new net: R2.2, U10.2 (CA2)
- new net: R3.1, U10.3 (PA0)
- new net: R4.2, U10.4 (PA1)
- new net: R5.1, U10.5 (PA2)
- new net: R6.2, U10.6 (PA3)
- new net: R8.2, U10.8 (PA5)
- new net: R9.1, U10.9 (PA6)
- new net: RN1.8 (R7.2), SW1.10, U8.15 (P_{6})
- new net: R37.1, U10.20 (PB4)
- new net: RN1.7 (R6.2), SW1.11, U8.13 (P_{5})
- new net: R16.2, U11.6 (PA3)
- new net: RN1.6 (R5.2), SW1.12, U8.11 (P_{4})
- new net: RN1.5 (R4.2), SW1.13, U8.8 (P_{3})
- new net: RN1.4 (R3.2), SW1.14, U8.6 (P_{2})
- new net: RN1.3 (R2.2), SW1.15, U8.4 (P_{1})
- new net: RN1.2 (R1.2), SW1.16, U8.2 (P_{0})
- new net: RN1.9 (R8.2), SW1.9, U8.17 (P_{7})
- new net: R32.2, U10.15 (CB2)
- new net: R33.1, U10.16 (PB0)
- new net: R34.2, U10.17 (PB1)
- new net: R35.1, U10.18 (PB2)
- new net: R36.2, U10.19 (PB3)
- new net: R38.2, U10.21 (PB5)
- new net: R39.1, U10.22 (PB6)
- new net: JP3.2 (C), RN4.1 (common)
- new net: R25.1, U11.18 (PB2)
- new net: R17.1, U11.7 (PA4)
- new net: D2.1 (K), U1.21 (IRQ)
- new net: R27.1, U11.20 (PB4)
- new net: R29.1, U11.22 (PB6)
- new net: R26.2, U11.19 (PB3)
- new net: R12.2, U11.2 (CA2)
- new net: U2.8, U3.4
- new net: R20.2, U11.10 (PA7)
- new net: R13.1, U11.3 (PA0)
- new net: R19.1, U11.9 (PA6)
- new net: R18.2, U11.8 (PA5)
- new net: R11.1, U11.1 (CA1)
- new net: D1.1 (K), U6.21 (IRQ)
- new net: R14.2, U11.4 (PA1)
- new net: R15.1, U11.5 (PA2)
- new net: JP4.2 (C), RN5.1 (common)
- new net: R28.2, U11.21 (PB5)
- new net: R21.1, U11.14 (CB1)
- new net: R22.2, U11.15 (CB2)
- new net: R23.1, U11.16 (PB0)
- new net: R24.2, U11.17 (PB1)
- new net: R30.2, U11.23 (PB7)
- new net: U3.6, U7.19 (~{OE})
- new net: U3.3, U3.5
- new net #PAGE_SELECT: U8.19 (P=R), U9.5 (G2B)
- new net #VIA_1_CS: U2.1, U6.23 (CS_{2}), U9.15 (Y0)
- new net #VIA_2_CS: U1.23 (CS_{2}), U2.2, U9.14 (Y1)
- new net #VIA_3_CS: U2.3, U9.13 (Y2)
- new net #VIA_4_CS: U2.4, U9.12 (Y3)
- new net #VIA_5_CS: U2.5, U9.11 (Y4)
- new net #VIA_6_CS: U2.6, U9.10 (Y5)
- new net #VIA_7_CS: U2.11, U9.9 (Y6)
- new net #VIA_8_CS: U2.12, U9.7 (Y7)
- new net A0: U1.38 (RS_{0}), U4.18 (Y_{0}), U6.38 (RS_{0})
- new net A1: U1.37 (RS_{1}), U4.17 (Y_{1}), U6.37 (RS_{1})
- new net A10: U5.16 (Y_{2}), U8.14 (R_{5})
- new net A11: U5.15 (Y_{3}), U8.12 (R_{4})
- new net A12: U5.14 (Y_{4}), U8.9 (R_{3})
- new net A13: U5.13 (Y_{5}), U8.7 (R_{2})
- new net A14: U5.12 (Y_{6}), U8.5 (R_{1})
- new net A15: U5.11 (Y_{7}), U8.3 (R_{0})
- new net A2: U1.36 (RS_{2}), U4.16 (Y_{2}), U6.36 (RS_{2})
- new net A3: U1.35 (RS_{3}), U4.15 (Y_{3}), U6.35 (RS_{3})
- new net A4: U4.14 (Y_{4}), U9.1 (A0)
- new net A5: U4.13 (Y_{5}), U9.2 (A1)
- new net A6: U4.12 (Y_{6}), U9.3 (A2)
- new net A7: U4.11 (Y_{7}), U9.6 (G1)
- new net A8: U5.18 (Y_{0}), U8.18 (R_{7})
- new net A9: U5.17 (Y_{1}), U8.16 (R_{6})
- new net D0: U1.33 (D_{0}), U6.33 (D_{0}), U7.2 (A0)
- new net D1: U1.32 (D_{1}), U6.32 (D_{1}), U7.3 (A1)
- new net D2: U1.31 (D_{2}), U6.31 (D_{2}), U7.4 (A2)
- new net D3: U1.30 (D_{3}), U6.30 (D_{3}), U7.5 (A3)
- new net D4: U1.29 (D_{4}), U6.29 (D_{4}), U7.6 (A4)
- new net D5: U1.28 (D_{5}), U6.28 (D_{5}), U7.7 (A5)
- new net D6: U1.27 (D_{6}), U6.27 (D_{6}), U7.8 (A6)
- new net D7: U1.26 (D_{7}), U6.26 (D_{7}), U7.9 (A7)
- new net PORT1_CA1: R1.2, RN2.2 (R1), U6.40 (CA_{1})
- new net PORT1_CA2: R2.1, RN2.3 (R2), U6.39 (CA_{2})
- new net PORT1_CB1: R31.2, RN5.2 (R1), U6.18 (CB_{1})
- new net PORT1_CB2: R32.1, RN5.3 (R2), U6.19 (CB_{2})
- new net PORT1_PA0: R3.2, RN2.4 (R3), U6.2 (PA_{0})
- new net PORT1_PA1: R4.1, RN2.5 (R4), U6.3 (PA_{1})
- new net PORT1_PA2: R5.2, RN2.6 (R5), U6.4 (PA_{2})
- new net PORT1_PA3: R6.1, RN2.7 (R6), U6.5 (PA_{3})
- new net PORT1_PA4: R7.2, RN2.8 (R7), U6.6 (PA_{4})
- new net PORT1_PA5: R8.1, RN2.9 (R8), U6.7 (PA_{5})
- new net PORT1_PA6: R9.2, RN2.10 (R9), U6.8 (PA_{6})
- new net PORT1_PA7: R10.1, RN2.11 (R10), U6.9 (PA_{7})
- new net PORT1_PB0: R33.2, RN5.4 (R3), U6.10 (PB_{0})
- new net PORT1_PB1: R34.1, RN5.5 (R4), U6.11 (PB_{1})
- new net PORT1_PB2: R35.2, RN5.6 (R5), U6.12 (PB_{2})
- new net PORT1_PB3: R36.1, RN5.7 (R6), U6.13 (PB_{3})
- new net PORT1_PB4: R37.2, RN5.8 (R7), U6.14 (PB_{4})
- new net PORT1_PB5: R38.1, RN5.9 (R8), U6.15 (PB_{5})
- new net PORT1_PB6: R39.2, RN5.10 (R9), U6.16 (PB_{6})
- new net PORT1_PB7: R40.1, RN5.11 (R10), U6.17 (PB_{7})
- new net PORT2_CA1: R11.2, RN3.2 (R1), U1.40 (CA_{1})
- new net PORT2_CA2: R12.1, RN3.3 (R2), U1.39 (CA_{2})
- new net PORT2_CB1: R21.2, RN4.2 (R1), U1.18 (CB_{1})
- new net PORT2_CB2: R22.1, RN4.3 (R2), U1.19 (CB_{2})
- new net PORT2_PA0: R13.2, RN3.4 (R3), U1.2 (PA_{0})
- new net PORT2_PA1: R14.1, RN3.5 (R4), U1.3 (PA_{1})
- new net PORT2_PA2: R15.2, RN3.6 (R5), U1.4 (PA_{2})
- new net PORT2_PA3: R16.1, RN3.7 (R6), U1.5 (PA_{3})
- new net PORT2_PA4: R17.2, RN3.8 (R7), U1.6 (PA_{4})
- new net PORT2_PA5: R18.1, RN3.9 (R8), U1.7 (PA_{5})
- new net PORT2_PA6: R19.2, RN3.10 (R9), U1.8 (PA_{6})
- new net PORT2_PA7: R20.1, RN3.11 (R10), U1.9 (PA_{7})
- new net PORT2_PB0: R23.2, RN4.4 (R3), U1.10 (PB_{0})
- new net PORT2_PB1: R24.1, RN4.5 (R4), U1.11 (PB_{1})
- new net PORT2_PB2: R25.2, RN4.6 (R5), U1.12 (PB_{2})
- new net PORT2_PB3: R26.1, RN4.7 (R6), U1.13 (PB_{3})
- new net PORT2_PB4: R27.2, RN4.8 (R7), U1.14 (PB_{4})
- new net PORT2_PB5: R28.1, RN4.9 (R8), U1.15 (PB_{5})
- new net PORT2_PB6: R29.2, RN4.10 (R9), U1.16 (PB_{6})
- new net PORT2_PB7: R30.1, RN4.11 (R10), U1.17 (PB_{7})
- no-connect marks 53 -> 54
Other:
- note added: "ONLY ENABLE DATA BUS WHEN ANY VIA ARE ENABLED AND IF THE CURRENT CYCLE IS VALID"
- title: TITLE -> PAR
- moved on the sheet: MH1

Commit message: bus overhaul and par wip
Parts:
- renumbered JP2 to JP1, JP1 to JP2, R11 to R1, R20 to R10, R1 to R11, R2 to R12, R3 to R13, R4 to R14, R5 to R15, R6 to R16, R7 to R17, R8 to R18, R9 to R19, R12 to R2, R10 to R20, R13 to R3, R14 to R4, R15 to R5, R16 to R6, R17 to R7, R18 to R8, R19 to R9, RN3 to RN2, RN2 to RN3, U11 to U10, U10 to U11, U6 to U2, U2 to U3, U3 to U4, U4 to U5, U5 to U6
Connections:
- net #IRQ: now also J1.b24 (IRQ); no longer J1.b8 (IRQ)
- net #PAGE_SELECT: now also U9.4 (G2A); no longer U9.5 (G2B)
- net #RESET: now also J1.b12 (RESET); no longer J1.b7 (RESET)
- net #VALID: now also J1.b15 (VALID); no longer J1.b4 (VALID)
- net GND: now also U9.5 (G2B); no longer U9.4 (G2A)
- net PHI2: now also J1.b13 (PHI2); no longer J1.b5 (PHI2)
- net R/W: now also J1.b14 (R/W); no longer J1.b6 (R/W)
- net at J1.b10 (A_{6}): now also U5.8 (A_{6})
- net at J1.b11 (A_{7}): now also U5.9 (A_{7})
- net at J1.b16 (D_{0}): now also U7.18 (B0)
- net at J1.b17 (D_{1}): now also U7.17 (B1)
- net at J1.b18 (D_{2}): now also U7.16 (B2)
- net at J1.b19 (D_{3}): now also U7.15 (B3)
- net at J1.b20 (D_{4}): now also U7.14 (B4)
- net at J1.b21 (D_{5}): now also U7.13 (B5)
- net at J1.b22 (D_{6}): now also U7.12 (B6); no longer U7.18 (B0)
- net at J1.b23 (D_{7}): now also U7.11 (B7); no longer U7.17 (B1)
- net at J1.b25 (NMI): no longer U7.15 (B3)
- net at J1.b26 (IRQ_{0}): no longer U7.14 (B4)
- net at J1.b27 (IRQ_{1}): no longer U7.13 (B5)
- net at J1.b28 (IRQ_{2}): no longer U7.12 (B6)
- net at J1.b29 (IRQ_{3}): no longer U7.11 (B7)
- net at J1.b9 (A_{5}): now also U5.7 (A_{5})
- net at J1.a10 (A_{14}): now also U6.8 (A_{6}); no longer U5.8 (A_{6})
- net at J1.a11 (A_{15}): now also U6.9 (A_{7}); no longer U5.9 (A_{7})
- net at J1.a12 (A_{16}): no longer U6.2 (A_{0})
- net at J1.a13 (A_{17}): no longer U6.3 (A_{1})
- net at J1.a14 (A_{18}): no longer U6.4 (A_{2})
- net at J1.a15 (A_{19}): no longer U6.5 (A_{3})
- net at J1.a16 (A_{20}): no longer U6.6 (A_{4})
- net at J1.a17 (A_{21}): no longer U6.7 (A_{5})
- net at J1.a18 (A_{22}): no longer U6.8 (A_{6})
- net at J1.a19 (A_{23}): no longer U6.9 (A_{7})
- net at U5.2 (A_{0}): now also J1.b4 (A_{0}); no longer J1.a4 (A_{0})
- net at U5.3 (A_{1}): now also J1.b5 (A_{1}); no longer J1.a5 (A_{1})
- net at U5.4 (A_{2}): now also J1.b6 (A_{2}); no longer J1.a6 (A_{2})
- net at U5.5 (A_{3}): now also J1.b7 (A_{3}); no longer J1.a7 (A_{3})
- net at U5.6 (A_{4}): now also J1.b8 (A_{4}); no longer J1.a8 (A_{4})
- net at J1.a9 (A_{13}): now also U6.7 (A_{5}); no longer U5.7 (A_{5})
- new net: J1.a4 (A_{8}), U6.2 (A_{0})
- new net: J1.a5 (A_{9}), U6.3 (A_{1})
- new net: J1.a6 (A_{10}), U6.4 (A_{2})
- new net: J1.a7 (A_{11}), U6.5 (A_{3})
- new net: J1.a8 (A_{12}), U6.6 (A_{4})
Other:
- note added: "ONLY ENABLE DATA BUS WHEN ANY VIA ARE ENABLED AND THE CURRENT CYCLE IS VALID"
- note removed: "ONLY ENABLE DATA BUS WHEN ANY VIA ARE ENABLED AND IF THE CURRENT CYCLE IS VALID"
- moved on the sheet: C1, C10, C2, C3, C4, C5, C6, C7, C8, C9, D1, D2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
