File: panels/PXX/PXX.kicad_pcb (KiCad board)
At the start: 2 copper layers, 80.9 x 128.4 mm, 25 parts

Commit message: pxx panel
Parts:
- added REF**: Panel_Switch_2M, IMNOTWOPR:Panel_Switch_2M, F.Cu at (126.7, 57.7)
- added REF**: Panel_Switch_2M, IMNOTWOPR:Panel_Switch_2M, F.Cu at (86.7, 57.7)
