File: modules/CLK/CLK.kicad_sch (KiCad schematic)
At the start: 27 parts, among them J1 CardConnector, SW1 1MS2T1B1M1QES, U1 74HCT14, U2 74HCT390, U3 74HCT390, U4 74HCT390, U5 74AHCT541, U6 555, Y1 1Mhz

Commit message: lightman cleanup; more work pending
Parts:
- removed D2: 1N4148, FormantKO:DO-35_P400mil, symbol IMNOTWOPR:1N4148
- added Q1: 2N3904, IMNOTWOPR:TO-92_Wide, symbol Transistor_BJT:2N3904
- added R4: 10k, IMNOTWOPR:R_Axial_DIN0207_P400mil, symbol IMNOTWOPR:R_Horizontal
- added R5: 4k7, IMNOTWOPR:R_Axial_DIN0207_P400mil, symbol IMNOTWOPR:R_Vertical
- added R6: 100K, IMNOTWOPR:R_Axial_DIN0207_P400mil, symbol IMNOTWOPR:R_Vertical
- D3: Legend LEGEND -> HEARTBEAT
Connections:
- net #RESET: now also Q1.3 (C), R5.1
- net +5V: now also R5.2
- net GND: now also U1.5, Q1.1 (E), R6.1
- net at U6.3 (OUT): now also R4.1; no longer U1.5
- new net: Q1.2 (B), R4.2, R6.2
- no-connect marks 100 -> 101
Other:
- note added: "R5 is a 4k7 pull-up resistor located on a bus terminator card."
- moved on the sheet: MH1
