File: lightman/hardware/lightman.kicad_sch (KiCad schematic)
At the start: 1 part

Commit message: lightman source
Parts:
- added C1: 100µ, Capacitor_THT:CP_Radial_D6.3mm_P2.50mm, symbol Device:C_Polarized
- added C10, C11, C12, C3, C4, C5, C6, C7, C8, C9: 100n, IMNOTWOPR:C_Rect_P200mil, symbol IMNOTWOPR:C
- added C2: 22µ, Capacitor_THT:CP_Radial_D5.0mm_P2.50mm, symbol Device:C_Polarized
- added C30, C31: 100n, Desval27:C_Disc_D5.0mm_W2.5mm_P200mil, symbol Desval27:C
- added D2: 1N5822, Diode_THT:D_DO-201AD_P15.24mm_Horizontal, symbol Diode:1N5822
- added D3: LED, LED_THT:LED_D5.0mm, symbol Device:LED
- added J1: DE15_Socket_HighDensity_MountingHoles, Connector_Dsub:DSUB-15-HD_Socket_Horizontal_P2.29x2.54mm_EdgePinOffset8.35mm_Housed_MountingHolesOffset10.89mm, symbol Connector:DE15_Socket_HighDensity_MountingHoles
- added J2: Mini-DIN-6, IMNOTWOPR:KMDGX6SBS, symbol Connector:Mini-DIN-6
- added J4: DE9_Pins, Connector_Dsub:DSUB-9_Pins_Horizontal_P2.77x2.54mm_EdgePinOffset9.40mm, symbol Connector:DE9_Pins
- added J5: Barrel_Jack_Switch, Connector_BarrelJack:BarrelJack_Horizontal, symbol Connector:Barrel_Jack_Switch
- added R10, R11, R12, R13, R14, R15, R4, R5, R6, R7, R8, R9: 1k, IMNOTWOPR:R_Axial_DIN0207_P400mil, symbol IMNOTWOPR:R
- added R21: 470, Desval27:R_Axial_DIN0207_400mil, symbol Desval27:R
- added SW23: POWER, Button_Switch_THT:SW_E-Switch_EG2219_DPDT_Angled, symbol Switch:SW_Slide_DPDT
- added U1, U3: MAX3232, IMNOTWOPR:DIP-16N, symbol Interface_UART:MAX3232
- added U2: L7805, Package_TO_SOT_THT:TO-220-3_Horizontal_TabDown, symbol Regulator_Linear:L7805
- added U4: (no value), IMNOTWOPR:DIP-12W, symbol IMNOTWOPR:LevelShifter
- A1: footprint Module:RaspberryPi_Pico_Common_Unspecified -> Module:RaspberryPi_Pico_Common_THT
Connections:
- net GND: now also A1.33 (AGND), C1.2, C10.2, C11.2, C12.2, C2.2, C30.2, C31.2, C5.2, C6.2, C7.2, D3.1 (K), J1.10, J1.5, J1.6, J1.7, J1.8, J1.SH, J2.3, J4.5, SW23.1 (A), U1.15 (GND), U2.2 (GND), U3.15 (GND), U4.11 (GND), U4.2 (GND)
- net PICO_TXD: now reaches A1.1 (GPIO0)
- net PICO_TXD: now also U1.11 (T1IN)
- net KEY_DATA_LO: now reaches A1.10 (GPIO7)
- net KEY_DATA_LO: now also U4.9 (LV2)
- net PICO_RXD: now reaches A1.2 (GPIO1)
- net PICO_RXD: now also U1.12 (R1OUT)
- net HSYNC: now reaches A1.21 (GPIO16)
- net HSYNC: now also J1.13
- net VSYNC: now reaches A1.22 (GPIO17)
- net VSYNC: now also J1.14
- net at A1.24 (GPIO18): now also R4.1, R5.1, R6.1, R7.1
- net at A1.25 (GPIO19): now also R10.1, R11.1, R8.1, R9.1
- net at A1.26 (GPIO20): now also R12.1, R13.1, R14.1, R15.1
- net +3V3: now reaches A1.36 (3V3)
- net +3V3: now also C12.1, C7.1, U1.16 (VCC), U3.16 (VCC), U4.12 (+3V3)
- net PICO_CTS: now reaches A1.4 (GPIO2)
- net PICO_CTS: now also U1.9 (R2OUT)
- net +5V: now reaches A1.40 (VBUS)
- net +5V: now also C2.1, C30.1, J2.4, U2.3 (OUT), U4.1 (+5V)
- net PICO_RTS: now reaches A1.5 (GPIO3)
- net PICO_RTS: now also U1.10 (T2IN)
- net PICO_DTR: now reaches A1.6 (GPIO4)
- net PICO_DTR: now also U3.11 (T1IN)
- net PICO_DSR: now reaches A1.7 (GPIO5)
- net PICO_DSR: now also U3.9 (R2OUT)
- net KEY_CLOCK_LO: now reaches A1.9 (GPIO6)
- net KEY_CLOCK_LO: now also U4.10 (LV1)
- new net: D3.2 (A), R21.2
- new net: C10.1, U3.6 (VS-)
- new net: C8.1, U3.1 (C1+)
- new net: C11.1, U3.2 (VS+)
- new net: C8.2, U3.3 (C1-)
- new net: C9.1, U3.4 (C2+)
- new net: C9.2, U3.5 (C2-)
- new net: J5.2, SW23.2 (B)
- new net: D2.1 (K), SW23.5 (B)
- new net: D2.2 (A), J5.1
- new net: C6.1, U1.6 (VS-)
- new net: C3.1, U1.1 (C1+)
- new net: C3.2, U1.3 (C1-)
- new net: C4.1, U1.4 (C2+)
- new net: C4.2, U1.5 (C2-)
- new net: C5.1, U1.2 (VS+)
- new net +9V: C1.1, C31.1, R21.1, SW23.4 (A), U2.1 (IN)
- new net BLUE: J1.3, R12.2, R13.2, R14.2, R15.2
- new net CTS: J4.8, U1.8 (R2IN)
- new net DCD: J4.1, U3.13 (R1IN)
- new net DSR: J4.6, U3.8 (R2IN)
- new net DTR: J4.4, U3.14 (T1OUT)
- new net GREEN: J1.2, R10.2, R11.2, R8.2, R9.2
- new net KEY_CLOCK_HI: J2.5, U4.3 (HV1)
- new net KEY_DATA_HI: J2.1, U4.4 (HV2)
- new net RED: J1.1, R4.2, R5.2, R6.2, R7.2
- new net RTR: U3.7 (T2OUT)
- new net RTS: J4.7, U1.7 (T2OUT)
- new net RXD: J4.2, U1.13 (R1IN)
- new net TXD: J4.3, U1.14 (T1OUT)
- no-connect marks 0 -> 34
Other:
- note added: "*RTR NOT ON D-Sub 9 Pin*"
- moved on the sheet: A1

Commit message: lightman pcb
Parts:
- added C13, C14, C15, C16, C17: 100n, IMNOTWOPR:C_Rect_P200mil, symbol IMNOTWOPR:C
- added F1: Polyfuse, Fuse:Fuse_Bourns_MF-RG700, symbol Device:Polyfuse
- added U5: MAX3232, IMNOTWOPR:DIP-16N, symbol Interface_UART:MAX3232
- D3: footprint LED_THT:LED_D5.0mm -> LED_THT:LED_D5.0mm_Horizontal_O1.27mm_Z3.0mm
- R21: value 470 -> 1k
- U4: value (none) -> LEVEL SHIFTER
Connections:
- net +3V3: now also C17.1, U5.16 (VCC)
- net +5V: now also R21.1
- net +9V: no longer R21.1
- net DCD: now also U5.13 (R1IN); no longer U3.13 (R1IN)
- net DSR: now also U3.13 (R1IN); no longer U3.8 (R2IN)
- net GND: now also C15.2, C16.2, C17.2, U5.15 (GND)
- net KEY_CLOCK_LO: now also A1.11 (GPIO8); no longer A1.9 (GPIO6)
- net KEY_DATA_LO: now also A1.12 (GPIO9); no longer A1.10 (GPIO7)
- net PICO_DSR: now also U3.12 (R1OUT); no longer U3.9 (R2OUT)
- net at J5.1: now also F1.1; no longer D2.2 (A)
- net RI: now reaches J4.9
- net RI: now also U5.8 (R2IN)
- net RTR: no longer names the net of U3.7 (T2OUT)
- new net: C14.1, U5.4 (C2+)
- new net: C14.2, U5.5 (C2-)
- new net: C13.1, U5.1 (C1+)
- new net: C13.2, U5.3 (C1-)
- new net: C15.1, U5.6 (VS-)
- new net: D2.2 (A), F1.2
- new net: C16.1, U5.2 (VS+)
- new net PICO_DCD: A1.9 (GPIO6), U5.12 (R1OUT)
- new net PICO_RI: A1.10 (GPIO7), U5.9 (R2OUT)
- no-connect marks 34 -> 35
Other:
- note removed: "*RTR NOT ON D-Sub 9 Pin*"
- moved on the sheet: C1, C10, C11, C12, C2, C3, C30, C31, C4, C5, C6, C7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

Commit message: lightman pcb
Parts:
- removed R12, R13, R14, R15: 1k, IMNOTWOPR:R_Axial_DIN0207_P400mil, symbol IMNOTWOPR:R
- C1: renamed from C31; footprint Desval27:C_Disc_D5.0mm_W2.5mm_P200mil -> IMNOTWOPR:C_Rect_P200mil; symbol Desval27:C -> IMNOTWOPR:C
- C4: renamed from C30; footprint Desval27:C_Disc_D5.0mm_W2.5mm_P200mil -> IMNOTWOPR:C_Rect_P200mil; symbol Desval27:C -> IMNOTWOPR:C
- R1: renamed from R21; footprint Desval27:R_Axial_DIN0207_400mil -> IMNOTWOPR:R_Axial_DIN0207_P400mil; symbol Desval27:R -> IMNOTWOPR:R_Vertical
- R2: renamed from R4; value 1k -> 470R
- R4: renamed from R6; value 1k -> 2k2
- R5: renamed from R7; value 1k -> 470R
- R7: renamed from R9; value 1k -> 2k2
- R8: renamed from R10; value 1k -> 390R
- renumbered C14 to C10, C6 to C11, C10 to C12, C15 to C13, C5 to C14, C11 to C15, C7 to C17, C12 to C18, C17 to C19, C1 to C2, C2 to C3, C3 to C5, C8 to C6, C13 to C7, C4 to C8, D2 to D1, D3 to D2, J5 to J1, J1 to J3, R5 to R3, R8 to R6, R11 to R9, SW23 to SW1, U4 to U1, U1 to U3, U3 to U4
Connections:
- net BLUE: now also R8.2, R9.2
- net GREEN: now also R5.2; no longer R8.2, R9.2
- net HSYNC: now also A1.17 (GPIO13); no longer A1.21 (GPIO16)
- net PICO_CTS: now also A1.5 (GPIO3); no longer A1.4 (GPIO2)
- net PICO_DSR: now also A1.6 (GPIO4); no longer A1.7 (GPIO5)
- net PICO_DTR: now also A1.7 (GPIO5); no longer A1.6 (GPIO4)
- net PICO_RTS: now also A1.4 (GPIO2); no longer A1.5 (GPIO3)
- net PICO_RXD: now also A1.1 (GPIO0); no longer A1.2 (GPIO1)
- net PICO_TXD: now also A1.2 (GPIO1); no longer A1.1 (GPIO0)
- net RED: no longer R5.2
- net VSYNC: now also A1.19 (GPIO14); no longer A1.22 (GPIO17)
- net G2: now reaches A1.26 (GPIO20)
- net G2: now also R7.1
- net R0: now reaches A1.20 (GPIO15)
- net R0: now also R2.1
- net B0: now reaches A1.27 (GPIO21)
- net B0: now also R8.1
- net B1: now reaches A1.29 (GPIO22)
- net B1: now also R9.1
- new net G0: A1.24 (GPIO18), R5.1
- new net G1: A1.25 (GPIO19), R6.1
- new net R1: A1.21 (GPIO16), R3.1
- new net R2: A1.22 (GPIO17), R4.1
- no-connect marks 35 -> 32
Other:
- moved on the sheet: J4, R2, R3, R4, R5, R6, R7, R8, R9

Commit message: routing-first-stage
Parts:
- A1: symbol MCU_Module:RaspberryPi_Pico -> IMNOTWOPR:RaspberryPi_Pico
- SW1: symbol Switch:SW_Slide_DPDT -> IMNOTWOPR:SW_Slide_DPDT
Connections:
- net PICO_CTS: now also A1.4 (GPIO2); no longer A1.5 (GPIO3)
- net PICO_RTS: now also A1.5 (GPIO3); no longer A1.4 (GPIO2)
- net PICO_RXD: now also A1.2 (GPIO1); no longer A1.1 (GPIO0)
- net PICO_TXD: now also A1.1 (GPIO0); no longer A1.2 (GPIO1)
Changed lines of the file:
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@@
 		)
 	)
-	(label "PICO_CTS"
+	(label "PICO_RTS"
 		(at 36.83 60.96 180)
 		(effects
@@
 		)
 	)
-	(label "PICO_RXD"
+	(label "PICO_TXD"
 		(at 36.83 53.34 180)
 		(effects
@@
 		)
 	)
-	(label "PICO_TXD"
+	(label "PICO_RXD"
 		(at 36.83 55.88 180)
 		(effects
@@
 		)
 	)
-	(label "PICO_RTS"
+	(label "PICO_CTS"
 		(at 36.83 58.42 180)
 		(effects
@@
 	)
 	(symbol
-		(lib_id "MCU_Module:RaspberryPi_Pico")
+		(lib_id "IMNOTWOPR:RaspberryPi_Pico")
 		(at 59.69 68.58 0)
 		(unit 1)
@@
 	)
 	(symbol
-		(lib_id "Switch:SW_Slide_DPDT")
+		(lib_id "IMNOTWOPR:SW_Slide_DPDT")
 		(at 90.17 242.57 270)
 		(mirror x)

Commit message: tracework for lightman
Parts:
- J2: symbol Connector:Mini-DIN-6 -> IMNOTWOPR:Mini-DIN-6
Connections:
- net GND: now also J2.MH
Changed lines of the file:
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@@
 	)
 	(symbol
+		(lib_id "power:GND")
+		(at 63.5 143.51 0)
+		(unit 1)
+		(body_style 1)
+		(exclude_from_sim no)
+		(in_bom yes)
+		(on_board yes)
+		(in_pos_files yes)
+		(dnp no)
+		(property "Reference" "#PWR024"
+			(at 63.5 149.86 0)
+			(hide yes)
+			(show_name no)
+			(do_not_autoplace no)
+			(effects
+				(font
+					(size 1.27 1.27)
+				)
+			)
+		)
+		(property "Value" "GND"
+			(at 63.5 147.32 0)
+			(show_name no)
+			(do_not_autoplace no)
+			(effects
+				(font
+					(size 1.27 1.27)
+				)
+			)
+		)
+		(property "Footprint" ""
+			(at 63.5 143.51 0)
+			(hide yes)
+			(show_name no)
+			(do_not_autoplace no)
+			(effects
+				(font
+					(size 1.27 1.27)
+				)
+			)
+		)
+		(property "Datasheet" ""
+			(at 63.5 143.51 0)
+			(hide yes)
+			(show_name no)
+			(do_not_autoplace no)
+			(effects
+				(font
+					(size 1.27 1.27)
+				)
+			)
+		)
+		(property "Description" "Power symbol creates a global label with name \"GND\" , ground"
+			(at 63.5 143.51 0)
+			(hide yes)
+			(show_name no)
+			(do_not_autoplace no)
+			(effects
+				(font
+					(size 1.27 1.27)
+				)
+			)
+		)
+		(pin "1"
+		)
+		(instances
+			(project "lightman"
+				(path "/bc5ce1ee-80a9-4a0a-a79a-291efbccde4f"
+					(reference "#PWR024")
+					(unit 1)
+				)
+			)
+		)
+	)
+	(symbol
 		(lib_id "power:+3V3")
 		(at 64.77 30.48 0)
@@
 	)
 	(symbol
-		(lib_id "Connector:Mini-DIN-6")
+		(lib_id "IMNOTWOPR:Mini-DIN-6")
 		(at 63.5 135.89 0)
 		(unit 1)
@@
 		(pin "3"
 		)
+		(pin "MH"
+		)
 		(instances

Commit message: lightman cleanup; more work pending
Parts:
- C2: footprint Capacitor_THT:CP_Radial_D6.3mm_P2.50mm -> Capacitor_THT:CP_Radial_D10.0mm_P5.00mm
- C3: footprint Capacitor_THT:CP_Radial_D5.0mm_P2.50mm -> Capacitor_THT:CP_Radial_D10.0mm_P5.00mm
Connections:
- net +3V3: now also U1.3 (LV); no longer U1.12 (+3V3)
- net +5V: now also U1.10 (HV); no longer U1.1 (+5V)
- net GND: now also U1.4 (GND), U1.9 (GND); no longer U1.11 (GND), U1.2 (GND)
- net KEY_CLOCK_HI: now also U1.11 (HV2); no longer U1.3 (HV1)
- net KEY_CLOCK_LO: now also U1.2 (LV2); no longer U1.10 (LV1)
- net KEY_DATA_HI: now also U1.12 (HV1); no longer U1.4 (HV2)
- net KEY_DATA_LO: now also U1.1 (LV1); no longer U1.9 (LV2)
Changed lines of the file:
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@@
 	(wire
 		(pts
-			(xy 26.67 166.37) (xy 44.45 166.37)
-		)
-		(stroke
-			(width 0)
-			(type default)
-		)
-	)
-	(wire
-		(pts
 			(xy 264.16 121.92) (xy 273.05 121.92)
 		)
@@
 	(wire
 		(pts
-			(xy 64.77 163.83) (xy 67.31 163.83)
-		)
-		(stroke
-			(width 0)
-			(type default)
-		)
-	)
-	(wire
-		(pts
 			(xy 30.48 118.11) (xy 180.34 118.11)
 		)
@@
 	(wire
 		(pts
+			(xy 64.77 171.45) (xy 68.58 171.45)
+		)
+		(stroke
+			(width 0)
+			(type default)
+		)
+	)
+	(wire
+		(pts
 			(xy 119.38 60.96) (xy 119.38 63.5)
 		)
@@
 	(wire
 		(pts
+			(xy 64.77 168.91) (xy 81.28 168.91)
+		)
+		(stroke
+			(width 0)
+			(type default)
+		)
+	)
+	(wire
+		(pts
 			(xy 106.68 237.49) (xy 113.03 237.49)
 		)
@@
 	(wire
 		(pts
-			(xy 64.77 166.37) (xy 82.55 166.37)
+			(xy 25.4 168.91) (xy 44.45 168.91)
 		)
 		(stroke
@@
 	(wire
 		(pts
-			(xy 212.09 121.92) (xy 223.52 121.92)
+			(xy 39.37 171.45) (xy 44.45 171.45)
 		)
 		(stroke
@@
 	(wire
 		(pts
-			(xy 41.91 163.83) (xy 44.45 163.83)
+			(xy 212.09 121.92) (xy 223.52 121.92)
 		)
 		(stroke
@@
 	)
 	(label "KEY_DATA_LO"
-		(at 64.77 171.45 0)
+		(at 44.45 163.83 180)
 		(effects
 			(font
 				(size 1.27 1.27)
 			)
-			(justify left bottom)
+			(justify right bottom)
 		)
 	)
@@
 	)
 	(label "KEY_DATA_HI"
-		(at 44.45 171.45 180)
+		(at 64.77 163.83 0)
 		(effects
 			(font
 				(size 1.27 1.27)
 			)
-			(justify right bottom)
+			(justify left bottom)
 		)
 	)
@@
 	)
 	(label "KEY_CLOCK_LO"
-		(at 64.77 168.91 0)
+		(at 44.45 166.37 180)
 		(effects
 			(font
 				(size 1.27 1.27)
 			)
-			(justify left bottom)
+			(justify right bottom)
 		)
 	)
 	(label "KEY_CLOCK_HI"
-		(at 44.45 168.91 180)
+		(at 64.77 166.37 0)
 		(effects
 			(font
 				(size 1.27 1.27)
 			)
-			(justify right bottom)
+			(justify left bottom)
 		)
 	)
@@
 	(symbol
 		(lib_id "power:+3V3")
-		(at 67.31 163.83 0)
+		(at 25.4 168.91 0)
 		(unit 1)
 		(body_style 1)
@@
 		(dnp no)
 		(property "Reference" "#PWR07"
-			(at 67.31 167.64 0)
+			(at 25.4 172.72 0)
 			(hide yes)
 			(show_name no)
@@
 		)
 		(property "Value" "+3V3"
-			(at 67.31 160.274 0)
+			(at 25.4 165.354 0)
 			(show_name no)
 			(do_not_autoplace no)
@@
 		)
 		(property "Footprint" ""
-			(at 67.31 163.83 0)
+			(at 25.4 168.91 0)
 			(hide yes)
 			(show_name no)
@@
 		)
 		(property "Datasheet" ""
-			(at 67.31 163.83 0)
+			(at 25.4 168.91 0)
 			(hide yes)
 			(show_name no)
@@
 		)
 		(property "Description" "Power symbol creates a global label with name \"+3V3\""
-			(at 67.31 163.83 0)
+			(at 25.4 168.91 0)
 			(hide yes)
 			(show_name no)
@@
 	(symbol
 		(lib_id "power:GND")
-		(at 82.55 166.37 0)
+		(at 68.58 171.45 0)
 		(unit 1)
 		(body_style 1)
@@
 		(dnp no)
 		(property "Reference" "#PWR012"
-			(at 82.55 172.72 0)
+			(at 68.58 177.8 0)
 			(hide yes)
 			(show_name no)
@@
 		)
 		(property "Value" "GND"
-			(at 82.804 170.18 0)
+			(at 68.834 175.26 0)
 			(show_name no)
 			(do_not_autoplace no)
@@
 		)
 		(property "Footprint" ""
-			(at 82.55 166.37 0)
+			(at 68.58 171.45 0)
 			(hide yes)
 			(show_name no)
@@
 		)
 		(property "Datasheet" ""
-			(at 82.55 166.37 0)
+			(at 68.58 171.45 0)
 			(hide yes)
 			(show_name no)
@@
 		)
 		(property "Description" "Power symbol creates a global label with name \"GND\" , ground"
-			(at 82.55 166.37 0)
+			(at 68.58 171.45 0)
 			(hide yes)
 			(show_name no)
@@
 			)
 		)
-		(property "Footprint" "Capacitor_THT:CP_Radial_D6.3mm_P2.50mm"
+		(property "Footprint" "Capacitor_THT:CP_Radial_D10.0mm_P5.00mm"
 			(at 120.3452 247.65 0)
 			(hide yes)
@@
 	(symbol
 		(lib_id "power:+5V")
-		(at 41.91 163.83 0)
+		(at 81.28 168.91 0)
 		(unit 1)
 		(body_style 1)
@@
 		(dnp no)
 		(property "Reference" "#PWR03"
-			(at 41.91 167.64 0)
+			(at 81.28 172.72 0)
 			(hide yes)
 			(show_name no)
@@
 		)
 		(property "Value" "+5V"
-			(at 41.91 160.274 0)
+			(at 81.28 165.354 0)
 			(show_name no)
 			(do_not_autoplace no)
@@
 		)
 		(property "Footprint" ""
-			(at 41.91 163.83 0)
+			(at 81.28 168.91 0)
 			(hide yes)
 			(show_name no)
@@
 		)
 		(property "Datasheet" ""
-			(at 41.91 163.83 0)
+			(at 81.28 168.91 0)
 			(hide yes)
 			(show_name no)
@@
 		)
 		(property "Description" "Power symbol creates a global label with name \"+5V\""
-			(at 41.91 163.83 0)
+			(at 81.28 168.91 0)
 			(hide yes)
 			(show_name no)
@@
 	(symbol
 		(lib_id "power:GND")
-		(at 26.67 166.37 0)
+		(at 39.37 171.45 0)
 		(unit 1)
 		(body_style 1)
@@
 		(dnp no)
 		(property "Reference" "#PWR01"
-			(at 26.67 172.72 0)
+			(at 39.37 177.8 0)
 			(hide yes)
 			(show_name no)
@@
 		)
 		(property "Value" "GND"
-			(at 26.924 170.18 0)
+			(at 39.624 175.26 0)
 			(show_name no)
 			(do_not_autoplace no)
@@
 		)
 		(property "Footprint" ""
-			(at 26.67 166.37 0)
+			(at 39.37 171.45 0)
 			(hide yes)
 			(show_name no)
@@
 		)
 		(property "Datasheet" ""
-			(at 26.67 166.37 0)
+			(at 39.37 171.45 0)
 			(hide yes)
 			(show_name no)
@@
 		)
 		(property "Description" "Power symbol creates a global label with name \"GND\" , ground"
-			(at 26.67 166.37 0)
+			(at 39.37 171.45 0)
 			(hide yes)
 			(show_name no)
@@
 			)
 		)
-		(property "Footprint" "Capacitor_THT:CP_Radial_D5.0mm_P2.50mm"
+		(property "Footprint" "Capacitor_THT:CP_Radial_D10.0mm_P5.00mm"
 			(at 145.7452 247.65 0)
 			(hide yes)

Commit message: lightman pcb gerbers
Parts:
- J4: footprint Connector_Dsub:DSUB-9_Pins_Horizontal_P2.77x2.54mm_EdgePinOffset9.40mm -> IMNOTWOPR:D-Sub 9 CNR Series; symbol Connector:DE9_Pins -> IMNOTWOPR:DE9_Pins
Connections:
- net GND: now also J4.MH
Changed lines of the file:
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@@
 		(rev "A")
 		(company "THE HOUSE OF GALAHAD")
+		(comment 1 "IMNOTWOPR")
+		(comment 2 "VGA SERIAL TERMINAL")
+		(comment 3 "75-1201-01")
 	)
 	(junction
@@
 	)
 	(symbol
-		(lib_id "Connector:DE9_Pins")
+		(lib_id "IMNOTWOPR:DE9_Pins")
 		(at 354.33 142.24 0)
 		(unit 1)
@@
 			)
 		)
-		(property "Footprint" "Connector_Dsub:DSUB-9_Pins_Horizontal_P2.77x2.54mm_EdgePinOffset9.40mm"
+		(property "Footprint" "IMNOTWOPR:D-Sub 9 CNR Series"
 			(at 354.33 142.24 0)
 			(hide yes)
@@
 		(pin "6"
 		)
+		(pin "MH"
+		)
 		(instances
 			(project "lightman"
@@
 					(unit 1)
 				)
+			)
+		)
+	)
+	(symbol
+		(lib_id "power:GND")
+		(at 354.33 158.75 0)
+		(unit 1)
+		(body_style 1)
+		(exclude_from_sim no)
+		(in_bom yes)
+		(on_board yes)
+		(in_pos_files yes)
+		(dnp no)
+		(property "Reference" "#PWR025"
+			(at 354.33 165.1 0)
+			(hide yes)
+			(show_name no)
+			(do_not_autoplace no)
+			(effects
+				(font
+					(size 1.27 1.27)
+				)
+			)
+		)
+		(property "Value" "GND"
+			(at 354.33 162.56 0)
+			(show_name no)
+			(do_not_autoplace no)
+			(effects
+				(font
+					(size 1.27 1.27)
+				)
+			)
+		)
+		(property "Footprint" ""
+			(at 354.33 158.75 0)
+			(hide yes)
+			(show_name no)
+			(do_not_autoplace no)
+			(effects
+				(font
+					(size 1.27 1.27)
+				)
+			)
+		)
+		(property "Datasheet" ""
+			(at 354.33 158.75 0)
+			(hide yes)
+			(show_name no)
+			(do_not_autoplace no)
+			(effects
+				(font
+					(size 1.27 1.27)
+				)
+			)
+		)
+		(property "Description" "Power symbol creates a global label with name \"GND\" , ground"
+			(at 354.33 158.75 0)
+			(hide yes)
+			(show_name no)
+			(do_not_autoplace no)
+			(effects
+				(font
+					(size 1.27 1.27)
+				)
+			)
+		)
+		(pin "1"
+		)
+		(instances
+			(project "lightman"
+				(path "/bc5ce1ee-80a9-4a0a-a79a-291efbccde4f"
+					(reference "#PWR025")
+					(unit 1)
+				)

Commit message: added host controlled LEDs to lightman
Parts:
- added D3, D4, D5, D6: LED_R, IMNOTWOPR:Wire_LED, symbol IMNOTWOPR:LED_R
- added R10, R11, R12, R13: 1k, Resistor_THT:R_Axial_DIN0207_L6.3mm_D2.5mm_P2.54mm_Vertical, symbol IMNOTWOPR:R_Vertical
- R1: footprint IMNOTWOPR:R_Axial_DIN0207_P400mil -> Resistor_THT:R_Axial_DIN0207_L6.3mm_D2.5mm_P2.54mm_Vertical
Connections:
- net GND: now also D3.1 (K), D4.1 (K), D5.1 (K), D6.1 (K)
- net L1_LED: now reaches A1.14 (GPIO10)
- net L1_LED: now also R10.2
- net L2_LED: now reaches A1.15 (GPIO11)
- net L2_LED: now also R11.2
- net L3_LED: now reaches A1.16 (GPIO12)
- net L3_LED: now also R12.2
- net L4_LED: now reaches A1.31 (GPIO26_ADC0)
- net L4_LED: now also R13.2
- new net: D4.2 (A), R11.1
- new net: D5.2 (A), R12.1
- new net: D6.2 (A), R13.1
- new net: D3.2 (A), R10.1
- no-connect marks 32 -> 28
