File: modules/P9V/P9V.kicad_pcb (KiCad board)
At the start: 2 copper layers, 160 x 100 mm, 23 parts, among them J1 CardConnector, J2 OUT_1, J3 OUT_2, J4 OUT_3, U1 L7809, U2 L7809

Commit message: P9V module and panel first iteration
Parts:
- moved J2 20.9 mm to (90.3, 65.8)
- moved D1 20.7 mm to (90.3, 55.0)
- moved J4 20.4 mm to (90.3, 129.3)
- moved D2 20.3 mm to (90.3, 82.9)
- moved D3 20.3 mm to (90.3, 118.5)
- moved J3 20.3 mm to (90.3, 95.0)
- moved R1 14.5 mm to (103.0, 53.1)
- moved R2 14.0 mm to (103.0, 81.0)
- moved R3 14.0 mm to (103.0, 116.6)
Routing:
- net GND: track 808.5 -> 626.3 mm
- net +9V_2: track 77.4 -> 56.8 mm
- net +9V_1: track 74.4 -> 55.6 mm
- net +12V_2: track 316.1 -> 307.6 mm
- net Net-(D3-A): track 12.7 -> 6.35 mm
- net Net-(D2-A): track 12.7 -> 6.35 mm
- net Net-(D1-A): track 12.7 -> 6.35 mm
- added copper zone on B.Cu, net +12V_2
- added copper zone on F.Cu, net +12V_2
