File: modules/RAM/RAM.kicad_pcb (KiCad board)
At the start: 2 copper layers, 160 x 100 mm, 37 parts, among them J1 CardConnector, SW1 PAGE SEL 1, SW2 SW_DIP_x04, SW3 SW_DIP_x04, SW4 SW_DIP_x04, U1 HM6264, U10 74HCT688, U11 74HCT688, U12 74HCT00, U13 74HCT32, U2 HM6264, U3 HM6264, U4 HM6264, U5 74AHCT245, U6 74AHCT541, U7 74AHCT541, U8 74HCT688, U9 74HCT688

Commit message: work on RAM and bus terminator
Parts:
- SW2: value SW_DIP_x04 -> PAGE SEL 2
- moved C1 2.54 mm to (181.8, 54.4)
- moved C10 2.54 mm to (190.7, 111.5)
- moved C13 2.54 mm to (190.7, 55.6)
- moved C14 2.54 mm to (190.7, 83.6)
- moved C6 2.54 mm to (175.4, 103.9)
- moved C9 2.54 mm to (175.4, 78.5)
- moved U12 2.54 mm to (175.4, 91.2)
- moved U13 2.54 mm to (175.4, 116.6)
- moved U5 2.54 mm to (190.7, 125.5)
- moved U6 2.54 mm to (190.7, 69.6)
- moved U7 2.54 mm to (190.7, 97.5)
Connections:
- J1 pad a10: unconnected-(J1A-A_{14}-Pada10) -> Net-(J1A-A_{14})
- J1 pad a11: unconnected-(J1A-A_{15}-Pada11) -> Net-(J1A-A_{15})
- J1 pad a3: +12V -> unconnected-(J1A-+12V-Pada3)
- J1 pad a30: +12V -> unconnected-(J1A-+12V-Pada30)
- J1 pad a4: unconnected-(J1A-A_{8}-Pada4) -> Net-(J1A-A_{8})
- J1 pad a5: unconnected-(J1A-A_{9}-Pada5) -> Net-(J1A-A_{9})
- J1 pad a6: unconnected-(J1A-A_{10}-Pada6) -> Net-(J1A-A_{10})
- J1 pad a7: unconnected-(J1A-A_{11}-Pada7) -> Net-(J1A-A_{11})
- J1 pad a8: unconnected-(J1A-A_{12}-Pada8) -> Net-(J1A-A_{12})
- J1 pad a9: unconnected-(J1A-A_{13}-Pada9) -> Net-(J1A-A_{13})
- J1 pad b10: unconnected-(J1B-A_{6}-Padb10) -> Net-(J1B-A_{6})
- J1 pad b11: unconnected-(J1B-A_{7}-Padb11) -> Net-(J1B-A_{7})
- J1 pad b14: Net-(J1B-R/W) -> /R/W
- J1 pad b15: Net-(J1B-VALID) -> /#VALID
- J1 pad b16: unconnected-(J1B-D_{0}-Padb16) -> Net-(J1B-D_{0})
- J1 pad b17: unconnected-(J1B-D_{1}-Padb17) -> Net-(J1B-D_{1})
- J1 pad b18: unconnected-(J1B-D_{2}-Padb18) -> Net-(J1B-D_{2})
- J1 pad b19: unconnected-(J1B-D_{3}-Padb19) -> Net-(J1B-D_{3})
- J1 pad b20: unconnected-(J1B-D_{4}-Padb20) -> Net-(J1B-D_{4})
- J1 pad b21: unconnected-(J1B-D_{5}-Padb21) -> Net-(J1B-D_{5})
- J1 pad b22: unconnected-(J1B-D_{6}-Padb22) -> Net-(J1B-D_{6})
- J1 pad b23: unconnected-(J1B-D_{7}-Padb23) -> Net-(J1B-D_{7})
- J1 pad b3: -12V -> unconnected-(J1B--12V-Padb3)
- J1 pad b30: -12V -> unconnected-(J1B--12V-Padb30)
- J1 pad b4: unconnected-(J1B-A_{0}-Padb4) -> Net-(J1B-A_{0})
- J1 pad b5: unconnected-(J1B-A_{1}-Padb5) -> Net-(J1B-A_{1})
- J1 pad b6: unconnected-(J1B-A_{2}-Padb6) -> Net-(J1B-A_{2})
- J1 pad b7: unconnected-(J1B-A_{3}-Padb7) -> Net-(J1B-A_{3})
- J1 pad b8: unconnected-(J1B-A_{4}-Padb8) -> Net-(J1B-A_{4})
- J1 pad b9: unconnected-(J1B-A_{5}-Padb9) -> Net-(J1B-A_{5})
- RN2 pad 1: unconnected-(RN2-common-Pad1) -> GND
- RN2 pad 2: unconnected-(RN2-R1-Pad2) -> Net-(RN2-R1)
- RN2 pad 3: unconnected-(RN2-R2-Pad3) -> Net-(RN2-R2)
- RN2 pad 4: unconnected-(RN2-R3-Pad4) -> Net-(RN2-R3)
- RN2 pad 5: unconnected-(RN2-R4-Pad5) -> /RAM2_DISABLE
- SW2 pad 1: unconnected-(SW2-Pad1) -> +5V
- SW2 pad 2: unconnected-(SW2-Pad2) -> +5V
- SW2 pad 3: unconnected-(SW2-Pad3) -> +5V
- SW2 pad 4: unconnected-(SW2-Pad4) -> +5V
- SW2 pad 5: unconnected-(SW2-Pad5) -> Net-(RN2-R1)
- SW2 pad 6: unconnected-(SW2-Pad6) -> Net-(RN2-R2)
- SW2 pad 7: unconnected-(SW2-Pad7) -> Net-(RN2-R3)
- SW2 pad 8: unconnected-(SW2-Pad8) -> /RAM2_DISABLE
- U1 pad 20: /#RAM1_SELECT -> unconnected-(U1A-CS_{1}-Pad20)
- U1 pad 26: unconnected-(U1A-CS_{2}-Pad26) -> +5V
- U12 pad 1: Net-(J1B-R/W) -> /R/W
- U12 pad 2: Net-(J1B-R/W) -> /R/W
- U13 pad 1: Net-(J1B-VALID) -> /R/W
- U13 pad 2: Net-(J1B-R/W) -> /#VALID
- U13 pad 5: Net-(J1B-VALID) -> /#VALID
- U13 pad 8: unconnected-(U13-Pad8) -> /#DATA_OE
- U2 pad 26: unconnected-(U2A-CS_{2}-Pad26) -> +5V
- U5 pad 1: unconnected-(U5A-A->B-Pad1) -> /R/W
- U5 pad 11: unconnected-(U5A-B7-Pad11) -> Net-(J1B-D_{7})
- U5 pad 12: unconnected-(U5A-B6-Pad12) -> Net-(J1B-D_{6})
- U5 pad 13: unconnected-(U5A-B5-Pad13) -> Net-(J1B-D_{5})
- U5 pad 14: unconnected-(U5A-B4-Pad14) -> Net-(J1B-D_{4})
- U5 pad 15: unconnected-(U5A-B3-Pad15) -> Net-(J1B-D_{3})
- U5 pad 16: unconnected-(U5A-B2-Pad16) -> Net-(J1B-D_{2})
- U5 pad 17: unconnected-(U5A-B1-Pad17) -> Net-(J1B-D_{1})
- U5 pad 18: unconnected-(U5A-B0-Pad18) -> Net-(J1B-D_{0})
- U5 pad 19: unconnected-(U5A-~{OE}-Pad19) -> /#DATA_OE
- U5 pad 2: unconnected-(U5A-A0-Pad2) -> /D0
- U5 pad 3: unconnected-(U5A-A1-Pad3) -> /D1
- U5 pad 4: unconnected-(U5A-A2-Pad4) -> /D2
- U5 pad 5: unconnected-(U5A-A3-Pad5) -> /D3
- U5 pad 6: unconnected-(U5A-A4-Pad6) -> /D4
- U5 pad 7: unconnected-(U5A-A5-Pad7) -> /D5
- U5 pad 8: unconnected-(U5A-A6-Pad8) -> /D6
- U5 pad 9: unconnected-(U5A-A7-Pad9) -> /D7
- U6 pad 1: unconnected-(U6A-OE_{1}-Pad1) -> GND
- U6 pad 11: unconnected-(U6A-Y_{7}-Pad11) -> /A15
- U6 pad 12: unconnected-(U6A-Y_{6}-Pad12) -> /A14
- U6 pad 13: unconnected-(U6A-Y_{5}-Pad13) -> /A13
- U6 pad 14: unconnected-(U6A-Y_{4}-Pad14) -> /A12
- U6 pad 15: unconnected-(U6A-Y_{3}-Pad15) -> /A11
- U6 pad 16: unconnected-(U6A-Y_{2}-Pad16) -> /A10
- U6 pad 17: unconnected-(U6A-Y_{1}-Pad17) -> /A9
- U6 pad 18: unconnected-(U6A-Y_{0}-Pad18) -> /A8
- U6 pad 19: unconnected-(U6A-OE_{2}-Pad19) -> GND
- U6 pad 2: unconnected-(U6A-A_{0}-Pad2) -> Net-(J1A-A_{8})
- U6 pad 3: unconnected-(U6A-A_{1}-Pad3) -> Net-(J1A-A_{9})
- U6 pad 4: unconnected-(U6A-A_{2}-Pad4) -> Net-(J1A-A_{10})
- U6 pad 5: unconnected-(U6A-A_{3}-Pad5) -> Net-(J1A-A_{11})
- U6 pad 6: unconnected-(U6A-A_{4}-Pad6) -> Net-(J1A-A_{12})
- U6 pad 7: unconnected-(U6A-A_{5}-Pad7) -> Net-(J1A-A_{13})
- U6 pad 8: unconnected-(U6A-A_{6}-Pad8) -> Net-(J1A-A_{14})
- U6 pad 9: unconnected-(U6A-A_{7}-Pad9) -> Net-(J1A-A_{15})
- U7 pad 1: unconnected-(U7A-OE_{1}-Pad1) -> GND
- U7 pad 11: unconnected-(U7A-Y_{7}-Pad11) -> /A7
- U7 pad 12: unconnected-(U7A-Y_{6}-Pad12) -> /A6
- U7 pad 13: unconnected-(U7A-Y_{5}-Pad13) -> /A5
- U7 pad 14: unconnected-(U7A-Y_{4}-Pad14) -> /A4
- U7 pad 15: unconnected-(U7A-Y_{3}-Pad15) -> /A3
- U7 pad 16: unconnected-(U7A-Y_{2}-Pad16) -> /A2
- U7 pad 17: unconnected-(U7A-Y_{1}-Pad17) -> /A1
- U7 pad 18: unconnected-(U7A-Y_{0}-Pad18) -> /A0
- U7 pad 19: unconnected-(U7A-OE_{2}-Pad19) -> GND
- U7 pad 2: unconnected-(U7A-A_{0}-Pad2) -> Net-(J1B-A_{0})
- U7 pad 3: unconnected-(U7A-A_{1}-Pad3) -> Net-(J1B-A_{1})
- U7 pad 4: unconnected-(U7A-A_{2}-Pad4) -> Net-(J1B-A_{2})
- U7 pad 5: unconnected-(U7A-A_{3}-Pad5) -> Net-(J1B-A_{3})
- U7 pad 6: unconnected-(U7A-A_{4}-Pad6) -> Net-(J1B-A_{4})
- U7 pad 7: unconnected-(U7A-A_{5}-Pad7) -> Net-(J1B-A_{5})
- U7 pad 8: unconnected-(U7A-A_{6}-Pad8) -> Net-(J1B-A_{6})
- U7 pad 9: unconnected-(U7A-A_{7}-Pad9) -> Net-(J1B-A_{7})
- U8 pad 19: /#RAM1_SELECT -> unconnected-(U8A-P=R-Pad19)
- U9 pad 1: unconnected-(U9A-G-Pad1) -> /RAM2_DISABLE
- U9 pad 11: unconnected-(U9A-P_{4}-Pad11) -> GND
- U9 pad 12: unconnected-(U9A-R_{4}-Pad12) -> GND
- U9 pad 13: unconnected-(U9A-P_{5}-Pad13) -> GND
- U9 pad 14: unconnected-(U9A-R_{5}-Pad14) -> GND
- U9 pad 15: unconnected-(U9A-P_{6}-Pad15) -> GND
- U9 pad 16: unconnected-(U9A-R_{6}-Pad16) -> GND
- U9 pad 17: unconnected-(U9A-P_{7}-Pad17) -> GND
- U9 pad 18: unconnected-(U9A-R_{7}-Pad18) -> GND
- U9 pad 2: unconnected-(U9A-P_{0}-Pad2) -> Net-(RN2-R3)
- U9 pad 4: unconnected-(U9A-P_{1}-Pad4) -> Net-(RN2-R2)
- U9 pad 6: unconnected-(U9A-P_{2}-Pad6) -> Net-(RN2-R1)
- U9 pad 8: unconnected-(U9A-P_{3}-Pad8) -> GND
- U9 pad 9: unconnected-(U9A-R_{3}-Pad9) -> GND
Routing:
- net Net-(J1B-A_{0}): track 0.00 -> 40.1 mm
- net Net-(J1B-A_{1}): track 0.00 -> 39.4 mm
- net Net-(J1B-A_{2}): track 0.00 -> 39.0 mm
- net Net-(J1B-A_{3}): track 0.00 -> 38.7 mm
- net Net-(J1B-A_{4}): track 0.00 -> 38.3 mm
- net Net-(J1B-A_{5}): track 0.00 -> 37.9 mm
- net Net-(J1B-A_{6}): track 0.00 -> 37.5 mm
- net Net-(J1B-A_{7}): track 0.00 -> 37.2 mm
- net Net-(J1B-D_{6}): track 0.00 -> 32.1 mm
- net Net-(J1B-D_{5}): track 0.00 -> 32.1 mm
- net Net-(J1B-D_{3}): track 0.00 -> 32.1 mm
- net Net-(J1B-D_{1}): track 0.00 -> 32.1 mm
- net Net-(J1B-D_{7}): track 0.00 -> 32.1 mm
- net Net-(J1B-D_{4}): track 0.00 -> 32.1 mm
- net Net-(J1B-D_{2}): track 0.00 -> 32.1 mm
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
Commit message: ram pcb update
Parts:
- added C15: 100n, IMNOTWOPR:C_Rect_P200mil, F.Cu at (175.4, 63.2)
- added D1: LED_R, IMNOTWOPR:Wire_LED, F.Cu at (62.8, 62.9)
- added D2: LED_R, IMNOTWOPR:Wire_LED, F.Cu at (62.8, 67.1)
- added D3: LED_R, IMNOTWOPR:Wire_LED, F.Cu at (62.8, 71.4)
- added D4: LED_R, IMNOTWOPR:Wire_LED, F.Cu at (62.8, 75.6)
- added R1: 1k, IMNOTWOPR:R_Axial_DIN0207_P400mil, F.Cu at (64.3, 82.8)
- added R2: 1k, IMNOTWOPR:R_Axial_DIN0207_P400mil, F.Cu at (64.3, 86.8)
- added R3: 1k, IMNOTWOPR:R_Axial_DIN0207_P400mil, F.Cu at (64.3, 90.7)
- added R4: 1k, IMNOTWOPR:R_Axial_DIN0207_P400mil, F.Cu at (64.3, 94.6)
- added U14: 74HCT04, IMNOTWOPR:DIP-14N, F.Cu at (175.4, 121.7)
- U12: value 74HCT00 -> 74HCT13
- moved U13 43.2 mm to (175.4, 73.4)
- moved C6 7.62 mm to (175.4, 111.5)
- moved C1 6.48 mm to (175.4, 55.6)
- moved C9 5.08 mm to (175.4, 83.6)
- moved U12 2.54 mm to (175.4, 93.7)
Connections:
- RN3 pad 1: unconnected-(RN3-common-Pad1) -> GND
- RN3 pad 2: unconnected-(RN3-R1-Pad2) -> Net-(RN3-R1)
- RN3 pad 3: unconnected-(RN3-R2-Pad3) -> Net-(RN3-R2)
- RN3 pad 4: unconnected-(RN3-R3-Pad4) -> Net-(RN3-R3)
- RN3 pad 5: unconnected-(RN3-R4-Pad5) -> /RAM3_DISABLE
- RN4 pad 1: unconnected-(RN4-common-Pad1) -> GND
- RN4 pad 2: unconnected-(RN4-R1-Pad2) -> Net-(RN4-R1)
- RN4 pad 3: unconnected-(RN4-R2-Pad3) -> Net-(RN4-R2)
- RN4 pad 4: unconnected-(RN4-R3-Pad4) -> Net-(RN4-R3)
- RN4 pad 5: unconnected-(RN4-R4-Pad5) -> Net-(RN4-R4)
- SW3 pad 1: unconnected-(SW3-Pad1) -> +5V
- SW3 pad 2: unconnected-(SW3-Pad2) -> +5V
- SW3 pad 3: unconnected-(SW3-Pad3) -> +5V
- SW3 pad 4: unconnected-(SW3-Pad4) -> +5V
- SW3 pad 5: unconnected-(SW3-Pad5) -> Net-(RN3-R1)
- SW3 pad 6: unconnected-(SW3-Pad6) -> Net-(RN3-R2)
- SW3 pad 7: unconnected-(SW3-Pad7) -> Net-(RN3-R3)
- SW3 pad 8: unconnected-(SW3-Pad8) -> /RAM3_DISABLE
- SW4 pad 1: unconnected-(SW4-Pad1) -> +5V
- SW4 pad 2: unconnected-(SW4-Pad2) -> +5V
- SW4 pad 3: unconnected-(SW4-Pad3) -> +5V
- SW4 pad 4: unconnected-(SW4-Pad4) -> +5V
- SW4 pad 5: unconnected-(SW4-Pad5) -> Net-(RN4-R1)
- SW4 pad 6: unconnected-(SW4-Pad6) -> Net-(RN4-R2)
- SW4 pad 7: unconnected-(SW4-Pad7) -> Net-(RN4-R3)
- SW4 pad 8: unconnected-(SW4-Pad8) -> Net-(RN4-R4)
- U1 pad 10: unconnected-(U1A-A_{0}-Pad10) -> /A0
- U1 pad 11: unconnected-(U1A-D_{0}-Pad11) -> /D0
- U1 pad 12: unconnected-(U1A-D_{1}-Pad12) -> /D1
- U1 pad 13: unconnected-(U1A-D_{2}-Pad13) -> /D2
- U1 pad 15: unconnected-(U1A-D_{3}-Pad15) -> /D3
- U1 pad 16: unconnected-(U1A-D_{4}-Pad16) -> /D4
- U1 pad 17: unconnected-(U1A-D_{5}-Pad17) -> /D5
- U1 pad 18: unconnected-(U1A-D_{6}-Pad18) -> /D6
- U1 pad 19: unconnected-(U1A-D_{7}-Pad19) -> /D7
- U1 pad 2: unconnected-(U1A-A_{12}-Pad2) -> /A12
- U1 pad 20: unconnected-(U1A-CS_{1}-Pad20) -> /#RAM1_SEL
- U1 pad 21: unconnected-(U1A-A_{10}-Pad21) -> /A10
- U1 pad 23: unconnected-(U1A-A_{11}-Pad23) -> /A11
- U1 pad 24: unconnected-(U1A-A_{9}-Pad24) -> /A9
- U1 pad 25: unconnected-(U1A-A_{8}-Pad25) -> /A8
- U1 pad 3: unconnected-(U1A-A_{7}-Pad3) -> /A7
- U1 pad 4: unconnected-(U1A-A_{6}-Pad4) -> /A6
- U1 pad 5: unconnected-(U1A-A_{5}-Pad5) -> /A5
- U1 pad 6: unconnected-(U1A-A_{4}-Pad6) -> /A4
- U1 pad 7: unconnected-(U1A-A_{3}-Pad7) -> /A3
- U1 pad 8: unconnected-(U1A-A_{2}-Pad8) -> /A2
- U1 pad 9: unconnected-(U1A-A_{1}-Pad9) -> /A1
- U10 pad 1: unconnected-(U10A-G-Pad1) -> /RAM3_DISABLE
- U10 pad 11: unconnected-(U10A-P_{4}-Pad11) -> GND
- U10 pad 12: unconnected-(U10A-R_{4}-Pad12) -> GND
- U10 pad 13: unconnected-(U10A-P_{5}-Pad13) -> GND
- U10 pad 14: unconnected-(U10A-R_{5}-Pad14) -> GND
- U10 pad 15: unconnected-(U10A-P_{6}-Pad15) -> GND
- U10 pad 16: unconnected-(U10A-R_{6}-Pad16) -> GND
- U10 pad 17: unconnected-(U10A-P_{7}-Pad17) -> GND
- U10 pad 18: unconnected-(U10A-R_{7}-Pad18) -> GND
- U10 pad 19: unconnected-(U10A-P=R-Pad19) -> /#RAM3_SEL
- U10 pad 2: unconnected-(U10A-P_{0}-Pad2) -> /A15
- U10 pad 3: unconnected-(U10A-R_{0}-Pad3) -> Net-(RN3-R3)
- U10 pad 4: unconnected-(U10A-P_{1}-Pad4) -> /A14
- U10 pad 5: unconnected-(U10A-R_{1}-Pad5) -> Net-(RN3-R2)
- U10 pad 6: unconnected-(U10A-P_{2}-Pad6) -> /A13
- U10 pad 7: unconnected-(U10A-R_{2}-Pad7) -> Net-(RN3-R1)
- U10 pad 8: unconnected-(U10A-P_{3}-Pad8) -> GND
- U10 pad 9: unconnected-(U10A-R_{3}-Pad9) -> GND
- U11 pad 1: unconnected-(U11A-G-Pad1) -> Net-(RN4-R4)
- U11 pad 11: unconnected-(U11A-P_{4}-Pad11) -> GND
- U11 pad 12: unconnected-(U11A-R_{4}-Pad12) -> GND
- U11 pad 13: unconnected-(U11A-P_{5}-Pad13) -> GND
- U11 pad 14: unconnected-(U11A-R_{5}-Pad14) -> GND
- U11 pad 15: unconnected-(U11A-P_{6}-Pad15) -> GND
- U11 pad 16: unconnected-(U11A-R_{6}-Pad16) -> GND
- U11 pad 17: unconnected-(U11A-P_{7}-Pad17) -> GND
- U11 pad 18: unconnected-(U11A-R_{7}-Pad18) -> GND
- U11 pad 19: unconnected-(U11A-P=R-Pad19) -> /#RAM4_SEL
- U11 pad 2: unconnected-(U11A-P_{0}-Pad2) -> /A15
- U11 pad 3: unconnected-(U11A-R_{0}-Pad3) -> Net-(RN4-R3)
- U11 pad 4: unconnected-(U11A-P_{1}-Pad4) -> /A14
- U11 pad 5: unconnected-(U11A-R_{1}-Pad5) -> Net-(RN4-R2)
- U11 pad 6: unconnected-(U11A-P_{2}-Pad6) -> /A13
- U11 pad 7: unconnected-(U11A-R_{2}-Pad7) -> Net-(RN4-R1)
- U11 pad 8: unconnected-(U11A-P_{3}-Pad8) -> GND
- U11 pad 9: unconnected-(U11A-R_{3}-Pad9) -> GND
- U12 pad 1: /R/W -> /#RAM1_SEL
- U12 pad 10: unconnected-(U12-Pad10) -> GND
- U12 pad 12: unconnected-(U12-Pad12) -> GND
- U12 pad 13: unconnected-(U12-Pad13) -> GND
- U12 pad 2: /R/W -> /#RAM2_SEL
- U12 pad 3: Net-(U12-Pad3) -> unconnected-(U12C-NC-Pad3)
- U12 pad 4: unconnected-(U12-Pad4) -> /#RAM3_SEL
- U12 pad 5: unconnected-(U12-Pad5) -> /#RAM4_SEL
- U12 pad 6: unconnected-(U12-Pad6) -> Net-(U12-Pad6)
- U12 pad 9: unconnected-(U12-Pad9) -> GND
- U13 pad 10: unconnected-(U13-Pad10) -> /#LOCAL
- U13 pad 12: unconnected-(U13-Pad12) -> GND
- U13 pad 13: unconnected-(U13-Pad13) -> GND
- U13 pad 4: Net-(U12-Pad3) -> Net-(U13-Pad4)
- U13 pad 9: unconnected-(U13-Pad9) -> /#VALID
- U2 pad 10: unconnected-(U2A-A_{0}-Pad10) -> /A0
- U2 pad 11: unconnected-(U2A-D_{0}-Pad11) -> /D0
- U2 pad 12: unconnected-(U2A-D_{1}-Pad12) -> /D1
- U2 pad 13: unconnected-(U2A-D_{2}-Pad13) -> /D2
- U2 pad 15: unconnected-(U2A-D_{3}-Pad15) -> /D3
- U2 pad 16: unconnected-(U2A-D_{4}-Pad16) -> /D4
- U2 pad 17: unconnected-(U2A-D_{5}-Pad17) -> /D5
- U2 pad 18: unconnected-(U2A-D_{6}-Pad18) -> /D6
- U2 pad 19: unconnected-(U2A-D_{7}-Pad19) -> /D7
- U2 pad 2: unconnected-(U2A-A_{12}-Pad2) -> /A12
- U2 pad 20: unconnected-(U2A-CS_{1}-Pad20) -> /#RAM2_SEL
- U2 pad 21: unconnected-(U2A-A_{10}-Pad21) -> /A10
- U2 pad 22: unconnected-(U2A-OE-Pad22) -> /#RAM_OE
- U2 pad 23: unconnected-(U2A-A_{11}-Pad23) -> /A11
- U2 pad 24: unconnected-(U2A-A_{9}-Pad24) -> /A9
- U2 pad 25: unconnected-(U2A-A_{8}-Pad25) -> /A8
- U2 pad 27: unconnected-(U2A-WE-Pad27) -> /#RAM_WE
- U2 pad 3: unconnected-(U2A-A_{7}-Pad3) -> /A7
- U2 pad 4: unconnected-(U2A-A_{6}-Pad4) -> /A6
- U2 pad 5: unconnected-(U2A-A_{5}-Pad5) -> /A5
- U2 pad 6: unconnected-(U2A-A_{4}-Pad6) -> /A4
- U2 pad 7: unconnected-(U2A-A_{3}-Pad7) -> /A3
- U2 pad 8: unconnected-(U2A-A_{2}-Pad8) -> /A2
- U2 pad 9: unconnected-(U2A-A_{1}-Pad9) -> /A1
- U3 pad 10: unconnected-(U3A-A_{0}-Pad10) -> /A0
- U3 pad 11: unconnected-(U3A-D_{0}-Pad11) -> /D0
- U3 pad 12: unconnected-(U3A-D_{1}-Pad12) -> /D1
- U3 pad 13: unconnected-(U3A-D_{2}-Pad13) -> /D2
- U3 pad 15: unconnected-(U3A-D_{3}-Pad15) -> /D3
- U3 pad 16: unconnected-(U3A-D_{4}-Pad16) -> /D4
- U3 pad 17: unconnected-(U3A-D_{5}-Pad17) -> /D5
- U3 pad 18: unconnected-(U3A-D_{6}-Pad18) -> /D6
- U3 pad 19: unconnected-(U3A-D_{7}-Pad19) -> /D7
- U3 pad 2: unconnected-(U3A-A_{12}-Pad2) -> /A12
- U3 pad 20: unconnected-(U3A-CS_{1}-Pad20) -> /#RAM3_SEL
- U3 pad 21: unconnected-(U3A-A_{10}-Pad21) -> /A10
- U3 pad 22: unconnected-(U3A-OE-Pad22) -> /#RAM_OE
- U3 pad 23: unconnected-(U3A-A_{11}-Pad23) -> /A11
- U3 pad 24: unconnected-(U3A-A_{9}-Pad24) -> /A9
- U3 pad 25: unconnected-(U3A-A_{8}-Pad25) -> /A8
- U3 pad 26: unconnected-(U3A-CS_{2}-Pad26) -> +5V
- U3 pad 27: unconnected-(U3A-WE-Pad27) -> /#RAM_WE
- U3 pad 3: unconnected-(U3A-A_{7}-Pad3) -> /A7
- U3 pad 4: unconnected-(U3A-A_{6}-Pad4) -> /A6
- U3 pad 5: unconnected-(U3A-A_{5}-Pad5) -> /A5
- U3 pad 6: unconnected-(U3A-A_{4}-Pad6) -> /A4
- U3 pad 7: unconnected-(U3A-A_{3}-Pad7) -> /A3
- U3 pad 8: unconnected-(U3A-A_{2}-Pad8) -> /A2
- U3 pad 9: unconnected-(U3A-A_{1}-Pad9) -> /A1
- U4 pad 10: unconnected-(U4A-A_{0}-Pad10) -> /A0
- U4 pad 11: unconnected-(U4A-D_{0}-Pad11) -> /D0
- U4 pad 12: unconnected-(U4A-D_{1}-Pad12) -> /D1
- U4 pad 13: unconnected-(U4A-D_{2}-Pad13) -> /D2
- U4 pad 15: unconnected-(U4A-D_{3}-Pad15) -> /D3
- U4 pad 16: unconnected-(U4A-D_{4}-Pad16) -> /D4
- U4 pad 17: unconnected-(U4A-D_{5}-Pad17) -> /D5
- U4 pad 18: unconnected-(U4A-D_{6}-Pad18) -> /D6
- U4 pad 19: unconnected-(U4A-D_{7}-Pad19) -> /D7
- U4 pad 2: unconnected-(U4A-A_{12}-Pad2) -> /A12
- U4 pad 20: unconnected-(U4A-CS_{1}-Pad20) -> /#RAM4_SEL
- U4 pad 21: unconnected-(U4A-A_{10}-Pad21) -> /A10
- U4 pad 22: unconnected-(U4A-OE-Pad22) -> /#RAM_OE
- U4 pad 23: unconnected-(U4A-A_{11}-Pad23) -> /A11
- U4 pad 24: unconnected-(U4A-A_{9}-Pad24) -> /A9
- U4 pad 25: unconnected-(U4A-A_{8}-Pad25) -> /A8
- U4 pad 26: unconnected-(U4A-CS_{2}-Pad26) -> +5V
- U4 pad 27: unconnected-(U4A-WE-Pad27) -> /#RAM_WE
- U4 pad 3: unconnected-(U4A-A_{7}-Pad3) -> /A7
- U4 pad 4: unconnected-(U4A-A_{6}-Pad4) -> /A6
- U4 pad 5: unconnected-(U4A-A_{5}-Pad5) -> /A5
- U4 pad 6: unconnected-(U4A-A_{4}-Pad6) -> /A4
- U4 pad 7: unconnected-(U4A-A_{3}-Pad7) -> /A3
- U4 pad 8: unconnected-(U4A-A_{2}-Pad8) -> /A2
- U4 pad 9: unconnected-(U4A-A_{1}-Pad9) -> /A1
- U8 pad 19: unconnected-(U8A-P=R-Pad19) -> /#RAM1_SEL
- U8 pad 2: Net-(RN1-R3) -> /A15
- U8 pad 3: unconnected-(U8A-R_{0}-Pad3) -> Net-(RN1-R3)
- U8 pad 4: Net-(RN1-R2) -> /A14
- U8 pad 5: unconnected-(U8A-R_{1}-Pad5) -> Net-(RN1-R2)
- U8 pad 6: Net-(RN1-R1) -> /A13
- U8 pad 7: unconnected-(U8A-R_{2}-Pad7) -> Net-(RN1-R1)
- U9 pad 19: unconnected-(U9A-P=R-Pad19) -> /#RAM2_SEL
- U9 pad 2: Net-(RN2-R3) -> /A15
- U9 pad 3: unconnected-(U9A-R_{0}-Pad3) -> Net-(RN2-R3)
- U9 pad 4: Net-(RN2-R2) -> /A14
- U9 pad 5: unconnected-(U9A-R_{1}-Pad5) -> Net-(RN2-R2)
- U9 pad 6: Net-(RN2-R1) -> /A13
- U9 pad 7: unconnected-(U9A-R_{2}-Pad7) -> Net-(RN2-R1)
Routing:
- net GND: track 8.67 -> 462.1 mm
- net +5V: track 0.00 -> 342.2 mm
- net /D0: track 0.00 -> 114.2 mm
- net /A3: track 0.00 -> 114.2 mm
- net /A1: track 0.00 -> 114.2 mm
- net /A0: track 0.00 -> 114.2 mm
- net /A7: track 0.00 -> 114.2 mm
- net /A5: track 0.00 -> 114.2 mm
- net /A6: track 0.00 -> 114.2 mm
- net /A4: track 0.00 -> 114.2 mm
- net /A12: track 0.00 -> 114.2 mm
- net /A2: track 0.00 -> 114.2 mm
- net /D2: track 0.00 -> 114.2 mm
- net /D1: track 0.00 -> 114.2 mm
- net /D5: track 0.00 -> 98.4 mm
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
Commit message: track work for ram
Parts:
- R1, R2, R3, R4: footprint IMNOTWOPR:R_Axial_DIN0207_P400mil -> Resistor_THT:R_Axial_DIN0207_L6.3mm_D2.5mm_P2.54mm_Vertical
- moved R2 104.8 mm to (156.4, 136.9), turned to 90 degrees
- moved R3 100.8 mm to (156.4, 131.8), turned to 90 degrees
- moved R4 97.5 mm to (156.4, 126.8), turned to 90 degrees
- moved D1 97.3 mm to (143.0, 117.9)
- moved R1 93.0 mm to (141.8, 134.4), turned to 90 degrees
- moved D2 88.4 mm to (135.4, 117.6)
- moved D3 88.4 mm to (135.4, 121.9)
- moved D4 88.4 mm to (135.4, 126.1)
- moved SW2 80.1 mm to (99.3, 124.2)
- moved C8 73.3 mm to (122.1, 134.4), turned to 0 degrees
- moved C5 70.7 mm to (84.0, 136.9), turned to 0 degrees
- moved C3 68.7 mm to (66.2, 136.9), turned to 0 degrees
- moved C4 65.4 mm to (104.3, 129.3), turned to 0 degrees
- moved C15 59.9 mm to (193.2, 120.4)
- moved C9 59.9 mm to (193.2, 140.7)
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Routing:
- net GND: track 462.1 -> 71.7 mm
- net +5V: track 342.2 -> 143.5 mm
- net /#RAM4_SEL: track 94.6 -> 0.00 mm
- net /A15: track 79.4 -> 0.00 mm
- net /A14: track 79.4 -> 0.00 mm
- net /A13: track 79.4 -> 0.00 mm
- net /#RAM3_SEL: track 68.1 -> 0.00 mm
- net Net-(RN4-R3): track 44.5 -> 0.00 mm
- net /#RAM2_SEL: track 42.7 -> 0.00 mm
- net /A3: track 114.2 -> 71.7 mm
- net /A1: track 114.2 -> 71.7 mm
- net /D0: track 114.2 -> 71.7 mm
- net /A5: track 114.2 -> 71.7 mm
- net /A7: track 114.2 -> 71.7 mm
- net /A6: track 114.2 -> 71.7 mm
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