File: modules/RAM/RAM.kicad_sch (KiCad schematic)
At the start: 37 parts, among them J1 CardConnector, SW1 PAGE SEL 1, SW2 SW_DIP_x04, SW3 SW_DIP_x04, SW4 SW_DIP_x04, U1 HM6264, U10 74HCT688, U11 74HCT688, U12 74HCT00, U13 74HCT32, U2 HM6264, U3 HM6264, U4 HM6264, U5 74AHCT245, U6 74AHCT541, U7 74AHCT541, U8 74HCT688, U9 74HCT688

Commit message: work on RAM and bus terminator
Parts:
- added unit 1 of U10
- added unit 1 of U11
- added unit 1 of U3
- added unit 1 of U4
- SW2: value SW_DIP_x04 -> PAGE SEL 2
Connections:
- net +5V: now also SW2.1, SW2.2, SW2.3, SW2.4, U1.26 (CS_{2}), U2.26 (CS_{2})
- net GND: now also RN2.1 (common), U6.1 (OE_{1}), U6.19 (OE_{2}), U7.1 (OE_{1}), U7.19 (OE_{2}), U9.11 (P_{4}), U9.12 (R_{4}), U9.13 (P_{5}), U9.14 (R_{5}), U9.15 (P_{6}), U9.16 (R_{6}), U9.17 (P_{7}), U9.18 (R_{7}), U9.8 (P_{3}), U9.9 (R_{3})
- net at J1.b10 (A_{6}): now also U7.8 (A_{6})
- net at J1.b11 (A_{7}): now also U7.9 (A_{7})
- net R/W: now reaches J1.b14 (R/W), U12.1, U12.2
- net R/W: now also U13.1, U5.1 (A->B); no longer U13.2
- net #VALID: now reaches J1.b15 (VALID), U13.5
- net #VALID: now also U13.2; no longer U13.1
- net at J1.b16 (D_{0}): now also U5.18 (B0)
- net at J1.b17 (D_{1}): now also U5.17 (B1)
- net at J1.b18 (D_{2}): now also U5.16 (B2)
- net at J1.b19 (D_{3}): now also U5.15 (B3)
- net at J1.b20 (D_{4}): now also U5.14 (B4)
- net at J1.b21 (D_{5}): now also U5.13 (B5)
- net at J1.b22 (D_{6}): now also U5.12 (B6)
- net at J1.b23 (D_{7}): now also U5.11 (B7)
- net at J1.b4 (A_{0}): now also U7.2 (A_{0})
- net at J1.b5 (A_{1}): now also U7.3 (A_{1})
- net at J1.b6 (A_{2}): now also U7.4 (A_{2})
- net at J1.b7 (A_{3}): now also U7.5 (A_{3})
- net at J1.b8 (A_{4}): now also U7.6 (A_{4})
- net at J1.b9 (A_{5}): now also U7.7 (A_{5})
- net at RN2.2 (R1): now also SW2.5, U9.6 (P_{2})
- net at RN2.3 (R2): now also SW2.6, U9.4 (P_{1})
- net at RN2.4 (R3): now also SW2.7, U9.2 (P_{0})
- net RAM2_DISABLE: now reaches RN2.5 (R4)
- net RAM2_DISABLE: now also SW2.8, U9.1 (G)
- net #DATA_OE: now reaches U5.19 (~{OE})
- net #DATA_OE: now also U13.8
- net D0: now reaches U5.2 (A0)
- net D1: now reaches U5.3 (A1)
- net D2: now reaches U5.4 (A2)
- net D3: now reaches U5.5 (A3)
- net D4: now reaches U5.6 (A4)
- net D5: now reaches U5.7 (A5)
- net D6: now reaches U5.8 (A6)
- net D7: now reaches U5.9 (A7)
- net at J1.a10 (A_{14}): now also U6.8 (A_{6})
- net at J1.a11 (A_{15}): now also U6.9 (A_{7})
- net at J1.a4 (A_{8}): now also U6.2 (A_{0})
- net at J1.a5 (A_{9}): now also U6.3 (A_{1})
- net at J1.a6 (A_{10}): now also U6.4 (A_{2})
- net at J1.a7 (A_{11}): now also U6.5 (A_{3})
- net at J1.a8 (A_{12}): now also U6.6 (A_{4})
- net at J1.a9 (A_{13}): now also U6.7 (A_{5})
- net A15: now reaches U6.11 (Y_{7})
- net A14: now reaches U6.12 (Y_{6})
- net A13: now reaches U6.13 (Y_{5})
- net A12: now reaches U6.14 (Y_{4})
- net A11: now reaches U6.15 (Y_{3})
- net A10: now reaches U6.16 (Y_{2})
- net A9: now reaches U6.17 (Y_{1})
- net A8: now reaches U6.18 (Y_{0})
- net A7: now reaches U7.11 (Y_{7})
- net A6: now reaches U7.12 (Y_{6})
- net A5: now reaches U7.13 (Y_{5})
- net A4: now reaches U7.14 (Y_{4})
- net A3: now reaches U7.15 (Y_{3})
- net A2: now reaches U7.16 (Y_{2})
- net A1: now reaches U7.17 (Y_{1})
- net A0: now reaches U7.18 (Y_{0})
- net #RAM1_SELECT: no longer names the net of U1.20 (CS_{1})
- net #RAM1_SELECT: no longer U8.19 (P=R)
- net +12V: no longer names the net of J1.a3 (+12V)
- net +12V: no longer J1.a30 (+12V)
- net -12V: no longer names the net of J1.b3 (-12V)
- net -12V: no longer J1.b30 (-12V)
- no-connect marks 75 -> 55
Other:
- moved on the sheet: RN1, RN2, RN3, RN4, SW1, SW2, SW3, SW4

Commit message: ram pcb update
Parts:
- removed U12: 74HCT00, IMNOTWOPR:DIP-14N, symbol IMNOTWOPR:74HCT00
- added C15: 100n, IMNOTWOPR:C_Rect_P200mil, symbol IMNOTWOPR:C
- added D1, D2, D3, D4: LED_R, IMNOTWOPR:Wire_LED, symbol IMNOTWOPR:LED_R
- added R1, R2, R3, R4: 1k, IMNOTWOPR:R_Axial_DIN0207_P400mil, symbol IMNOTWOPR:R_Horizontal
- added U12: 74HCT13, IMNOTWOPR:DIP-14N, symbol IMNOTWOPR:74HCT13
- added U14: 74HCT04, IMNOTWOPR:DIP-14N, symbol IMNOTWOPR:74HCT04
Connections:
- net #RAM_OE: now also U2.22 (OE), U3.22 (OE), U4.22 (OE)
- net #RAM_WE: now also U2.27 (WE), U3.27 (WE), U4.27 (WE)
- net #VALID: now also U13.9
- net +5V: now also SW3.1, SW3.2, SW3.3, SW3.4, SW4.1, SW4.2, SW4.3, SW4.4, U3.26 (CS_{2}), U4.26 (CS_{2}), C15.1, U12.14 (VCC), U14.14 (V_{CC})
- net A0: now also U1.10 (A_{0}), U2.10 (A_{0}), U3.10 (A_{0}), U4.10 (A_{0})
- net A1: now also U1.9 (A_{1}), U2.9 (A_{1}), U3.9 (A_{1}), U4.9 (A_{1})
- net A10: now also U1.21 (A_{10}), U2.21 (A_{10}), U3.21 (A_{10}), U4.21 (A_{10})
- net A11: now also U1.23 (A_{11}), U2.23 (A_{11}), U3.23 (A_{11}), U4.23 (A_{11})
- net A12: now also U1.2 (A_{12}), U2.2 (A_{12}), U3.2 (A_{12}), U4.2 (A_{12})
- net A13: now also U10.6 (P_{2}), U11.6 (P_{2}), U8.6 (P_{2}), U9.6 (P_{2})
- net A14: now also U10.4 (P_{1}), U11.4 (P_{1}), U8.4 (P_{1}), U9.4 (P_{1})
- net A15: now also U10.2 (P_{0}), U11.2 (P_{0}), U8.2 (P_{0}), U9.2 (P_{0})
- net A2: now also U1.8 (A_{2}), U2.8 (A_{2}), U3.8 (A_{2}), U4.8 (A_{2})
- net A3: now also U1.7 (A_{3}), U2.7 (A_{3}), U3.7 (A_{3}), U4.7 (A_{3})
- net A4: now also U1.6 (A_{4}), U2.6 (A_{4}), U3.6 (A_{4}), U4.6 (A_{4})
- net A5: now also U1.5 (A_{5}), U2.5 (A_{5}), U3.5 (A_{5}), U4.5 (A_{5})
- net A6: now also U1.4 (A_{6}), U2.4 (A_{6}), U3.4 (A_{6}), U4.4 (A_{6})
- net A7: now also U1.3 (A_{7}), U2.3 (A_{7}), U3.3 (A_{7}), U4.3 (A_{7})
- net A8: now also U1.25 (A_{8}), U2.25 (A_{8}), U3.25 (A_{8}), U4.25 (A_{8})
- net A9: now also U1.24 (A_{9}), U2.24 (A_{9}), U3.24 (A_{9}), U4.24 (A_{9})
- net D0: now also U1.11 (D_{0}), U2.11 (D_{0}), U3.11 (D_{0}), U4.11 (D_{0})
- net D1: now also U1.12 (D_{1}), U2.12 (D_{1}), U3.12 (D_{1}), U4.12 (D_{1})
- net D2: now also U1.13 (D_{2}), U2.13 (D_{2}), U3.13 (D_{2}), U4.13 (D_{2})
- net D3: now also U1.15 (D_{3}), U2.15 (D_{3}), U3.15 (D_{3}), U4.15 (D_{3})
- net D4: now also U1.16 (D_{4}), U2.16 (D_{4}), U3.16 (D_{4}), U4.16 (D_{4})
- net D5: now also U1.17 (D_{5}), U2.17 (D_{5}), U3.17 (D_{5}), U4.17 (D_{5})
- net D6: now also U1.18 (D_{6}), U2.18 (D_{6}), U3.18 (D_{6}), U4.18 (D_{6})
- net D7: now also U1.19 (D_{7}), U2.19 (D_{7}), U3.19 (D_{7}), U4.19 (D_{7})
- net GND: now also RN3.1 (common), RN4.1 (common), U10.11 (P_{4}), U10.12 (R_{4}), U10.13 (P_{5}), U10.14 (R_{5}), U10.15 (P_{6}), U10.16 (R_{6}), U10.17 (P_{7}), U10.18 (R_{7}), U10.8 (P_{3}), U10.9 (R_{3}), U11.11 (P_{4}), U11.12 (R_{4}), U11.13 (P_{5}), U11.14 (R_{5}), U11.15 (P_{6}), U11.16 (R_{6}), U11.17 (P_{7}), U11.18 (R_{7}), U11.8 (P_{3}), U11.9 (R_{3}), U13.12, U13.13, C15.2, D1.1 (K), D2.1 (K), D3.1 (K), D4.1 (K), U12.10, U12.12, U12.13, U12.7 (GND), U12.9, U14.7 (GND)
- net R/W: now also U14.1
- net #RAM2_SEL: now reaches U2.20 (CS_{1})
- net #RAM2_SEL: now also U9.19 (P=R), U12.2, U14.9
- net at RN1.2 (R1), SW1.5: now also U8.7 (R_{2}); no longer U8.6 (P_{2})
- net at RN1.3 (R2), SW1.6: now also U8.5 (R_{1}); no longer U8.4 (P_{1})
- net at RN1.4 (R3), SW1.7: now also U8.3 (R_{0}); no longer U8.2 (P_{0})
- net at SW3.5: now also RN3.2 (R1), U10.7 (R_{2})
- net at SW3.6: now also RN3.3 (R2), U10.5 (R_{1})
- net at SW3.7: now also RN3.4 (R3), U10.3 (R_{0})
- net RAM3_DISABLE: now reaches SW3.8
- net RAM3_DISABLE: now also RN3.5 (R4), U10.1 (G)
- net at U11.1 (G): now also RN4.5 (R4), SW4.8
- net #RAM4_SEL: now reaches U11.19 (P=R)
- net #RAM4_SEL: now also U4.20 (CS_{1}), U12.5, U14.13
- net at U11.3 (R_{0}): now also RN4.4 (R3), SW4.7
- net at U11.5 (R_{1}): now also RN4.3 (R2), SW4.6
- net at U11.7 (R_{2}): now also RN4.2 (R1), SW4.5
- net at RN2.2 (R1), SW2.5: now also U9.7 (R_{2}); no longer U9.6 (P_{2})
- net at RN2.3 (R2), SW2.6: now also U9.5 (R_{1}); no longer U9.4 (P_{1})
- net at RN2.4 (R3), SW2.7: now also U9.3 (R_{0}); no longer U9.2 (P_{0})
- net #LOCAL: now reaches U13.10
- net #LOCAL: now also U14.4
- net #RAM3_SEL: now reaches U10.19 (P=R)
- net #RAM3_SEL: now also U3.20 (CS_{1}), U12.4, U14.11
- net at U13.4: now also U14.2
- net #RAM1_SEL: now reaches U1.20 (CS_{1})
- net #RAM1_SEL: now also U8.19 (P=R), U12.1, U14.5
- new net: D4.2 (A), R4.2
- new net: U12.6, U14.3
- new net: D1.2 (A), R1.2
- new net: R1.1, U14.6
- new net: R2.1, U14.8
- new net: D2.2 (A), R2.2
- new net: D3.2 (A), R3.2
- new net: R4.1, U14.12
- new net: R3.1, U14.10
- no-connect marks 55 -> 57
Other:
- note added: "OPTIONAL "PAGE IN USE" LEDs"
- moved on the sheet: C1, C10, C11, C12, C13, C14, C2, C3, C4, C5, C6, C7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

Commit message: track work for ram
Parts:
- R1, R2, R3, R4: footprint IMNOTWOPR:R_Axial_DIN0207_P400mil -> Resistor_THT:R_Axial_DIN0207_L6.3mm_D2.5mm_P2.54mm_Vertical
Changed lines of the file:
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@@
 			)
 		)
-		(property "Footprint" "IMNOTWOPR:R_Axial_DIN0207_P400mil"
+		(property "Footprint" "Resistor_THT:R_Axial_DIN0207_L6.3mm_D2.5mm_P2.54mm_Vertical"
 			(at 101.6 215.9 0)
 			(hide yes)
@@
 			)
 		)
-		(property "Footprint" "IMNOTWOPR:R_Axial_DIN0207_P400mil"
+		(property "Footprint" "Resistor_THT:R_Axial_DIN0207_L6.3mm_D2.5mm_P2.54mm_Vertical"
 			(at 101.6 203.2 0)
 			(hide yes)
@@
 			)
 		)
-		(property "Footprint" "IMNOTWOPR:R_Axial_DIN0207_P400mil"
+		(property "Footprint" "Resistor_THT:R_Axial_DIN0207_L6.3mm_D2.5mm_P2.54mm_Vertical"
 			(at 101.6 241.3 0)
 			(hide yes)
@@
 			)
 		)
-		(property "Footprint" "IMNOTWOPR:R_Axial_DIN0207_P400mil"
+		(property "Footprint" "Resistor_THT:R_Axial_DIN0207_L6.3mm_D2.5mm_P2.54mm_Vertical"
 			(at 101.6 228.6 0)
 			(hide yes)
